File: PRopendous/Hardware/PROpendous/PROpendous-Connectors_JTAG.sch (KiCad schematic (older format))
At the start: 25 parts, among them IC16 PRTR, Q1 NCH, U2 USB-B, U4 JTAG

Commit message: Updated files.  DDR SDRAM schematic completed.
Parts:
- removed D2: LED, symbol D_LED
- removed IC16: PRTR, symbol PRTR5V0U2X
- removed JP0, JP1, JP2: JUMPER-3, symbol JUMPER-3
- removed L10: FB, symbol L_MINI
- removed Q1: NCH, symbol MOSFET_N_OPENDOUS
- removed R24, R25: 1M, symbol R_MINI
- removed R26: 12k, symbol R_MINI
- removed R27, R77, R78, R79, R80, R81, R82: 10k, symbol R_MINI
- removed R29: 33, symbol R_MINI
- removed R33: 1k, symbol R_MINI
- removed R73, R74, R75, R76: 4k7, symbol R_MINI
- removed U2: USB-B, symbol USBCONN
- removed U4: JTAG, symbol CONN_JTAG_ARM
- added P1: Serial-JTAG, symbol CONN_4
- added R5: 0, symbol R_MINI
Connections:
- net labels added: VDDIO_3V3
- net labels removed: ARM_TDO, GNDPWR, GPIO0, GPIO1, GPIO2, JTAGSEL, TCK, TDI, TDO, TMS, TRST_N, USB_DM, USB_DP, USB_RREF, USB_VBUS, VBUS, VSUP3, ^JTAG_SRST
- wire segments 76 -> 7
- no-connect marks 2 -> 0
Other:
- note added: "DNP"
- note added: "Serial JTAG Debugger\nhas its own power"
- note removed: "(2N7002)"
- note removed: "(Default)"
- note removed: "(SOT-23)"
- note removed: "0"
- note removed: "1"
- note removed: "1%"
- note removed: "2"
- note removed: "Blink on Error"
- note removed: "Boot Device"
- note removed: "Boot Mode Select"
- note removed: "Boot Status"
- note removed: "DFU"
- note removed: "Debugger can RESET board"
- note removed: "GPIO Pin"
- note removed: "JTAG"
- note removed: "MMC"
- note removed: "Mode Select Jumpers"
- note removed: "NAND"
- note removed: "NOR"
- note removed: "Note: JTAGSEL (JTAG TDO Mux) pulled up to 3V sets ARM-DEBUG Mode"
- note removed: "PRTR5V0U2X"
- note removed: "Reserved"
- note removed: "SPI NOR"
- note removed: "Test"
- note removed: "UART"
- note removed: "USB"

Commit message: Updated PROpendous i.MX233 project.  DDR SDRAM layout is complete.
Parts:
- added C31, C33: 0.1uF, symbol C_MINI
- added C32, C34: 1uF, symbol C_MINI
- added U2: microSD, symbol CONN_MICROSD
- added U3: SD, symbol CONN_SD
Connections:
- net labels removed: SSP1_DETECT-GPMI_CE3N-USB_ID
- wire segments 7 -> 29
- no-connect marks 0 -> 2
Other:
- note added: "3M 29-08-05"
- note added: "3M SD-RSMT-2"
- note added: "Captive"
- note added: "External"

Commit message: Updated PROpendous project.  Schematic is complete but not yet finalized.  Layout partially complete.
Parts:
- added C36: 0.01uF, symbol C_MINI
- added C37: 68uF, symbol CP_TANTALUM_MINI
- added F1: 1206L, symbol FUSE-MINI
- added IC4: AP2171, symbol USB_SWITCH_ACTIVEHIGH
- added IC5: FSUSB20, symbol FSUSB20
- added L3, L4, L5: FB, symbol L_MINI
- added P2: Expansion, symbol CONN_25X2
- added R20, R22, R23: 15k, symbol R_MINI
- added R21: 10k, symbol R_MINI
- added U5: USB-miniB, symbol USBCONN-HOSTCAPABLE
- added U6: USB-A, symbol USBCONN
Connections:
- net labels added: DMa, DMb, DPa, DPb, GNDPWR, TSC_IN1, TSC_IN2, TSC_VBAT2, TSC_VREF, USB_DM, USB_DP, VBUS, VBUS_HOST, VDD5V
- net labels removed: EMI_A00, EMI_A01, EMI_A02, EMI_A03, EMI_A04, EMI_A05, EMI_A06, EMI_A07, EMI_A08, EMI_A09, EMI_A10, EMI_A11, EMI_A12, EMI_BA0, EMI_BA1, EMI_CASn, EMI_CE0n, EMI_CKE, EMI_CLK, EMI_CLKn, EMI_D00, EMI_D01, EMI_D02, EMI_D03, EMI_D04, EMI_D05, EMI_D06, EMI_D07, EMI_D08, EMI_D09, EMI_D10, EMI_D11, EMI_D12, EMI_D13, EMI_D14, EMI_D15, EMI_DQM0, EMI_DQM1, EMI_DQS0, EMI_DQS1, EMI_RASn, EMI_WEn, HPL, HPR, LINE1_INL, LINE1_INR, LRADC1, MIC, VAG, VDAC1, XTALI, XTALO
- wire segments 29 -> 85
- no-connect marks 2 -> 3
Other:
- note added: "AP2171 has Active-High Enable\nand current-limiting"
- note added: "Connecting the board through its USB-miniB connector\nwill power the board by supplying VDD5V. Otherwise\nthe battery is used for power."
- note added: "Expansion Header"
- note added: "Expansion Header Pinout Not Yet Finalized!\nBut these will be the available signals."
- note added: "Littelfuse 1206L035"
- note added: "The FSUSB20 has 7kV of ESD Protection"
- note added: "USB requires 90 Ohm differential impedance which for a\nstandard 1/16" 1oz FR4 double-sided board has been\ncalculated to require 22mil traces at 7mil spacing. Make\nsure to have a solid ground plane underneath the USB lines\nand keep 5x the spacing on either side of the traces (35mil)."
- note added: "When PWM2-GPMI_RDY3 enables the\nUSB Host VBUS Generator it will also\nswitch the active USB connector to USB-A"
- moved on the sheet: C31, C32, C33, C34, P1, R5, U3

Commit message: Minor update to schematic.  Removed USB Power switch and added some notes.
Parts:
- removed C36: 0.01uF, symbol C_MINI
- removed C37: 68uF, symbol CP_TANTALUM_MINI
- removed F1: 1206L, symbol FUSE-MINI
- removed IC4: AP2171, symbol USB_SWITCH_ACTIVEHIGH
- removed L3, L4, L5: FB, symbol L_MINI
- removed R20: 15k, symbol R_MINI
- removed R21: 10k, symbol R_MINI
- added C75: 0.1uF, symbol C_MINI
Connections:
- net labels added: FSUSB20_nOE, GND_USB-B
- net labels removed: VDD5V
- wire segments 85 -> 65
Other:
- note added: "Debug"
- note added: "Storage"
- note added: "USB"
- note added: "USB 90 Ohm differential impedance can also be\naccomplished using 13.4mil traces spaced 8mil\napart with GND traces 7mil outside of either trace\nin a differential coplanar waveguide configuration\nwhen a solid underside GND plane is not available."
- note removed: "AP2171 has Active-High Enable\nand current-limiting"
- note removed: "Connecting the board through its USB-miniB connector\nwill power the board by supplying VDD5V. Otherwise\nthe battery is used for power."
- note removed: "Littelfuse 1206L035"
- moved on the sheet: C31, C32, C33, C34, IC5, R22, R23, U3, U6

Commit message: Updated PROpendous Project.  PCB layout is nearing completion.
Parts:
- removed P2: Expansion, symbol CONN_25X2
- added C77: 0.1uF, symbol C_MINI
- added L18: FB, symbol L_MINI
- added P2: ExpansionA, symbol CONN_17X2
- added P3: ExpansionB, symbol CONN_5X2
- added U4: JTAG, symbol CONN_JTAG_ARM
Connections:
- net labels added: SSP1_DETECT-GPMI_CE3N-USB_ID, USB-A_GND
- wire segments 65 -> 73
- no-connect marks 3 -> 6
Other:
- note added: "ERC Corrections"
- note added: "Expansion Headers"
- note added: "JTAG shares pins with SSP1 so it cannot be used\nat the same time as the external SD card"
- note added: "USB requires 90 Ohm differential impedance which for a\nstandard 1/16" 1oz FR4 double-sided board has been\ncalculated to require 22mil traces at 7mil spacing. Make\nsure to have a solid ground plane underneath the USB lines\nand keep 12mil spacing on either side of the traces to GND."
- note removed: "Expansion Header"
- note removed: "Expansion Header Pinout Not Yet Finalized!\nBut these will be the available signals."
- note removed: "USB 90 Ohm differential impedance can also be\naccomplished using 13.4mil traces spaced 8mil\napart with GND traces 7mil outside of either trace\nin a differential coplanar waveguide configuration\nwhen a solid underside GND plane is not available."
- note removed: "USB requires 90 Ohm differential impedance which for a\nstandard 1/16" 1oz FR4 double-sided board has been\ncalculated to require 22mil traces at 7mil spacing. Make\nsure to have a solid ground plane underneath the USB lines\nand keep 5x the spacing on either side of the traces (35mil)."
- moved on the sheet: P1, R5

Commit message: Updated layout.
Parts:
- U4: value JTAG -> ARM_JTAG
Connections:
- net labels removed: TSC_IN1
- no-connect marks 6 -> 5
Other:
- note added: "GPMI_RDn is on both headers"
Changed lines of the file:
@@
-EESchema Schematic File Version 2  date 24/04/2010 02:27:16
+EESchema Schematic File Version 2  date 25/04/2010 06:05:23
 LIBS:opendous
 LIBS:device
@@
 Sheet 4 8
 Title "PROpendous"
-Date "24 apr 2010"
+Date "25 apr 2010"
 Rev "1.0"
 Comp "Opendous Inc. (www.opendous.org)"
@@
 Comment4 "www.PROpendous.org"
 $EndDescr
+Text Notes 9550 3325 0    30   ~ 0
+GPMI_RDn is on both headers
+Text Notes 7300 2675 0    30   ~ 0
+GPMI_RDn is on both headers
+Text GLabel 8350 2650 0    40   BiDi ~ 0
+GPMI_RDn
 Text Notes 7100 4700 0    40   ~ 0
 JTAG shares pins with SSP1 so it cannot be used\nat the same time as the external SD card
@@
 	1    0    0    -1
 $EndComp
-NoConn ~ 9150 2650
 $Comp
 L CONN_17X2 P2
@@
 Text GLabel 8350 1750 0    40   BiDi ~ 0
 LCD_CS
-Text GLabel 9150 2150 2    40   BiDi ~ 0
+Text GLabel 8350 2150 0    40   BiDi ~ 0
 GPMI_ALE-LCD_D17
 Text GLabel 7300 5300 0    40   BiDi ~ 0
@@
 Text GLabel 9150 1750 2    40   BiDi ~ 0
 LCD_ENABLE-I2C_SCL
-Text GLabel 8350 2250 0    40   BiDi ~ 0
+Text GLabel 9150 2250 2    40   BiDi ~ 0
 GPMI_RDY1-SSP2_CMD
 Text GLabel 9150 3400 2    40   BiDi ~ 0
@@
 Text GLabel 8350 1850 0    40   BiDi ~ 0
 LCD_RESET-GPMI_CE3n
-Text GLabel 9150 2250 2    40   BiDi ~ 0
+Text GLabel 8350 2250 0    40   BiDi ~ 0
 GPMI_D00-LCD_D8-SSP2_DATA0
 Text GLabel 8350 3500 0    40   BiDi ~ 0
@@
 Text GLabel 9150 1850 2    40   BiDi ~ 0
 LCD_WR
-Text GLabel 8350 2350 0    40   BiDi ~ 0
+Text GLabel 9150 2350 2    40   BiDi ~ 0
 GPMI_D01-LCD_D9-SSP2_DATA1
 Text GLabel 9150 3500 2    40   BiDi ~ 0
@@
 Text GLabel 7300 5800 0    40   BiDi ~ 0
 SSP1_CMD-JTAG_TDO
-Text GLabel 8350 1950 0    40   BiDi ~ 0
+Text GLabel 9150 1950 2    40   BiDi ~ 0
 LCD_RS
-Text GLabel 9150 2350 2    40   BiDi ~ 0
+Text GLabel 8350 2350 0    40   BiDi ~ 0
 GPMI_D02-LCD_D10-SSP2_DATA2
 Text GLabel 8350 3600 0    40   BiDi ~ 0
@@
 Text GLabel 7300 5400 0    40   BiDi ~ 0
 SSP1_DATA0-JTAG_TDI
-Text GLabel 9150 1950 2    40   BiDi ~ 0
+Text GLabel 8350 1950 0    40   BiDi ~ 0
 LCD_HSYNC-I2C_SDA
-Text GLabel 8350 2450 0    40   BiDi ~ 0
+Text GLabel 9150 2450 2    40   BiDi ~ 0
 GPMI_D03-LCD_D11-SSP2_DATA3
-Text GLabel 8350 2050 0    40   BiDi ~ 0
+Text GLabel 9150 2050 2    40   BiDi ~ 0
 LCD_VSYNC-LCD_BUSY
-Text GLabel 8350 2550 0    40   BiDi ~ 0
+Text GLabel 9150 2550 2    40   BiDi ~ 0
 GPMI_D05-LCD_D13-SSP2_DATA5
 Text GLabel 7300 5700 0    40   BiDi ~ 0
 SSP1_DATA2-I2C_SDA-JTAG_RTCK
-Text GLabel 9150 2050 2    40   BiDi ~ 0
+Text GLabel 8350 2050 0    40   BiDi ~ 0
 LCD_DOTCK-GPMI_RDY3
-Text GLabel 9150 2450 2    40   BiDi ~ 0
+Text GLabel 8350 2450 0    40   BiDi ~ 0
 GPMI_D04-LCD_D12-SSP2_DATA4
 Text GLabel 7300 5500 0    40   BiDi ~ 0
 SSP1_DATA3-JTAG_TMS
-Text GLabel 8350 2650 0    40   BiDi ~ 0
+Text GLabel 9150 2650 2    40   BiDi ~ 0
 GPMI_D07-LCD_D15-SSP2_DATA7
-Text GLabel 8350 2150 0    40   BiDi ~ 0
+Text GLabel 9150 2150 2    40   BiDi ~ 0
 GPMI_CLE-LCD_D16
-Text GLabel 9150 2550 2    40   BiDi ~ 0
+Text GLabel 8350 2550 0    40   BiDi ~ 0
 GPMI_D06-LCD_D14-SSP2_DATA6
 Text GLabel 8350 1150 0    40   BiDi ~ 0
@@
 AR Path="/49F49582/49F7B888" Ref="U10"  Part="1"
 F 0 "U10" H 7600 5100 50  0000 C CNN
-F 1 "JTAG" H 7800 6200 50  0000 C CNN
+F 1 "ARM_JTAG" H 7800 6200 50  0000 C CNN
 	1    7800 5650
 	1    0    0    -1
 $EndComp
-Text GLabel 10200 3550 2    40   BiDi ~ 0
-TSC_IN1
 Text GLabel 9150 3600 2    40   BiDi ~ 0
 TSC_IN2

Commit message: Updated layout.  Extended expansion connector and moved microSD.
Parts:
- removed P2: ExpansionA, symbol CONN_17X2
- removed P3: ExpansionB, symbol CONN_5X2
- added P2: Expansion, symbol CONN_20X2
Connections:
- net labels removed: TSC_IN2, TSC_VBAT2, TSC_VREF
Other:
- note added: "Expansion Header"
- note removed: "Expansion Headers"
- note removed: "GPMI_RDn is on both headers"
Changed lines of the file:
@@
-EESchema Schematic File Version 2  date 25/04/2010 06:05:23
+EESchema Schematic File Version 2  date 25/04/2010 07:03:32
 LIBS:opendous
 LIBS:device
@@
 Comment4 "www.PROpendous.org"
 $EndDescr
-Text Notes 9550 3325 0    30   ~ 0
-GPMI_RDn is on both headers
-Text Notes 7300 2675 0    30   ~ 0
-GPMI_RDn is on both headers
-Text GLabel 8350 2650 0    40   BiDi ~ 0
-GPMI_RDn
+$Comp
+L CONN_20X2 P2
+U 1 1 4BD415A8
+P 8650 2350
+F 0 "P2" H 8650 3400 60  0000 C CNN
+F 1 "Expansion" V 8650 2350 50  0000 C CNN
+	1    8650 2350
+	1    0    0    -1
+$EndComp
 Text Notes 7100 4700 0    40   ~ 0
 JTAG shares pins with SSP1 so it cannot be used\nat the same time as the external SD card
@@
 	11200 1200 11200 500
 Wire Wire Line
-	8200 1000 8200 950
-Wire Wire Line
-	8200 950  8350 950
-Wire Wire Line
-	8350 950  8350 1050
-Wire Wire Line
-	9150 1050 9300 1050
-Wire Wire Line
-	9300 1050 9300 1000
+	8100 1350 8100 1300
+Wire Wire Line
+	8100 1300 8250 1300
+Wire Wire Line
+	8250 1300 8250 1400
+Wire Wire Line
+	9050 1400 9200 1400
+Wire Wire Line
+	9200 1400 9200 1350
 Wire Wire Line
 	7300 5000 8300 5000
@@
 	7800 5000 7800 4950
 Connection ~ 7800 5000
-$Comp
-L CONN_5X2 P3
-U 1 1 4BD23742
-P 8750 3500
-F 0 "P3" H 8750 3800 60  0000 C CNN
-F 1 "ExpansionB" V 8750 3500 50  0000 C CNN
-	1    8750 3500
-	1    0    0    -1
-$EndComp
 NoConn ~ 7300 6100
 NoConn ~ 7300 6000
@@
 L GND #PWR034
 U 1 1 4BD22797
-P 8200 1000
-F 0 "#PWR034" H 8200 1000 30  0001 C CNN
-F 1 "GND" H 8200 930 30  0001 C CNN
-	1    8200 1000
+P 8100 1350
+F 0 "#PWR034" H 8100 1350 30  0001 C CNN
+F 1 "GND" H 8100 1280 30  0001 C CNN
+	1    8100 1350
 	1    0    0    -1
 $EndComp
@@
 L VDDIO_3V3 #PWR035
 U 1 1 4BD22796
-P 9300 1000
-F 0 "#PWR035" H 9300 1100 30  0001 C CNN
-F 1 "VDDIO_3V3" H 9300 1100 30  0000 C CNN
-	1    9300 1000
-	1    0    0    -1
-$EndComp
-$Comp
-L CONN_17X2 P2
-U 1 1 4BD2276B
-P 8750 1850
-F 0 "P2" H 8750 2750 60  0000 C CNN
-F 1 "ExpansionA" V 8750 1850 50  0000 C CNN
-	1    8750 1850
+P 9200 1350
+F 0 "#PWR035" H 9200 1450 30  0001 C CNN
+F 1 "VDDIO_3V3" H 9200 1450 30  0000 C CNN
+	1    9200 1350
 	1    0    0    -1
 $EndComp
@@
 	1    0    0    -1
 $EndComp
-Text GLabel 8350 3300 0    40   BiDi ~ 0
+Text GLabel 8250 3000 0    40   BiDi ~ 0
 LRADC0
 $Comp
@@
 	1    0    0    -1
 $EndComp
-Text Notes 8200 750  0    80   Italic 16
-Expansion Headers
+Text Notes 8100 1100 0    80   Italic 16
+Expansion Header
 Text Notes 4400 5800 0    40   ~ 0
 When PWM2-GPMI_RDY3 enables the\nUSB Host VBUS Generator it will also\nswitch the active USB connector to USB-A
@@
 Text GLabel 9750 5700 0    40   BiDi ~ 0
 PSWITCH
-Text GLabel 8350 1350 0    40   BiDi ~ 0
+Text GLabel 8250 1700 0    40   BiDi ~ 0
 LCD_D00
-Text GLabel 9150 1350 2    40   BiDi ~ 0
+Text GLabel 9050 1700 2    40   BiDi ~ 0
 LCD_D01
-Text GLabel 8350 1450 0    40   BiDi ~ 0
+Text GLabel 8250 1800 0    40   BiDi ~ 0
 LCD_D02
-Text GLabel 9150 1450 2    40   BiDi ~ 0
+Text GLabel 9050 1800 2    40   BiDi ~ 0
 LCD_D03
-Text GLabel 8350 1550 0    40   BiDi ~ 0
+Text GLabel 8250 1900 0    40   BiDi ~ 0
 LCD_D04
-Text GLabel 9150 1550 2    40   BiDi ~ 0
+Text GLabel 9050 1900 2    40   BiDi ~ 0
 LCD_D05
-Text GLabel 8350 1650 0    40   BiDi ~ 0
+Text GLabel 8250 2000 0    40   BiDi ~ 0
 LCD_D06
-Text GLabel 9150 1650 2    40   BiDi ~ 0
+Text GLabel 9050 2000 2    40   BiDi ~ 0
 LCD_D07
-Text GLabel 8350 1750 0    40   BiDi ~ 0
+Text GLabel 8250 2100 0    40   BiDi ~ 0
 LCD_CS
-Text GLabel 8350 2150 0    40   BiDi ~ 0
+Text GLabel 8250 2500 0    40   BiDi ~ 0
 GPMI_ALE-LCD_D17
 Text GLabel 7300 5300 0    40   BiDi ~ 0
 SSP1_SCK-JTAG_TRST
-Text GLabel 9150 1750 2    40   BiDi ~ 0
+Text GLabel 9050 2100 2    40   BiDi ~ 0
 LCD_ENABLE-I2C_SCL
-Text GLabel 9150 2250 2    40   BiDi ~ 0
+Text GLabel 9050 2600 2    40   BiDi ~ 0
 GPMI_RDY1-SSP2_CMD
-Text GLabel 9150 3400 2    40   BiDi ~ 0
+Text GLabel 9050 3100 2    40   BiDi ~ 0
 GPMI_RDn
-Text GLabel 8350 3400 0    40   BiDi ~ 0
+Text GLabel 9050 3300 2    40   BiDi ~ 0
 GPMI_CE1n
-Text GLabel 8350 1850 0    40   BiDi ~ 0
+Text GLabel 8250 2200 0    40   BiDi ~ 0
 LCD_RESET-GPMI_CE3n
-Text GLabel 8350 2250 0    40   BiDi ~ 0
+Text GLabel 8250 2600 0    40   BiDi ~ 0
 GPMI_D00-LCD_D8-SSP2_DATA0
-Text GLabel 8350 3500 0    40   BiDi ~ 0
+Text GLabel 8250 3100 0    40   BiDi ~ 0
 GPMI_RDY0-SSP2_DETECT
-Text GLabel 9150 3300 2    40   BiDi ~ 0
+Text GLabel 8250 3300 0    40   BiDi ~ 0
 GPMI_CE0n
-Text GLabel 9150 1850 2    40   BiDi ~ 0
+Text GLabel 9050 2200 2    40   BiDi ~ 0
 LCD_WR
-Text GLabel 9150 2350 2    40   BiDi ~ 0
+Text GLabel 9050 2700 2    40   BiDi ~ 0
 GPMI_D01-LCD_D9-SSP2_DATA1
-Text GLabel 9150 3500 2    40   BiDi ~ 0
+Text GLabel 9050 3200 2    40   BiDi ~ 0
 GPMI_WRn-SSP2_SCK
 Text GLabel 7300 5800 0    40   BiDi ~ 0
 SSP1_CMD-JTAG_TDO
-Text GLabel 9150 1950 2    40   BiDi ~ 0
+Text GLabel 9050 2300 2    40   BiDi ~ 0
 LCD_RS
-Text GLabel 8350 2350 0    40   BiDi ~ 0
+Text GLabel 8250 2700 0    40   BiDi ~ 0
 GPMI_D02-LCD_D10-SSP2_DATA2
-Text GLabel 8350 3600 0    40   BiDi ~ 0
+Text GLabel 8250 3200 0    40   BiDi ~ 0
 GPMI_WPn
 Text GLabel 7300 5400 0    40   BiDi ~ 0
 SSP1_DATA0-JTAG_TDI
-Text GLabel 8350 1950 0    40   BiDi ~ 0
+Text GLabel 8250 2300 0    40   BiDi ~ 0
 LCD_HSYNC-I2C_SDA
-Text GLabel 9150 2450 2    40   BiDi ~ 0
+Text GLabel 9050 2800 2    40   BiDi ~ 0
 GPMI_D03-LCD_D11-SSP2_DATA3
-Text GLabel 9150 2050 2    40   BiDi ~ 0
+Text GLabel 9050 2400 2    40   BiDi ~ 0
 LCD_VSYNC-LCD_BUSY
-Text GLabel 9150 2550 2    40   BiDi ~ 0
+Text GLabel 9050 2900 2    40   BiDi ~ 0
 GPMI_D05-LCD_D13-SSP2_DATA5
 Text GLabel 7300 5700 0    40   BiDi ~ 0
 SSP1_DATA2-I2C_SDA-JTAG_RTCK
-Text GLabel 8350 2050 0    40   BiDi ~ 0
+Text GLabel 8250 2400 0    40   BiDi ~ 0
 LCD_DOTCK-GPMI_RDY3
-Text GLabel 8350 2450 0    40   BiDi ~ 0
+Text GLabel 8250 2800 0    40   BiDi ~ 0
 GPMI_D04-LCD_D12-SSP2_DATA4
 Text GLabel 7300 5500 0    40   BiDi ~ 0
 SSP1_DATA3-JTAG_TMS
-Text GLabel 9150 2650 2    40   BiDi ~ 0
+Text GLabel 9050 3000 2    40   BiDi ~ 0
 GPMI_D07-LCD_D15-SSP2_DATA7
-Text GLabel 9150 2150 2    40   BiDi ~ 0
+Text GLabel 9050 2500 2    40   BiDi ~ 0
 GPMI_CLE-LCD_D16
-Text GLabel 8350 2550 0    40   BiDi ~ 0
+Text GLabel 8250 2900 0    40   BiDi ~ 0
 GPMI_D06-LCD_D14-SSP2_DATA6
-Text GLabel 8350 1150 0    40   BiDi ~ 0
+Text GLabel 8250 1500 0    40   BiDi ~ 0
 PWM0-ROTARYA-DUART_RX
-Text GLabel 9150 1150 2    40   BiDi ~ 0
+Text GLabel 9050 1500 2    40   BiDi ~ 0
 PWM1-ROTARYB-DUART_TX
-Text GLabel 8350 1250 0    40   BiDi ~ 0
+Text GLabel 8250 1600 0    40   BiDi ~ 0
 I2C_SCL-GPMI_RDY2-AUART1_TX
-Text GLabel 9150 1250 2    40   BiDi ~ 0
+Text GLabel 9050 1600 2    40   BiDi ~ 0
 I2C_SDA-GPMI_CE2n-AUART1_RX
 $Comp
@@
 	1    0    0    -1
 $EndComp
-Text GLabel 9150 3600 2    40   BiDi ~ 0
-TSC_IN2
-Text GLabel 9150 3700 2    40   BiDi ~ 0
-TSC_VBAT2
-Text GLabel 8350 3700 0    40   BiDi ~ 0
-TSC_VREF
 $EndSCHEMATC
