File: PRopendous/Hardware/PROpendous/PROpendous-Connectors_JTAG.sch (KiCad schematic (older format))
At the start: 18 parts, among them IC5 FSUSB20, P1 Serial-JTAG, P2 Expansion, U2 microSD, U3 SD, U4 ARM_JTAG, U5 USB-miniB, U6 USB-A

Commit message: Updated PROpendous design with correct FSUSB20 footprint.  Added pictures of minimally assembled board and related testing.
Parts:
- added C82: 1uF, symbol C_MINI
Other:
- note added: "SSP1_DETECT-GPMI_CE3N-USB_ID is also used\nto enable LCD backlight so be careful with conflicts"
- moved on the sheet: C31, C32

Commit message: Updated the design.  JTAG header now includes VDD_XTAL and SSP1_Detect.  1.8" LCD has been removed and LCD backlight control is now connected to GPMI_CE1n.  The clock signals for the DDR SDRAM are now the longest EMI traces at 0.76".
Parts:
- added C83: 0.1uF, symbol C_MINI
- added R53: 0, symbol R_MINI
Connections:
- net labels added: FSUSB20_S, VDD_XTAL
- wire segments 73 -> 77
- no-connect marks 5 -> 3
Other:
- note added: "Debug/Expansion Headers"
- note added: "JTAG nSRST, DBGRQ, and DBGACK pins are\nconnected to non-JTAG pins so that the JTAG\nheader can be used as an expansion header.\nThey must be disconnected when using JTAG.\nBend the pins down when JTAG debugging.\n"
- note added: "LCD Backlight Enable"
- note added: "USB requires 90 Ohm differential impedance which for a\nstandard 1/16" 1oz FR4 double-sided board has been\ncalculated to require 22mil traces at 7mil spacing. Make\nsure to have a solid ground trace underneath the USB lines\nand keep 12mil spacing on either side of the traces to GND."
- note added: "When FSUSB20_S (PWM2-GPMI_RDY3) enables\nthe USB-A connector it will also enable the\nUSB Host VBUS Generator in the Power_Boot sheet"
- note removed: "Debug"
- note removed: "SSP1_DETECT-GPMI_CE3N-USB_ID is also used\nto enable LCD backlight so be careful with conflicts"
- note removed: "USB requires 90 Ohm differential impedance which for a\nstandard 1/16" 1oz FR4 double-sided board has been\ncalculated to require 22mil traces at 7mil spacing. Make\nsure to have a solid ground plane underneath the USB lines\nand keep 12mil spacing on either side of the traces to GND."
- note removed: "When PWM2-GPMI_RDY3 enables the\nUSB Host VBUS Generator it will also\nswitch the active USB connector to USB-A"
- moved on the sheet: C75, C77, IC5, L18, P1, R23, R5, U10, U6
