File: PRopendous/Hardware/PROpendous/PROpendous-Connectors_JTAG.sch (KiCad schematic (older format))
At the start: 21 parts, among them IC5 FSUSB20, P1 Serial-JTAG, P2 Expansion, U2 microSD, U3 SD, U4 ARM_JTAG, U5 USB-miniB, U6 USB-A

Commit message: Updated PROpendous design with minor correction to silkscreen and two more bypass capacitors for the microSD connector.  Also added Buttons Module design files.
Parts:
- added C84, C85: 0.1uF, symbol C_MINI
Other:
- moved on the sheet: C31, C32, C33, C34, C82
Changed lines of the file:
@@
-EESchema Schematic File Version 2  date 13/10/2010 11:22:35
+EESchema Schematic File Version 2  date 20/10/2010 05:47:04
 LIBS:opendous
 LIBS:device
@@
 Sheet 4 8
 Title "PROpendous"
-Date "28 sep 2010"
+Date "20 oct 2010"
 Rev "1.0"
 Comp "Opendous Inc. (www.opendous.org)"
@@
 Comment4 "www.PROpendous.org"
 $EndDescr
-$Comp
-L VDD_XTAL #PWR033
-U 1 1 4CA16B7B
-P 8600 5450
-F 0 "#PWR033" H 8600 5550 30  0001 C CNN
-F 1 "VDD_XTAL" H 8600 5550 30  0000 C CNN
-	1    8600 5450
-	1    0    0    -1
-$EndComp
-$Comp
-L C_MINI C83
-U 1 1 4CA16B77
-P 8600 5600
-F 0 "C83" V 8550 5650 30  0000 C CNN
-F 1 "0.1uF" V 8650 5670 25  0000 C CNN
-	1    8600 5600
-	0    1    1    0
-$EndComp
-$Comp
-L GND #PWR034
-U 1 1 4CA16B76
-P 8600 5750
-F 0 "#PWR034" H 8600 5750 30  0001 C CNN
-F 1 "GND" H 8600 5680 30  0001 C CNN
-	1    8600 5750
-	1    0    0    -1
-$EndComp
+Wire Wire Line
+	4750 3450 4750 3550
+Connection ~ 4750 3250
+Wire Wire Line
+	4550 3250 4950 3250
 Wire Wire Line
 	8600 5500 8600 5450
@@
 Connection ~ 8300 5700
 Wire Wire Line
-	8300 4900 8300 5900
+	8300 5900 8300 4900
 Wire Wire Line
 	1950 5600 1950 5550
@@
 Wire Wire Line
 	9800 5400 9800 5500
-Connection ~ 4750 3250
-Wire Wire Line
-	4750 3150 4750 3250
-Wire Wire Line
-	4850 3450 4650 3450
-Wire Wire Line
-	4650 3250 4850 3250
-Connection ~ 4750 3450
-Wire Wire Line
-	4750 3550 4750 3450
+Wire Wire Line
+	4750 3250 4750 3150
 Wire Wire Line
 	2850 2200 2950 2200
@@
 Wire Wire Line
 	5200 1850 5200 2000
-Wire Wire Line
-	2800 2950 2400 2950
+Connection ~ 2700 2950
+Connection ~ 2700 3150
+Wire Wire Line
+	2600 2950 2600 2850
+Wire Wire Line
+	4300 5650 4100 5650
+Connection ~ 4200 5650
+Wire Wire Line
+	2900 2950 2300 2950
+Connection ~ 2500 2950
+Wire Wire Line
+	2900 3150 2300 3150
+Connection ~ 2500 3150
+Connection ~ 2600 3150
 Connection ~ 2600 2950
 Wire Wire Line
-	2800 3150 2400 3150
-Connection ~ 2600 3150
-Wire Wire Line
-	2600 2950 2600 2850
-Wire Wire Line
-	4100 5650 4300 5650
-Connection ~ 4200 5650
+	4950 3450 4550 3450
+Connection ~ 4750 3450
+$Comp
+L C_MINI C85
+U 1 1 4CBEBA49
+P 4550 3350
+F 0 "C85" V 4500 3400 30  0000 C CNN
+F 1 "0.1uF" V 4600 3420 25  0000 C CNN
+	1    4550 3350
+	0    1    1    0
+$EndComp
+$Comp
+L C_MINI C84
+U 1 1 4CBEB7E3
+P 2300 3050
+F 0 "C84" V 2250 3100 30  0000 C CNN
+F 1 "0.1uF" V 2350 3120 25  0000 C CNN
+	1    2300 3050
+	0    1    1    0
+$EndComp
+$Comp
+L VDD_XTAL #PWR033
+U 1 1 4CA16B7B
+P 8600 5450
+F 0 "#PWR033" H 8600 5550 30  0001 C CNN
+F 1 "VDD_XTAL" H 8600 5550 30  0000 C CNN
+	1    8600 5450
+	1    0    0    -1
+$EndComp
+$Comp
+L C_MINI C83
+U 1 1 4CA16B77
+P 8600 5600
+F 0 "C83" V 8550 5650 30  0000 C CNN
+F 1 "0.1uF" V 8650 5670 25  0000 C CNN
+	1    8600 5600
+	0    1    1    0
+$EndComp
+$Comp
+L GND #PWR034
+U 1 1 4CA16B76
+P 8600 5750
+F 0 "#PWR034" H 8600 5750 30  0001 C CNN
+F 1 "GND" H 8600 5680 30  0001 C CNN
+	1    8600 5750
+	1    0    0    -1
+$EndComp
 $Comp
 L VDD_XTAL #PWR035
@@
 L C_MINI C82
 U 1 1 4C00A63F
-P 2800 3050
-F 0 "C82" V 2750 3100 30  0000 C CNN
-F 1 "1uF" V 2850 3100 25  0000 C CNN
-	1    2800 3050
+P 2900 3050
+F 0 "C82" V 2850 3100 30  0000 C CNN
+F 1 "1uF" V 2950 3100 25  0000 C CNN
+	1    2900 3050
 	0    1    1    0
 $EndComp
@@
 L C_MINI C33
 U 1 1 4BCA210D
-P 4650 3350
-F 0 "C33" V 4600 3400 30  0000 C CNN
-F 1 "0.1uF" V 4700 3420 25  0000 C CNN
-	1    4650 3350
+P 4750 3350
+F 0 "C33" V 4700 3400 30  0000 C CNN
+F 1 "0.1uF" V 4800 3420 25  0000 C CNN
+	1    4750 3350
 	0    1    1    0
 $EndComp
@@
 L C_MINI C34
 U 1 1 4BCA210B
-P 4850 3350
-F 0 "C34" V 4800 3400 30  0000 C CNN
-F 1 "1uF" V 4900 3400 25  0000 C CNN
-	1    4850 3350
+P 4950 3350
+F 0 "C34" V 4900 3400 30  0000 C CNN
+F 1 "1uF" V 5000 3400 25  0000 C CNN
+	1    4950 3350
 	0    1    1    0
 $EndComp
@@
 L C_MINI C32
 U 1 1 4BCA20E6
-P 2600 3050
-F 0 "C32" V 2550 3100 30  0000 C CNN
-F 1 "1uF" V 2650 3100 25  0000 C CNN
-	1    2600 3050
+P 2700 3050
+F 0 "C32" V 2650 3100 30  0000 C CNN
+F 1 "1uF" V 2750 3100 25  0000 C CNN
+	1    2700 3050
 	0    1    1    0
 $EndComp
@@
 L C_MINI C31
 U 1 1 4BCA20D5
-P 2400 3050
-F 0 "C31" V 2350 3100 30  0000 C CNN
-F 1 "0.1uF" V 2450 3120 25  0000 C CNN
-	1    2400 3050
-	0    1    1    0
-$EndComp
+P 2500 3050
+F 0 "C31" V 2450 3100 30  0000 C CNN
+F 1 "0.1uF" V 2550 3120 25  0000 C CNN
+	1    2500 3050
+	0    1    1    0
+$EndComp

Commit message: Updated PROpendous design.  PWM2-GPMI_RDY3 now controls the LCD backlight and GPMI_CE1n now controls USB Host enable.  The function of these pins was switched as PWM2 makes more sense as a backlight control.
Connections:
- net labels removed: PWM2-GPMI_RDY3
Other:
- note added: "Depopulating R53 will allow you\nto use the Host/Debug LED in the\nPower_Boot sheet without also\nenabling USB Hosting"
- note added: "USB Connector Switch Control"
- note added: "When FSUSB20_S (GPMI_CE1n) enables\nthe USB-A connector it will also enable the\nUSB Host VBUS Generator and turn on the\nUSB_HOST LED in the Power_Boot sheet"
- note removed: "LCD Backlight Enable"
- note removed: "When FSUSB20_S (PWM2-GPMI_RDY3) enables\nthe USB-A connector it will also enable the\nUSB Host VBUS Generator in the Power_Boot sheet"
- moved on the sheet: R22, R53
Changed lines of the file:
@@
-EESchema Schematic File Version 2  date 20/10/2010 05:47:04
+EESchema Schematic File Version 2  date 21/10/2010 09:30:50
 LIBS:opendous
 LIBS:device
@@
 Sheet 4 8
 Title "PROpendous"
-Date "20 oct 2010"
-Rev "1.0"
+Date "21 oct 2010"
+Rev "1.1"
 Comp "Opendous Inc. (www.opendous.org)"
 Comment1 ""
@@
 Comment4 "www.PROpendous.org"
 $EndDescr
-Wire Wire Line
-	4750 3450 4750 3550
-Connection ~ 4750 3250
-Wire Wire Line
-	4550 3250 4950 3250
-Wire Wire Line
-	8600 5500 8600 5450
-Wire Wire Line
-	8600 5700 8600 5750
-Wire Wire Line
-	7200 5600 7300 5600
-Wire Wire Line
-	2600 3250 2600 3150
-Connection ~ 5200 1950
-Wire Wire Line
-	5100 1950 5200 1950
-Wire Wire Line
-	8600 5100 8600 5150
-Wire Wire Line
-	8600 4900 8600 4850
-Wire Wire Line
-	7300 4800 7300 4600
-Connection ~ 8300 5000
-Connection ~ 8300 5100
-Connection ~ 8300 5200
-Connection ~ 8300 5300
-Connection ~ 8300 5400
-Connection ~ 8300 5500
-Connection ~ 8300 5600
-Connection ~ 8300 5700
-Wire Wire Line
-	8300 5900 8300 4900
-Wire Wire Line
-	1950 5600 1950 5550
-Wire Wire Line
-	1950 5550 1900 5550
-Wire Wire Line
-	5300 1800 5300 1750
-Wire Wire Line
-	5300 1750 5100 1750
-Wire Wire Line
-	2800 6850 2800 6800
-Wire Wire Line
-	1725 6475 1725 6450
-Wire Wire Line
-	1725 6450 1600 6450
-Wire Wire Line
-	3250 5750 3700 5750
-Wire Wire Line
-	2350 6050 2150 6050
-Wire Wire Line
-	2150 6050 2150 6150
-Wire Wire Line
-	2150 6150 1600 6150
-Wire Wire Line
-	2350 5750 2050 5750
-Wire Wire Line
-	2050 5750 2050 5350
-Wire Wire Line
-	2050 5350 1600 5350
-Wire Wire Line
-	1950 6250 1600 6250
-Wire Wire Line
-	1700 5675 1700 5650
-Wire Wire Line
-	1700 5650 1600 5650
-Wire Wire Line
-	2250 2100 1200 2100
-Wire Wire Line
-	9800 5000 9800 5100
-Wire Wire Line
-	9800 5100 9900 5100
-Wire Wire Line
-	10200 5300 9750 5300
-Wire Wire Line
-	10200 5200 9750 5200
-Wire Wire Line
-	10200 5100 10100 5100
-Wire Wire Line
-	10200 5400 9800 5400
-Wire Wire Line
-	9800 5400 9800 5500
-Wire Wire Line
-	4750 3250 4750 3150
-Wire Wire Line
-	2850 2200 2950 2200
-Wire Wire Line
-	2950 2200 2950 2300
-Wire Wire Line
-	1200 2100 1200 2150
-Wire Wire Line
-	2250 2000 1200 2000
-Wire Wire Line
-	1200 2000 1200 1950
-Wire Wire Line
-	3350 2350 3350 2400
-Wire Wire Line
-	3350 2400 4400 2400
-Wire Wire Line
-	3350 2550 3350 2500
-Wire Wire Line
-	3350 2500 4400 2500
-Wire Wire Line
-	2800 6300 2800 6200
-Wire Wire Line
-	2800 5500 2800 5300
-Wire Wire Line
-	3700 6050 3700 5950
-Wire Wire Line
-	1650 5450 1600 5450
-Wire Wire Line
-	4200 6050 4200 5850
-Wire Wire Line
-	1600 5250 2150 5250
-Wire Wire Line
-	2150 5250 2150 5650
-Wire Wire Line
-	2150 5650 2350 5650
-Wire Wire Line
-	1600 6050 2050 6050
-Wire Wire Line
-	2050 6050 2050 5950
-Wire Wire Line
-	2050 5950 2350 5950
-Wire Wire Line
-	3250 5650 3900 5650
-Wire Wire Line
-	1600 6350 1950 6350
-Wire Wire Line
-	1950 6350 1950 6375
-Wire Wire Line
-	2800 7050 2800 7100
-Wire Wire Line
-	1700 5550 1600 5550
+Text Notes 4300 6150 0    40   ~ 0
+Depopulating R53 will allow you\nto use the Host/Debug LED in the\nPower_Boot sheet without also\nenabling USB Hosting
+Wire Wire Line
+	4200 5650 4300 5650
+Connection ~ 3900 5650
+Wire Wire Line
+	4000 5650 3250 5650
+Connection ~ 4750 3450
+Wire Wire Line
+	4550 3450 4950 3450
+Connection ~ 2600 2950
+Connection ~ 2600 3150
+Connection ~ 2500 3150
+Wire Wire Line
+	2300 3150 2900 3150
+Connection ~ 2500 2950
+Wire Wire Line
+	2300 2950 2900 2950
+Wire Wire Line
+	2600 2950 2600 2850
+Connection ~ 2700 3150
+Connection ~ 2700 2950
+Wire Wire Line
+	5200 2000 5200 1850
+Wire Wire Line
+	5200 1850 5100 1850
+Connection ~ 7800 4600
+Wire Wire Line
+	7800 4550 7800 4600
+Wire Wire Line
+	8300 4800 8300 4600
+Wire Wire Line
+	8300 4600 7300 4600
+Wire Wire Line
+	9200 1350 9200 1400
+Wire Wire Line
+	9200 1400 9050 1400
+Wire Wire Line
+	8250 1400 8250 1300
+Wire Wire Line
+	8250 1300 8100 1300
+Wire Wire Line
+	8100 1300 8100 1350
+Wire Notes Line
+	11200 1200 11200 500
+Wire Notes Line
+	11200 1200 10600 1200
+Wire Notes Line
+	10600 1200 10600 500
 Wire Notes Line
 	10600 500  11200 500
-Wire Notes Line
-	10600 500  10600 1200
-Wire Notes Line
-	10600 1200 11200 1200
-Wire Notes Line
-	11200 1200 11200 500
-Wire Wire Line
-	8100 1350 8100 1300
-Wire Wire Line
-	8100 1300 8250 1300
-Wire Wire Line
-	8250 1300 8250 1400
-Wire Wire Line
-	9050 1400 9200 1400
-Wire Wire Line
-	9200 1400 9200 1350
-Wire Wire Line
-	7300 4600 8300 4600
-Wire Wire Line
-	8300 4600 8300 4800
-Wire Wire Line
-	7800 4550 7800 4600
-Connection ~ 7800 4600
-Wire Wire Line
-	5100 1850 5200 1850
-Wire Wire Line
-	5200 1850 5200 2000
-Connection ~ 2700 2950
-Connection ~ 2700 3150
-Wire Wire Line
-	2600 2950 2600 2850
-Wire Wire Line
-	4300 5650 4100 5650
-Connection ~ 4200 5650
-Wire Wire Line
-	2900 2950 2300 2950
-Connection ~ 2500 2950
-Wire Wire Line
-	2900 3150 2300 3150
-Connection ~ 2500 3150
-Connection ~ 2600 3150
-Connection ~ 2600 2950
-Wire Wire Line
-	4950 3450 4550 3450
-Connection ~ 4750 3450
+Wire Wire Line
+	1700 5550 1600 5550
+Wire Wire Line
+	2800 7050 2800 7100
+Wire Wire Line
+	1950 6375 1950 6350
+Wire Wire Line
+	1950 6350 1600 6350
+Wire Wire Line
+	2350 5950 2050 5950
+Wire Wire Line
+	2050 5950 2050 6050
+Wire Wire Line
+	2050 6050 1600 6050
+Wire Wire Line
+	2350 5650 2150 5650
+Wire Wire Line
+	2150 5650 2150 5250
+Wire Wire Line
+	2150 5250 1600 5250
+Wire Wire Line
+	3900 6050 3900 5850
+Wire Wire Line
+	1650 5450 1600 5450
+Wire Wire Line
+	3700 6050 3700 5950
+Wire Wire Line
+	2800 5500 2800 5300
+Wire Wire Line
+	2800 6300 2800 6200
+Wire Wire Line
+	4400 2500 3350 2500
+Wire Wire Line
+	3350 2500 3350 2550
+Wire Wire Line
+	4400 2400 3350 2400
+Wire Wire Line
+	3350 2400 3350 2350
+Wire Wire Line
+	1200 1950 1200 2000
+Wire Wire Line
+	1200 2000 2250 2000
+Wire Wire Line
+	1200 2150 1200 2100
+Wire Wire Line
+	2950 2300 2950 2200
+Wire Wire Line
+	2950 2200 2850 2200
+Wire Wire Line
+	4750 3150 4750 3250
+Wire Wire Line
+	9800 5500 9800 5400
+Wire Wire Line
+	9800 5400 10200 5400
+Wire Wire Line
+	10200 5100 10100 5100
+Wire Wire Line
+	10200 5200 9750 5200
+Wire Wire Line
+	10200 5300 9750 5300
+Wire Wire Line
+	9900 5100 9800 5100
+Wire Wire Line
+	9800 5100 9800 5000
+Wire Wire Line
+	1200 2100 2250 2100
+Wire Wire Line
+	1600 5650 1700 5650
+Wire Wire Line
+	1700 5650 1700 5675
+Wire Wire Line
+	1950 6250 1600 6250
+Wire Wire Line
+	1600 5350 2050 5350
+Wire Wire Line
+	2050 5350 2050 5750
+Wire Wire Line
+	2050 5750 2350 5750
+Wire Wire Line
+	1600 6150 2150 6150
+Wire Wire Line
+	2150 6150 2150 6050
+Wire Wire Line
+	2150 6050 2350 6050
+Wire Wire Line
+	3250 5750 3700 5750
+Wire Wire Line
+	1600 6450 1725 6450
+Wire Wire Line
+	1725 6450 1725 6475
+Wire Wire Line
+	2800 6850 2800 6800
+Wire Wire Line
+	5100 1750 5300 1750
+Wire Wire Line
+	5300 1750 5300 1800
+Wire Wire Line
+	1900 5550 1950 5550
+Wire Wire Line
+	1950 5550 1950 5600
+Wire Wire Line
+	8300 4900 8300 5900
+Connection ~ 8300 5700
+Connection ~ 8300 5600
+Connection ~ 8300 5500
+Connection ~ 8300 5400
+Connection ~ 8300 5300
+Connection ~ 8300 5200
+Connection ~ 8300 5100
+Connection ~ 8300 5000
+Wire Wire Line
+	7300 4600 7300 4800
+Wire Wire Line
+	8600 4900 8600 4850
+Wire Wire Line
+	8600 5100 8600 5150
+Wire Wire Line
+	5100 1950 5200 1950
+Connection ~ 5200 1950
+Wire Wire Line
+	2600 3250 2600 3150
+Wire Wire Line
+	7200 5600 7300 5600
+Wire Wire Line
+	8600 5700 8600 5750
+Wire Wire Line
+	8600 5500 8600 5450
+Wire Wire Line
+	4950 3250 4550 3250
+Connection ~ 4750 3250
+Wire Wire Line
+	4750 3450 4750 3550
 $Comp
 L C_MINI C85
@@
 L R_MINI R53
 U 1 1 4CA14980
-P 4000 5650
-F 0 "R53" H 3950 5700 25  0000 C CNN
-F 1 "0" H 4050 5700 20  0000 C CNN
-	1    4000 5650
+P 4100 5650
+F 0 "R53" H 4050 5700 25  0000 C CNN
+F 1 "0" H 4150 5700 20  0000 C CNN
+	1    4100 5650
 	1    0    0    -1
 $EndComp
 Text Notes 9475 3325 0    30   ~ 0
-LCD Backlight Enable
+USB Connector Switch Control
 Text Notes 7200 6100 0    40   ~ 0
 JTAG nSRST, DBGRQ, and DBGACK pins are\nconnected to non-JTAG pins so that the JTAG\nheader can be used as an expansion header.\nThey must be disconnected when using JTAG.\nBend the pins down when JTAG debugging.\n
@@
 Text Notes 8100 1100 0    80   Italic 16
 Expansion Header
-Text Notes 4350 5850 0    40   ~ 0
-When FSUSB20_S (PWM2-GPMI_RDY3) enables\nthe USB-A connector it will also enable the\nUSB Host VBUS Generator in the Power_Boot sheet
+Text Notes 4300 5850 0    40   ~ 0
+When FSUSB20_S (GPMI_CE1n) enables\nthe USB-A connector it will also enable the\nUSB Host VBUS Generator and turn on the\nUSB_HOST LED in the Power_Boot sheet
 $Comp
 L GND #PWR048
 U 1 1 4BCC707A
-P 4200 6050
-F 0 "#PWR048" H 4200 6050 30  0001 C CNN
-F 1 "GND" H 4200 5980 30  0001 C CNN
-	1    4200 6050
+P 3900 6050
+F 0 "#PWR048" H 3900 6050 30  0001 C CNN
+F 1 "GND" H 3900 5980 30  0001 C CNN
+	1    3900 6050
 	1    0    0    -1
 $EndComp
@@
 L R_MINI R22
 U 1 1 4BCC59F1
-P 4200 5750
-F 0 "R22" V 4175 5800 25  0000 C CNN
-F 1 "15k" V 4225 5800 20  0000 C CNN
-	1    4200 5750
+P 3900 5750
+F 0 "R22" V 3875 5800 25  0000 C CNN
+F 1 "15k" V 3925 5800 20  0000 C CNN
+	1    3900 5750
 	0    1    1    0
 $EndComp
@@
 GPMI_RDY1-SSP2_CMD
 Text GLabel 4300 5650 2    40   BiDi ~ 0
-PWM2-GPMI_RDY3
+GPMI_CE1n
 Text GLabel 2250 1750 0    40   BiDi ~ 0
 GPMI_D00-LCD_D8-SSP2_DATA0

Commit message: Minor update of Connectors_JTAG sheet with note about updated microSD connector part number.
Other:
- note added: "101-00303-68"
- note added: "Amphenol"
- note removed: "3M 29-08-05"
Changed lines of the file:
@@
-EESchema Schematic File Version 2  date 21/10/2010 09:30:50
+EESchema Schematic File Version 2  date 21/10/2010 18:49:25
 LIBS:opendous
 LIBS:device
@@
 Comment4 "www.PROpendous.org"
 $EndDescr
+Text Notes 2350 2600 0    40   ~ 0
+101-00303-68
 Text Notes 4300 6150 0    40   ~ 0
 Depopulating R53 will allow you\nto use the Host/Debug LED in the\nPower_Boot sheet without also\nenabling USB Hosting
@@
 	0    1    1    0
 $EndComp
-Text Notes 2350 2550 0    40   ~ 0
-3M 29-08-05
+Text Notes 2450 2550 0    40   ~ 0
+Amphenol
 Text Notes 4450 2850 0    40   ~ 0
 3M SD-RSMT-2
