File: PRopendous/Hardware/PROpendous/PROpendous-Memory.sch (KiCad schematic (older format))
At the start: 2 parts, among them IC17 AT45DBxx1D-SU

Commit message: Updated files.  DDR SDRAM schematic completed.
Parts:
- removed IC17: AT45DBxx1D-SU, symbol AT45DBXX1
- removed R34: 10k, symbol R_MINI
- added C10, C11, C12, C13, C16, C17, C6, C7, C8, C9: 0.1uF, symbol C_MINI
- added C14, C15: 10uF, symbol C_MINI
- added IC2: DDR_SDRAM_MT46_X16, symbol DDR_SDRAM_MT46_X16
- added R4, R7: 47k, symbol R_MINI
- added R8, R9: 1k, symbol R_MINI
Connections:
- net labels added: VDDM_2V5
- net labels removed: VSUP3
- wire segments 12 -> 19
- no-connect marks 0 -> 7
Other:
- note added: "1%"
- note added: "64Mbytes DDR SDRAM"
- note added: "Notes:\n - All capacitors are X5R, 6.3V, 20%, ESR < 300mOhm or better unless otherwise noted\n - All resistors are 5% unless otherwise noted\n - Assuming 2-layer standard 1/16" FR4 (Dk=4.4, Df=0.02) and 8mil-8mil-20mil trace-space-via design\n - Per Micron TN-46-02, Lvia=1.12nH, Leq=0.87+1.12=2nH so NcapMVTT=69, NcapV25=28"
- note removed: "SPI Boot Flash"

Commit message: Updated PROpendous i.MX233 project.  DDR SDRAM layout is complete.
Parts:
- added C16, C17, C20, C21: 10uF, symbol C_MINI
- added C22, C23, C24, C25: 10nF, symbol C_MINI
- added C26, C27: 68uF, symbol CP_TANTALUM_MINI
- added R10: 100, symbol R_MINI
- renumbered C16 to C18, C17 to C19
Connections:
- net labels added: DDR_VREF
- wire segments 19 -> 22
Other:
- note added: "Must be kept +/- 50mV at\nnearest bypass capacitor"
- note added: "Notes:\n - All capacitors are X5R, 6.3V, 20%, ESR < 300mOhm or better unless otherwise noted\n - All resistors are 5% unless otherwise noted\n - Assuming 2-layer standard 1/16" FR4 (Dk=4.4, Df=0.02) and 7mil-7mil-15mil trace-space-via design\n - Per Micron TN-46-02, need about 7 0.1uF bypass caps but to meet TN-46-14 layout guidelines use a\n lot more and consider external copper foil reference p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"
- note added: "Rt"
- note removed: "Notes:\n - All capacitors are X5R, 6.3V, 20%, ESR < 300mOhm or better unless otherwise noted\n - All resistors are 5% unless otherwise noted\n - Assuming 2-layer standard 1/16" FR4 (Dk=4.4, Df=0.02) and 8mil-8mil-20mil trace-space-via design\n - Per Micron TN-46-02, Lvia=1.12nH, Leq=0.87+1.12=2nH so NcapMVTT=69, NcapV25=28"
Changed lines of the file:
@@
-EESchema Schematic File Version 2  date 07/04/2010 20:14:10
+EESchema Schematic File Version 2  date 17/04/2010 17:25:37
 LIBS:opendous
 LIBS:device
@@
 EELAYER END
 $Descr A4 11700 8267
-Sheet 3 6
+Sheet 3 7
 Title "PROpendous"
-Date "8 apr 2010"
+Date "17 apr 2010"
 Rev "1.0"
 Comp "Opendous Inc. (www.opendous.org)"
@@
 Comment4 "www.PROpendous.org"
 $EndDescr
-Text Notes 2600 900  0    60   ~ 0
-64Mbytes DDR SDRAM
+Connection ~ 3050 5400
+Wire Wire Line
+	3050 5500 3050 5400
+Connection ~ 4550 5400
+Wire Wire Line
+	1350 5400 4750 5400
+Connection ~ 4350 5400
+Connection ~ 1950 5400
+Connection ~ 2150 5400
+Connection ~ 1750 5400
+Connection ~ 1750 5200
+Connection ~ 1550 5200
+Connection ~ 1550 5400
+Wire Wire Line
+	1100 3900 1000 3900
+Wire Wire Line
+	4400 4350 4400 4400
+Connection ~ 4600 4100
+Wire Wire Line
+	4600 4150 4600 4050
+Connection ~ 4400 4350
+Wire Wire Line
+	4200 4350 4600 4350
+Connection ~ 4400 3850
+Wire Wire Line
+	4200 3850 4600 3850
+Connection ~ 4150 5400
+Connection ~ 4150 5200
+Connection ~ 3950 5200
 Wire Wire Line
 	1700 3850 1700 3900
@@
 Wire Wire Line
 	1600 3650 2250 3650
-Connection ~ 3050 5200
-Wire Wire Line
-	3050 5200 3050 5100
 Connection ~ 2350 5400
-Wire Wire Line
-	3950 5400 2150 5400
 Connection ~ 2750 5400
 Connection ~ 3150 5400
@@
 Connection ~ 2750 5200
 Connection ~ 2350 5200
-Connection ~ 4300 4350
-Wire Wire Line
-	4300 4350 4300 4400
-Connection ~ 4300 3850
-Wire Wire Line
-	4300 3850 4300 3800
 Wire Wire Line
 	4200 4050 4200 4150
@@
 Connection ~ 3050 4600
 Connection ~ 2950 4600
-Wire Wire Line
-	3850 4100 4400 4100
 Connection ~ 4200 4100
-Wire Wire Line
-	4200 3850 4400 3850
-Wire Wire Line
-	4200 4350 4400 4350
 Connection ~ 2550 5200
 Connection ~ 2950 5200
 Connection ~ 3350 5200
-Wire Wire Line
-	2150 5200 3950 5200
 Connection ~ 3750 5200
 Connection ~ 3750 5400
@@
 Connection ~ 2550 5400
 Wire Wire Line
-	3050 5400 3050 5500
-Connection ~ 3050 5400
-Wire Wire Line
 	1700 3250 1700 3200
+Connection ~ 3950 5400
+Wire Wire Line
+	3850 4100 4600 4100
+Wire Wire Line
+	4400 3800 4400 3850
+Wire Wire Line
+	1000 3700 1100 3700
+Connection ~ 1950 5200
+Connection ~ 2150 5200
+Connection ~ 4350 5200
+Wire Wire Line
+	1350 5200 4750 5200
+Connection ~ 4550 5200
+Wire Wire Line
+	3050 5200 3050 5100
+Connection ~ 3050 5200
+$Comp
+L VDDM_2V5 #PWR019
+U 1 1 4BBCEBA8
+P 3050 5100
+F 0 "#PWR019" H 3050 5200 30  0001 C CNN
+F 1 "VDDM_2V5" H 3050 5200 30  0000 C CNN
+	1    3050 5100
+	1    0    0    -1
+$EndComp
+$Comp
+L CP_TANTALUM_MINI C27
+U 1 1 4BC981AE
+P 4750 5300
+F 0 "C27" V 4700 5350 30  0000 C CNN
+F 1 "68uF" V 4800 5350 25  0000 C CNN
+	1    4750 5300
+	0    1    1    0
+$EndComp
+$Comp
+L CP_TANTALUM_MINI C26
+U 1 1 4BC981A1
+P 4550 5300
+F 0 "C26" V 4500 5350 30  0000 C CNN
+F 1 "68uF" V 4600 5350 25  0000 C CNN
+	1    4550 5300
+	0    1    1    0
+$EndComp
+Text GLabel 6600 7700 2    40   BiDi ~ 0
+DDR_VREF
+Text Label 6600 7700 2    35   ~ 0
+DDR_VREF
+Text Label 3850 4100 0    35   ~ 0
+DDR_VREF
+$Comp
+L C_MINI C22
+U 1 1 4BC96D3F
+P 1350 5300
+F 0 "C22" V 1300 5350 30  0000 C CNN
+F 1 "10nF" V 1400 5370 25  0000 C CNN
+	1    1350 5300
+	0    1    1    0
+$EndComp
+$Comp
+L C_MINI C23
+U 1 1 4BC96D3E
+P 1550 5300
+F 0 "C23" V 1500 5350 30  0000 C CNN
+F 1 "10nF" V 1600 5370 25  0000 C CNN
+	1    1550 5300
+	0    1    1    0
+$EndComp
+$Comp
+L C_MINI C25
+U 1 1 4BC96D3D
+P 1950 5300
+F 0 "C25" V 1900 5350 30  0000 C CNN
+F 1 "10nF" V 2000 5370 25  0000 C CNN
+	1    1950 5300
+	0    1    1    0
+$EndComp
+$Comp
+L C_MINI C24
+U 1 1 4BC96D3C
+P 1750 5300
+F 0 "C24" V 1700 5350 30  0000 C CNN
+F 1 "10nF" V 1800 5370 25  0000 C CNN
+	1    1750 5300
+	0    1    1    0
+$EndComp
+Text Notes 950  3850 0    60   ~ 0
+Rt
+$Comp
+L R_MINI R10
+U 1 1 4BC96327
+P 1100 3800
+F 0 "R10" V 1075 3850 25  0000 C CNN
+F 1 "100" V 1125 3850 20  0000 C CNN
+	1    1100 3800
+	0    1    1    0
+$EndComp
+Text GLabel 1000 3900 0    40   BiDi ~ 0
+EMI_CLKn
+Text GLabel 1000 3700 0    40   BiDi ~ 0
+EMI_CLK
+Text Notes 4725 4125 0    40   ~ 0
+Must be kept +/- 50mV at\nnearest bypass capacitor
+$Comp
+L C_MINI C20
+U 1 1 4BC3A0BD
+P 4600 3950
+F 0 "C20" V 4550 4000 30  0000 C CNN
+F 1 "10uF" V 4650 4000 25  0000 C CNN
+	1    4600 3950
+	0    1    1    0
+$EndComp
+$Comp
+L C_MINI C21
+U 1 1 4BC3A0BC
+P 4600 4250
+F 0 "C21" V 4550 4300 30  0000 C CNN
+F 1 "10uF" V 4650 4300 25  0000 C CNN
+	1    4600 4250
+	0    1    1    0
+$EndComp
+$Comp
+L C_MINI C16
+U 1 1 4BC39B55
+P 4150 5300
+F 0 "C16" V 4100 5350 30  0000 C CNN
+F 1 "10uF" V 4200 5350 25  0000 C CNN
+	1    4150 5300
+	0    1    1    0
+$EndComp
+$Comp
+L C_MINI C17
+U 1 1 4BC39B54
+P 4350 5300
+F 0 "C17" V 4300 5350 30  0000 C CNN
+F 1 "10uF" V 4400 5350 25  0000 C CNN
+	1    4350 5300
+	0    1    1    0
+$EndComp
+Text Notes 2600 900  0    60   ~ 0
+64Mbytes DDR SDRAM
 $Comp
 L R_MINI R7
@@
 $EndComp
 $Comp
-L GND #PWR018
+L GND #PWR020
 U 1 1 4BBCED31
 P 1700 3900
-F 0 "#PWR018" H 1700 3900 30  0001 C CNN
+F 0 "#PWR020" H 1700 3900 30  0001 C CNN
 F 1 "GND" H 1700 3830 30  0001 C CNN
 	1    1700 3900
@@
 $EndComp
 $Comp
-L VDDM_2V5 #PWR019
+L VDDM_2V5 #PWR021
 U 1 1 4BBCED2D
 P 1700 3200
-F 0 "#PWR019" H 1700 3300 30  0001 C CNN
+F 0 "#PWR021" H 1700 3300 30  0001 C CNN
 F 1 "VDDM_2V5" H 1700 3300 30  0000 C CNN
 	1    1700 3200
@@
 $EndComp
 $Comp
-L VDDM_2V5 #PWR020
-U 1 1 4BBCEBA8
-P 3050 5100
-F 0 "#PWR020" H 3050 5200 30  0001 C CNN
-F 1 "VDDM_2V5" H 3050 5200 30  0000 C CNN
-	1    3050 5100
-	1    0    0    -1
-$EndComp
-$Comp
-L GND #PWR021
+L GND #PWR022
 U 1 1 4BBCEB9B
 P 3050 5500
-F 0 "#PWR021" H 3050 5500 30  0001 C CNN
+F 0 "#PWR022" H 3050 5500 30  0001 C CNN
 F 1 "GND" H 3050 5430 30  0001 C CNN
 	1    3050 5500
@@
 U 1 1 4BBCEB87
 P 3950 5300
-F 0 "C15" V 3900 5340 30  0000 C CNN
+F 0 "C15" V 3900 5350 30  0000 C CNN
 F 1 "10uF" V 4000 5350 25  0000 C CNN
 	1    3950 5300
@@
 U 1 1 4BBCEB79
 P 3750 5300
-F 0 "C14" V 3700 5340 30  0000 C CNN
+F 0 "C14" V 3700 5350 30  0000 C CNN
 F 1 "10uF" V 3800 5350 25  0000 C CNN
 	1    3750 5300
@@
 U 1 1 4BBCEB5B
 P 2950 5300
-F 0 "C10" V 2900 5340 30  0000 C CNN
+F 0 "C10" V 2900 5350 30  0000 C CNN
 F 1 "0.1uF" V 3000 5370 25  0000 C CNN
 	1    2950 5300
@@
 U 1 1 4BBCEB5A
 P 3150 5300
-F 0 "C11" V 3100 5340 30  0000 C CNN
+F 0 "C11" V 3100 5350 30  0000 C CNN
 F 1 "0.1uF" V 3200 5370 25  0000 C CNN
 	1    3150 5300
@@
 U 1 1 4BBCEB59
 P 3550 5300
-F 0 "C13" V 3500 5340 30  0000 C CNN
+F 0 "C13" V 3500 5350 30  0000 C CNN
 F 1 "0.1uF" V 3600 5370 25  0000 C CNN
 	1    3550 5300
@@
 U 1 1 4BBCEB58
 P 3350 5300
-F 0 "C12" V 3300 5340 30  0000 C CNN
+F 0 "C12" V 3300 5350 30  0000 C CNN
 F 1 "0.1uF" V 3400 5370 25  0000 C CNN
 	1    3350 5300
@@
 $EndComp
 $Comp
-L C_MINI C17
+L C_MINI C19
 U 1 1 4BBCEAA2
 P 4400 4250
-F 0 "C17" V 4350 4290 30  0000 C CNN
+F 0 "C19" V 4350 4300 30  0000 C CNN
 F 1 "0.1uF" V 4450 4320 25  0000 C CNN
 	1    4400 4250
@@
 $EndComp
 $Comp
-L C_MINI C16
+L C_MINI C18
 U 1 1 4BBCEA91
 P 4400 3950
-F 0 "C16" V 4350 3990 30  0000 C CNN
+F 0 "C18" V 4350 4000 30  0000 C CNN
 F 1 "0.1uF" V 4450 4020 25  0000 C CNN
 	1    4400 3950
@@
 $EndComp
 $Comp
-L VDDM_2V5 #PWR022
+L VDDM_2V5 #PWR023
 U 1 1 4BBCEA5E
-P 4300 3800
-F 0 "#PWR022" H 4300 3900 30  0001 C CNN
-F 1 "VDDM_2V5" H 4300 3900 30  0000 C CNN
-	1    4300 3800
-	1    0    0    -1
-$EndComp
-$Comp
-L GND #PWR023
+P 4400 3800
+F 0 "#PWR023" H 4400 3900 30  0001 C CNN
+F 1 "VDDM_2V5" H 4400 3900 30  0000 C CNN
+	1    4400 3800
+	1    0    0    -1
+$EndComp
+$Comp
+L GND #PWR024
 U 1 1 4BBCEA59
-P 4300 4400
-F 0 "#PWR023" H 4300 4400 30  0001 C CNN
-F 1 "GND" H 4300 4330 30  0001 C CNN
-	1    4300 4400
+P 4400 4400
+F 0 "#PWR024" H 4400 4400 30  0001 C CNN
+F 1 "GND" H 4400 4330 30  0001 C CNN
+	1    4400 4400
 	1    0    0    -1
 $EndComp
@@
 NoConn ~ 3850 3850
 $Comp
-L GND #PWR024
+L GND #PWR025
 U 1 1 4BBCEA0F
 P 3050 4700
-F 0 "#PWR024" H 3050 4700 30  0001 C CNN
+F 0 "#PWR025" H 3050 4700 30  0001 C CNN
 F 1 "GND" H 3050 4630 30  0001 C CNN
 	1    3050 4700
@@
 $EndComp
 $Comp
-L VDDM_2V5 #PWR025
+L VDDM_2V5 #PWR026
 U 1 1 4BBCE9DE
 P 3050 1200
-F 0 "#PWR025" H 3050 1300 30  0001 C CNN
+F 0 "#PWR026" H 3050 1300 30  0001 C CNN
 F 1 "VDDM_2V5" H 3050 1300 30  0000 C CNN
 	1    3050 1200
@@
 $EndComp
 Text Notes 1050 6850 0    60   ~ 0
-Notes:\n - All capacitors are X5R, 6.3V, 20%, ESR < 300mOhm or better unless otherwise noted\n - All resistors are 5% unless otherwise noted\n - Assuming 2-layer standard 1/16" FR4 (Dk=4.4, Df=0.02) and 8mil-8mil-20mil trace-space-via design\n - Per Micron TN-46-02, Lvia=1.12nH, Leq=0.87+1.12=2nH so NcapMVTT=69, NcapV25=28
+Notes:\n - All capacitors are X5R, 6.3V, 20%, ESR < 300mOhm or better unless otherwise noted\n - All resistors are 5% unless otherwise noted\n - Assuming 2-layer standard 1/16" FR4 (Dk=4.4, Df=0.02) and 7mil-7mil-15mil trace-space-via design\n - Per Micron TN-46-02, need about 7 0.1uF bypass caps but to meet TN-46-14 layout guidelines use a\n    lot more and consider external copper foil reference planes\n - Cannot meet DDR routing guidelines (TN-46-14) on 2-layers so just keep all signals as short as possible\n    to limit effects on Signal Integrity (SI) of incorrect inter/intra-pair spacing\n - Only using one DDR device so should not require Rt
 Text GLabel 8750 1650 2    40   BiDi ~ 0
 LCD_D00

Commit message: Updated PROpendous project.  Schematic is complete but not yet finalized.  Layout partially complete.
Connections:
- net labels removed: DEBUG, GPMI_ALE-LCD_D17, GPMI_CE0n, GPMI_CE1n, GPMI_CLE-LCD_D16, GPMI_D00-LCD_D8-SSP2_DATA0, GPMI_D01-LCD_D9-SSP2_DATA1, GPMI_D02-LCD_D10-SSP2_DATA2, GPMI_D03-LCD_D11-SSP2_DATA3, GPMI_D04-LCD_D12-SSP2_DATA4, GPMI_D05-LCD_D13-SSP2_DATA5, GPMI_D06-LCD_D14-SSP2_DATA6, GPMI_D07-LCD_D15-SSP2_DATA7, GPMI_RDY0-SSP2_DETECT, GPMI_RDY1-SSP2_CMD, GPMI_RDn, GPMI_WPn, GPMI_WRn-SSP2_SCK, HPL, HPR, I2C_SCL-GPMI_RDY2-AUART1_TX, I2C_SDA-GPMI_CE2n-AUART1_RX, LCD_CS, LCD_D00, LCD_D01, LCD_D02, LCD_D03, LCD_D04, LCD_D05, LCD_D06, LCD_D07, LCD_DOTCK-GPMI_RDY3, LCD_ENABLE-I2C_SCL, LCD_HSYNC-I2C_SDA, LCD_RESET-GPMI_CE3n, LCD_RS, LCD_VSYNC-LCD_BUSY, LCD_WR, LINE1_INL, LINE1_INR, LRADC0, LRADC1, MIC, PSWITCH, PWM0-ROTARYA-DUART_RX, PWM1-ROTARYB-DUART_TX, PWM2-GPMI_RDY3, SSP1_CMD-JTAG_TDO, SSP1_DATA0-JTAG_TDI, SSP1_DATA1-I2C_SCL-JTAG_TCLK, SSP1_DATA2-I2C_SDA-JTAG_RTCK, SSP1_DATA3-JTAG_TMS, SSP1_DETECT-GPMI_CE3N-USB_ID, SSP1_SCK-JTAG_TRST, USB_DM, USB_DP, VAG, VDAC1, XTALI, XTALO
Other:
- note added: "Notes:\n - All capacitors are X5R, 6.3V, 20%, ESR < 300mOhm or better unless otherwise noted\n - All resistors are 5% unless otherwise noted\n - Assuming 2-layer standard 1/16" FR4 (Dk=4.4, Df=0.02) and 7mil-7mil-15mil trace-space-drill design\n - Per Micron TN-46-02, need about 7 0.1uF bypass caps but to meet TN-46-14 layout guidelines use a\n lot more and consider external copper foil reference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"
- note removed: "Notes:\n - All capacitors are X5R, 6.3V, 20%, ESR < 300mOhm or better unless otherwise noted\n - All resistors are 5% unless otherwise noted\n - Assuming 2-layer standard 1/16" FR4 (Dk=4.4, Df=0.02) and 7mil-7mil-15mil trace-space-via design\n - Per Micron TN-46-02, need about 7 0.1uF bypass caps but to meet TN-46-14 layout guidelines use a\n lot more and consider external copper foil reference p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"
- moved on the sheet: C10, C11, C12, C13, C14, C15, C16, C17, C18, C19, C20, C21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

Commit message: Minor update to schematic.  Removed USB Power switch and added some notes.
Other:
- note added: "- However, all the traces are < 0.8" long and therefore have an electrical length of <8deg at 200MHz.\n Also, most signals have only one via. Only UDQS (EMI_DQS1) has three vias. Since there is very little\n room anyway, do not use termination resistors.\n - Only using one DDR device so should not require Rt and cannot fit it near i.MX233 IC anyway\n - For additional design and layout notes see T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"
Changed lines of the file:
@@
-EESchema Schematic File Version 2  date 19/04/2010 19:59:31
+EESchema Schematic File Version 2  date 21/04/2010 18:06:05
 LIBS:opendous
 LIBS:device
@@
 Sheet 3 8
 Title "PROpendous"
-Date "19 apr 2010"
+Date "21 apr 2010"
 Rev "1.0"
 Comp "Opendous Inc. (www.opendous.org)"
@@
 Comment4 "www.PROpendous.org"
 $EndDescr
+Text Notes 850  6850 0    60   ~ 0
+ - However, all the traces are < 0.8" long and therefore have an electrical length of <8deg at 200MHz.\n    Also, most signals have only one via. Only UDQS (EMI_DQS1) has three vias. Since there is very little\n    room anyway, do not use termination resistors.\n - Only using one DDR device so should not require Rt and cannot fit it near i.MX233 IC anyway\n - For additional design and layout notes see TN-46-11\n - TN AppNotes are available at www.micron.com
+Connection ~ 5950 4700
+Wire Wire Line
+	5950 4700 5950 4800
+Connection ~ 5800 4700
+Connection ~ 6000 4700
+Connection ~ 6200 4700
 Connection ~ 5950 5500
 Wire Wire Line
@@
 Connection ~ 7450 5500
 Wire Wire Line
-	4250 5500 7650 5500
+	7650 5500 4250 5500
 Connection ~ 7250 5500
 Connection ~ 4850 5500
@@
 Connection ~ 7500 4200
 Wire Wire Line
-	7500 4250 7500 4150
+	7500 4150 7500 4250
 Connection ~ 7300 4450
 Wire Wire Line
-	7100 4450 7500 4450
+	7500 4450 7100 4450
 Connection ~ 7300 3950
 Wire Wire Line
-	7100 3950 7500 3950
+	7500 3950 7100 3950
 Connection ~ 7050 5500
 Connection ~ 7050 5300
@@
 Connection ~ 4600 3550
 Wire Wire Line
-	5150 3550 4500 3550
+	4500 3550 5150 3550
 Connection ~ 4600 3750
 Wire Wire Line
-	4500 3750 5150 3750
+	5150 3750 4500 3750
 Connection ~ 5250 5500
 Connection ~ 5650 5500
@@
 Connection ~ 5250 5300
 Wire Wire Line
-	7100 4150 7100 4250
+	7100 4250 7100 4150
 Connection ~ 7300 4200
 Wire Wire Line
-	7300 4250 7300 4150
-Wire Wire Line
-	5950 4700 5950 4800
-Connection ~ 5750 4700
-Connection ~ 6050 4700
+	7300 4150 7300 4250
 Connection ~ 6200 1400
 Wire Wire Line
-	5600 1400 6300 1400
+	6300 1400 5600 1400
 Connection ~ 6000 1400
 Connection ~ 5800 1400
@@
 	5950 1400 5950 1300
 Connection ~ 5950 1400
-Connection ~ 6150 4700
-Wire Wire Line
-	5650 4700 6250 4700
-Connection ~ 5950 4700
-Connection ~ 5850 4700
 Connection ~ 7100 4200
 Connection ~ 5450 5300
@@
 Connection ~ 7250 5300
 Wire Wire Line
-	4250 5300 7650 5300
+	7650 5300 4250 5300
 Connection ~ 7450 5300
 Wire Wire Line
 	5950 5300 5950 5200
 Connection ~ 5950 5300
+Connection ~ 6100 4700
+Connection ~ 5900 4700
+Wire Wire Line
+	5600 4700 6300 4700
+Connection ~ 5700 4700
+$Comp
+L DDR_SDRAM_MT46_X16 IC2
+U 1 1 4BCEA1AD
+P 5950 3050
+F 0 "IC2" H 6500 1500 40  0000 C CNN
+F 1 "DDR_SDRAM_MT46_X16" H 5950 3400 40  0000 C CNN
+	1    5950 3050
+	1    0    0    -1
+$EndComp
 $Comp
 L VDDM_2V5 #PWR023
@@
 F 1 "VDDM_2V5" H 4600 3400 30  0000 C CNN
 	1    4600 3300
-	1    0    0    -1
-$EndComp
-$Comp
-L DDR_SDRAM_MT46_X16 IC2
-U 1 1 4BBCEC39
-P 5950 3050
-F 0 "IC2" H 6500 1500 40  0000 C CNN
-F 1 "DDR_SDRAM_MT46_X16" H 5950 3400 40  0000 C CNN
-	1    5950 3050
 	1    0    0    -1
 $EndComp
@@
 	0    1    1    0
 $EndComp
-Text Notes 1050 6850 0    60   ~ 0
-Notes:\n - All capacitors are X5R, 6.3V, 20%, ESR < 300mOhm or better unless otherwise noted\n - All resistors are 5% unless otherwise noted\n - Assuming 2-layer standard 1/16" FR4 (Dk=4.4, Df=0.02) and 7mil-7mil-15mil trace-space-drill design\n - Per Micron TN-46-02, need about 7 0.1uF bypass caps but to meet TN-46-14 layout guidelines use a\n    lot more and consider external copper foil reference planes\n - Cannot meet DDR routing guidelines (TN-46-14) on 2-layers so just keep all signals as short as possible\n    to limit effects on Signal Integrity (SI) of incorrect inter/intra-pair spacing\n - Only using one DDR device so should not require Rt and cannot fit it near i.MX233 IC anyway
+Text Notes 850  6050 0    60   ~ 0
+Notes:\n - All capacitors are X5R, 6.3V, 20%, ESR < 300mOhm or better unless otherwise noted\n - All resistors are 5% unless otherwise noted\n - Assuming 2-layer standard 1/16" FR4 (Dk=4.4, Df=0.02) and 7mil-7mil-15mil trace-space-drill design\n - Per Micron TN-46-02, need about 7 0.1uF bypass caps but to meet TN-46-14 layout guidelines use a\n    lot more and consider external copper foil reference planes\n - Cannot meet DDR routing guidelines (TN-46-14) on 2-layers so just keep all signals as short as possible\n    to limit effects on Signal Integrity (SI) of incorrect inter/intra-pair spacing\n - On 2-layer boards impedance of the lines is large so termination resistors should be used per TN-46-06.
 Text GLabel 5150 4450 0    40   BiDi ~ 0
 EMI_DQS1

Commit message: Updated PROpendous Project.  PCB layout is nearing completion.
Other:
- note added: "Notes:\n - All capacitors are X5R, 6.3V, 20%, ESR < 300mOhm or better unless otherwise noted\n - All resistors are 5% unless otherwise noted\n - Assuming 2-layer standard 1/16" FR4 (Dk=4.4, Df=0.02) and 7mil-7mil-15mil trace-space-drill design\n - Per Micron TN-46-02, need about 7 0.1uF bypass caps but to fake TN-46-14 layout guidelines of GND planes\n use a lot more and consider external copper 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"
- note removed: "Notes:\n - All capacitors are X5R, 6.3V, 20%, ESR < 300mOhm or better unless otherwise noted\n - All resistors are 5% unless otherwise noted\n - Assuming 2-layer standard 1/16" FR4 (Dk=4.4, Df=0.02) and 7mil-7mil-15mil trace-space-drill design\n - Per Micron TN-46-02, need about 7 0.1uF bypass caps but to meet TN-46-14 layout guidelines use a\n lot more and consider external copper foil reference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"
Changed lines of the file:
@@
-EESchema Schematic File Version 2  date 21/04/2010 18:06:05
+EESchema Schematic File Version 2  date 24/04/2010 02:27:16
 LIBS:opendous
 LIBS:device
@@
 Sheet 3 8
 Title "PROpendous"
-Date "21 apr 2010"
+Date "24 apr 2010"
 Rev "1.0"
 Comp "Opendous Inc. (www.opendous.org)"
@@
 $EndComp
 Text Notes 850  6050 0    60   ~ 0
-Notes:\n - All capacitors are X5R, 6.3V, 20%, ESR < 300mOhm or better unless otherwise noted\n - All resistors are 5% unless otherwise noted\n - Assuming 2-layer standard 1/16" FR4 (Dk=4.4, Df=0.02) and 7mil-7mil-15mil trace-space-drill design\n - Per Micron TN-46-02, need about 7 0.1uF bypass caps but to meet TN-46-14 layout guidelines use a\n    lot more and consider external copper foil reference planes\n - Cannot meet DDR routing guidelines (TN-46-14) on 2-layers so just keep all signals as short as possible\n    to limit effects on Signal Integrity (SI) of incorrect inter/intra-pair spacing\n - On 2-layer boards impedance of the lines is large so termination resistors should be used per TN-46-06.
+Notes:\n - All capacitors are X5R, 6.3V, 20%, ESR < 300mOhm or better unless otherwise noted\n - All resistors are 5% unless otherwise noted\n - Assuming 2-layer standard 1/16" FR4 (Dk=4.4, Df=0.02) and 7mil-7mil-15mil trace-space-drill design\n - Per Micron TN-46-02, need about 7 0.1uF bypass caps but to fake TN-46-14 layout guidelines of GND planes\n    use a lot more and consider external copper foil reference planes\n - Cannot meet DDR routing guidelines (TN-46-14) on 2-layers so just keep all signals as short as possible\n    to limit effects on Signal Integrity (SI) of incorrect inter/intra-pair spacing and characteristic trace impedance\n - On 2-layer boards impedance of the lines is large so termination resistors should be used per TN-46-06.
 Text GLabel 5150 4450 0    40   BiDi ~ 0
 EMI_DQS1
