File: PRopendous/Hardware/PROpendous/PROpendous-Memory.sch (KiCad schematic (older format))
At the start: 28 parts, among them IC2 DDR_SDRAM_MT46_X16

Commit message: Updated design files.  Added picture of finished PCB.
Parts:
- C27: value 68uF -> 47uF
Other:
- note added: "C26 ESR = 900mOhm"
- note added: "C27 ESR = 3-Ohm"
Changed lines of the file:
@@
-EESchema Schematic File Version 2  date 27/04/2010 18:25:33
+EESchema Schematic File Version 2  date 07/05/2010 11:28:22
 LIBS:opendous
 LIBS:device
@@
 LIBS:valves
 LIBS:power
-LIBS:PROpendous-cache
 EELAYER 24  0
 EELAYER END
@@
 Sheet 3 8
 Title "PROpendous"
-Date "27 apr 2010"
+Date "7 may 2010"
 Rev "1.0"
 Comp "Opendous Inc. (www.opendous.org)"
@@
 Comment4 "www.PROpendous.org"
 $EndDescr
+Text Notes 7400 5250 0    30   ~ 0
+C26 ESR = 900mOhm
+Text Notes 7600 5600 0    30   ~ 0
+C27 ESR = 3-Ohm
 Text Notes 850  6850 0    60   ~ 0
  - However, all the traces are < 0.8" long and therefore have an electrical length of <8deg at 200MHz.\n    Also, most signals have only one via. Only UDQS (EMI_DQS1) has three vias. Since there is very little\n    room anyway, do not use termination resistors.\n - Only using one DDR device so should not require Rt and cannot fit it near i.MX233 IC anyway\n - For additional design and layout notes see TN-46-11\n - TN AppNotes are available at www.micron.com
@@
 P 7650 5400
 F 0 "C27" V 7600 5450 30  0000 C CNN
-F 1 "68uF" V 7700 5450 25  0000 C CNN
+F 1 "47uF" V 7700 5450 25  0000 C CNN
 	1    7650 5400
 	0    1    1    0

Commit message: Switch to ceramic capacitors for bulk decoupling which are less expensive than similarly low-ESR tantalum capacitors.
Parts:
- removed C27: 47uF, symbol CP_TANTALUM_MINI
- added C27: 47uF, symbol C_MINI
- C26: value 68uF -> 47uF
Other:
- note removed: "C26 ESR = 900mOhm"
- note removed: "C27 ESR = 3-Ohm"
Changed lines of the file:
@@
-EESchema Schematic File Version 2  date 07/06/2010 07:15:05
+EESchema Schematic File Version 2  date 17/06/2010 09:45:34
 LIBS:opendous
 LIBS:device
@@
 LIBS:valves
 LIBS:power
-LIBS:PROpendous-cache
 EELAYER 24  0
 EELAYER END
@@
 Sheet 3 8
 Title "PROpendous"
-Date "7 jun 2010"
+Date "17 jun 2010"
 Rev "1.0"
 Comp "Opendous Inc. (www.opendous.org)"
@@
 Comment4 "www.PROpendous.org"
 $EndDescr
-Text Notes 7400 5250 0    30   ~ 0
-C26 ESR = 900mOhm
-Text Notes 7600 5600 0    30   ~ 0
-C27 ESR = 3-Ohm
+$Comp
+L CP_TANTALUM_MINI C26
+U 1 1 4C1A1AD3
+P 7650 5400
+F 0 "C26" V 7600 5450 30  0000 C CNN
+F 1 "47uF" V 7700 5450 25  0000 C CNN
+	1    7650 5400
+	0    1    1    0
+$EndComp
+$Comp
+L C_MINI C27
+U 1 1 4C1A1730
+P 7450 5400
+F 0 "C27" V 7400 5450 30  0000 C CNN
+F 1 "47uF" V 7500 5450 25  0000 C CNN
+	1    7450 5400
+	0    1    1    0
+$EndComp
 Text Notes 850  6850 0    60   ~ 0
  - However, all the traces are < 0.8" long and therefore have an electrical length of <8deg at 200MHz.\n    Also, most signals have only one via. Only UDQS (EMI_DQS1) has three vias. Since there is very little\n    room anyway, do not use termination resistors.\n - Only using one DDR device so should not require Rt and cannot fit it near i.MX233 IC anyway\n - For additional design and layout notes see TN-46-11\n - TN AppNotes are available at www.micron.com
@@
 	1    0    0    -1
 $EndComp
-$Comp
-L CP_TANTALUM_MINI C27
-U 1 1 4BC981AE
-P 7650 5400
-F 0 "C27" V 7600 5450 30  0000 C CNN
-F 1 "47uF" V 7700 5450 25  0000 C CNN
-	1    7650 5400
-	0    1    1    0
-$EndComp
-$Comp
-L CP_TANTALUM_MINI C26
-U 1 1 4BC981A1
-P 7450 5400
-F 0 "C26" V 7400 5450 30  0000 C CNN
-F 1 "68uF" V 7500 5450 25  0000 C CNN
-	1    7450 5400
-	0    1    1    0
-$EndComp
 Text GLabel 6600 7700 2    40   BiDi ~ 0
