File: PRopendous/Hardware/PROpendous/PROpendous-Vias.sch (KiCad schematic (older format))
At the start: 0 parts

Commit message: Updated files.  DDR SDRAM schematic completed.
Connections:
- net labels added: VDD4V2, VDD5V, VDDA, VDDD, VDDIO_3V3, VDDM_2V5, VDD_BATT, VDD_XTAL

Commit message: Updated PROpendous i.MX233 project.  DDR SDRAM layout is complete.
Parts:
- added V1, V10, V100, V101, V102, V103, V104, V105, V106, V107, V108, V109, V11, V110, V111, V112, V113, V114, V115, V116, V117, V118, V119, V12, V120, V121, V122, V123, V124, V125, V126, V127, V128, V129, V13, V130, V131, V132, V133, V134, V135, V136, V137, V138, V139, V14, V140, V141, V142, V143, V144, V145, V146, V147, V148, V149, V15, V150, V151, V152, V153, V154, V155, V156, V157, V158, V159, V16, V160, V161, V162, V163, V164, V165, V166, V167, V168, V169, V17, V170, V171, V172, V173, V174, V175, V176, V177, V178, V179, V18, V180, V181, V182, V183, V184, V185, V186, V187, V188, V189, V19, V190, V191, V192, V193, V194, V195, V196, V197, V198, V199, V2, V20, V200, V201, V202, V203, V204, V205, V206, V207, V208, V209, V21, V210, V211, V212, V213, V214, V215, V216, V217, V218, V219, V22, V220, V221, V222, V223, V224, V225, V226, V227, V228, V229, V23, V230, V231, V232, V233, V234, V235, V236, V237, V238, V239, V24, V240, V241, V242, V243, V244, V245, V246, V247, V248, V249, V25, V250, V251, V252, V253, V254, V255, V256, V257, V258, V259, V26, V260, V261, V262, V263, V264, V265, V266, V267, V268, V269, V27, V270, V271, V272, V273, V274, V275, V276, V277, V278, V279, V28, V280, V281, V282, V283, V284, V285, V286, V287, V288, V289, V29, V290, V291, V292, V293, V294, V295, V296, V297, V298, V299, V3, V30, V300, V301, V302, V303, V304, V305, V306, V307, V308, V309, V31, V310, V311, V312, V313, V314, V315, V316, V317, V318, V319, V32, V320, V321, V322, V323, V324, V33, V34, V35, V36, V37, V38, V39, V4, V40, V41, V42, V43, V44, V45, V46, V47, V48, V49, V5, V50, V51, V52, V53, V54, V55, V56, V57, V58, V59, V6, V60, V61, V62, V63, V64, V65, V66, V67, V68, V69, V7, V70, V71, V72, V73, V74, V75, V76, V77, V78, V79, V8, V80, V81, V82, V83, V84, V85, V86, V87, V88, V89, V9, V90, V91, V92, V93, V94, V95, V96, V97, V98, V99: VIA, symbol VIA
Connections:
- net labels added: DDR_VREF, GND
- wire segments 0 -> 44

Commit message: Updated PROpendous project.  Schematic is complete but not yet finalized.  Layout partially complete.
Connections:
- net labels added: TSC_IN1, TSC_IN2, TSC_VBAT1, TSC_VBAT2, TSC_VREF
- wire segments 44 -> 56
Other:
- note added: "When routing a board this complex, it helps to have persistant vias (vias that behave like components) in order to plan board layout"
- note removed: "When routing a board this complex, it helps to have persistant vias (vias that behave like components)"
Changed lines of the file:
@@
-EESchema Schematic File Version 2  date 17/04/2010 17:25:37
+EESchema Schematic File Version 2  date 19/04/2010 19:59:31
 LIBS:opendous
 LIBS:device
@@
 EELAYER END
 $Descr A4 11700 8267
-Sheet 7 7
+Sheet 8 8
 Title "PROpendous"
-Date "17 apr 2010"
+Date "19 apr 2010"
 Rev "1.0"
 Comp "Opendous Inc. (www.opendous.org)"
@@
 Comment4 "www.PROpendous.org"
 $EndDescr
-Connection ~ 7950 3100
+Connection ~ 7950 4300
+Wire Wire Line
+	8000 4400 7950 4400
+Wire Wire Line
+	7950 4400 7950 800
+Connection ~ 7950 4100
+Wire Wire Line
+	7950 4200 8000 4200
+Connection ~ 7950 3900
+Wire Wire Line
+	7950 4000 8000 4000
+Connection ~ 7950 3700
+Wire Wire Line
+	7950 3800 8000 3800
+Connection ~ 7950 3500
+Wire Wire Line
+	7950 3600 8000 3600
+Connection ~ 7950 3300
 Wire Wire Line
-	7950 3200 7950 800
+	7950 3400 8000 3400
+Connection ~ 7950 3100
 Wire Wire Line
 	7950 3200 8000 3200
@@
 	7950 3100 8000 3100
 Connection ~ 7950 3000
+Wire Wire Line
+	7950 3300 8000 3300
+Connection ~ 7950 3200
+Wire Wire Line
+	7950 3500 8000 3500
+Connection ~ 7950 3400
+Wire Wire Line
+	7950 3700 8000 3700
+Connection ~ 7950 3600
+Wire Wire Line
+	7950 3900 8000 3900
+Connection ~ 7950 3800
+Wire Wire Line
+	7950 4100 8000 4100
+Connection ~ 7950 4000
+Wire Wire Line
+	7950 4300 8000 4300
+Connection ~ 7950 4200
 $Comp
 L VIA V323
@@
 $EndComp
 $Comp
-L VDDM_2V5 #PWR073
+L VDDM_2V5 #PWR0133
 U 1 1 4BC98266
 P 3200 7300
-F 0 "#PWR073" H 3200 7400 30  0001 C CNN
+F 0 "#PWR0133" H 3200 7400 30  0001 C CNN
 F 1 "VDDM_2V5" V 3200 7500 30  0000 C CNN
 	1    3200 7300
@@
 $EndComp
 $Comp
-L VDDM_2V5 #PWR074
+L VDDM_2V5 #PWR0134
 U 1 1 4BC98265
 P 3300 7300
-F 0 "#PWR074" H 3300 7400 30  0001 C CNN
+F 0 "#PWR0134" H 3300 7400 30  0001 C CNN
 F 1 "VDDM_2V5" V 3300 7500 30  0000 C CNN
 	1    3300 7300
@@
 $EndComp
 $Comp
-L VDDM_2V5 #PWR075
+L VDDM_2V5 #PWR0135
 U 1 1 4BC98264
 P 3500 7300
-F 0 "#PWR075" H 3500 7400 30  0001 C CNN
+F 0 "#PWR0135" H 3500 7400 30  0001 C CNN
 F 1 "VDDM_2V5" V 3500 7500 30  0000 C CNN
 	1    3500 7300
@@
 $EndComp
 $Comp
-L VDDM_2V5 #PWR076
+L VDDM_2V5 #PWR0136
 U 1 1 4BC98263
 P 3400 7300
-F 0 "#PWR076" H 3400 7400 30  0001 C CNN
+F 0 "#PWR0136" H 3400 7400 30  0001 C CNN
 F 1 "VDDM_2V5" V 3400 7500 30  0000 C CNN
 	1    3400 7300
@@
 $EndComp
 $Comp
-L VDDM_2V5 #PWR077
+L VDDM_2V5 #PWR0137
 U 1 1 4BC98261
 P 3600 7300
-F 0 "#PWR077" H 3600 7400 30  0001 C CNN
+F 0 "#PWR0137" H 3600 7400 30  0001 C CNN
 F 1 "VDDM_2V5" V 3600 7500 30  0000 C CNN
 	1    3600 7300
@@
 $EndComp
 $Comp
-L VDDM_2V5 #PWR078
+L VDDM_2V5 #PWR0138
 U 1 1 4BC98260
 P 3500 7300
-F 0 "#PWR078" H 3500 7400 30  0001 C CNN
+F 0 "#PWR0138" H 3500 7400 30  0001 C CNN
 F 1 "VDDM_2V5" V 3500 7500 30  0000 C CNN
 	1    3500 7300
@@
 $EndComp
 $Comp
-L VDDM_2V5 #PWR079
+L VDDM_2V5 #PWR0139
 U 1 1 4BC9825F
 P 3100 7300
-F 0 "#PWR079" H 3100 7400 30  0001 C CNN
+F 0 "#PWR0139" H 3100 7400 30  0001 C CNN
 F 1 "VDDM_2V5" V 3100 7500 30  0000 C CNN
 	1    3100 7300
@@
 $EndComp
 $Comp
-L VDDM_2V5 #PWR080
+L VDDM_2V5 #PWR0140
 U 1 1 4BC97F6E
 P 3700 7300
-F 0 "#PWR080" H 3700 7400 30  0001 C CNN
+F 0 "#PWR0140" H 3700 7400 30  0001 C CNN
 F 1 "VDDM_2V5" V 3700 7500 30  0000 C CNN
 	1    3700 7300
@@
 $EndComp
 $Comp
-L VDDM_2V5 #PWR081
+L VDDM_2V5 #PWR0141
 U 1 1 4BC97115
 P 4400 7300
-F 0 "#PWR081" H 4400 7400 30  0001 C CNN
+F 0 "#PWR0141" H 4400 7400 30  0001 C CNN
 F 1 "VDDM_2V5" V 4400 7500 30  0000 C CNN
 	1    4400 7300
@@
 $EndComp
 $Comp
-L VDDM_2V5 #PWR082
+L VDDM_2V5 #PWR0142
 U 1 1 4BC97114
 P 4500 7300
-F 0 "#PWR082" H 4500 7400 30  0001 C CNN
+F 0 "#PWR0142" H 4500 7400 30  0001 C CNN
 F 1 "VDDM_2V5" V 4500 7500 30  0000 C CNN
 	1    4500 7300
@@
 $EndComp
 $Comp
-L VDDM_2V5 #PWR083
+L VDDM_2V5 #PWR0143
 U 1 1 4BC97113
 P 4700 7300
-F 0 "#PWR083" H 4700 7400 30  0001 C CNN
+F 0 "#PWR0143" H 4700 7400 30  0001 C CNN
 F 1 "VDDM_2V5" V 4700 7500 30  0000 C CNN
 	1    4700 7300
@@
 $EndComp
 $Comp
-L VDDM_2V5 #PWR084
+L VDDM_2V5 #PWR0144
 U 1 1 4BC97112
 P 4600 7300
-F 0 "#PWR084" H 4600 7400 30  0001 C CNN
+F 0 "#PWR0144" H 4600 7400 30  0001 C CNN
 F 1 "VDDM_2V5" V 4600 7500 30  0000 C CNN
 	1    4600 7300
@@
 $EndComp
 $Comp
-L VDDM_2V5 #PWR085
+L VDDM_2V5 #PWR0145
 U 1 1 4BC97110
 P 4800 7300
-F 0 "#PWR085" H 4800 7400 30  0001 C CNN
+F 0 "#PWR0145" H 4800 7400 30  0001 C CNN
 F 1 "VDDM_2V5" V 4800 7500 30  0000 C CNN
 	1    4800 7300
@@
 $EndComp
 $Comp
-L VDDM_2V5 #PWR086
+L VDDM_2V5 #PWR0146
 U 1 1 4BC9710F
 P 4700 7300
-F 0 "#PWR086" H 4700 7400 30  0001 C CNN
+F 0 "#PWR0146" H 4700 7400 30  0001 C CNN
 F 1 "VDDM_2V5" V 4700 7500 30  0000 C CNN
 	1    4700 7300
@@
 $EndComp
 $Comp
-L VDDM_2V5 #PWR087
+L VDDM_2V5 #PWR0147
 U 1 1 4BC94F2E
 P 4100 7300
-F 0 "#PWR087" H 4100 7400 30  0001 C CNN
+F 0 "#PWR0147" H 4100 7400 30  0001 C CNN
 F 1 "VDDM_2V5" V 4100 7500 30  0000 C CNN
 	1    4100 7300
@@
 $EndComp
 $Comp
-L VDDM_2V5 #PWR088
+L VDDM_2V5 #PWR0148
 U 1 1 4BC94F2D
 P 4300 7300
-F 0 "#PWR088" H 4300 7400 30  0001 C CNN
+F 0 "#PWR0148" H 4300 7400 30  0001 C CNN
 F 1 "VDDM_2V5" V 4300 7500 30  0000 C CNN
 	1    4300 7300
@@
 $EndComp
 $Comp
-L VDDM_2V5 #PWR089
+L VDDM_2V5 #PWR0149
 U 1 1 4BC94F2C
 P 4200 7300
-F 0 "#PWR089" H 4200 7400 30  0001 C CNN
+F 0 "#PWR0149" H 4200 7400 30  0001 C CNN
 F 1 "VDDM_2V5" V 4200 7500 30  0000 C CNN
 	1    4200 7300
@@
 $EndComp
 $Comp
-L VDDM_2V5 #PWR090
+L VDDM_2V5 #PWR0150
 U 1 1 4BC94F1A
 P 4000 7300
-F 0 "#PWR090" H 4000 7400 30  0001 C CNN
+F 0 "#PWR0150" H 4000 7400 30  0001 C CNN
 F 1 "VDDM_2V5" V 4000 7500 30  0000 C CNN
 	1    4000 7300
@@
 $EndComp
 $Comp
-L VDDM_2V5 #PWR091
+L VDDM_2V5 #PWR0151
 U 1 1 4BC94F19
 P 4100 7300
-F 0 "#PWR091" H 4100 7400 30  0001 C CNN
+F 0 "#PWR0151" H 4100 7400 30  0001 C CNN
 F 1 "VDDM_2V5" V 4100 7500 30  0000 C CNN
 	1    4100 7300
@@
 $EndComp
 $Comp
-L VDDM_2V5 #PWR092
+L VDDM_2V5 #PWR0152
 U 1 1 4BC94F15
 P 3900 7300
-F 0 "#PWR092" H 3900 7400 30  0001 C CNN
+F 0 "#PWR0152" H 3900 7400 30  0001 C CNN
 F 1 "VDDM_2V5" V 3900 7500 30  0000 C CNN
 	1    3900 7300
@@
 $EndComp
 $Comp
-L VDDM_2V5 #PWR093
+L VDDM_2V5 #PWR0153
 U 1 1 4BC94EFD
 P 3800 7300
-F 0 "#PWR093" H 3800 7400 30  0001 C CNN
+F 0 "#PWR0153" H 3800 7400 30  0001 C CNN
 F 1 "VDDM_2V5" V 3800 7500 30  0000 C CNN
 	1    3800 7300
@@
 EMI_DQS1
 $Comp
-L GND #PWR094
+L GND #PWR0154
 U 1 1 4BC39D91
 P 8100 850
-F 0 "#PWR094" H 8100 850 30  0001 C CNN
+F 0 "#PWR0154" H 8100 850 30  0001 C CNN
 F 1 "GND" H 8100 780 30  0001 C CNN
 	1    8100 850
@@
 EMI_A06
 Text Notes 550  600  0    60   ~ 0
-When routing a board this complex, it helps to have persistant vias (vias that behave like components)
+When routing a board this complex, it helps to have persistant vias (vias that behave like components) in order to plan board layout
 Text GLabel 9600 1650 0    40   BiDi ~ 0
 LCD_D00
@@
 PSWITCH
 $Comp
-L VDD5V #PWR095
+L VDD5V #PWR0155
 U 1 1 4BBCE20A
 P 3950 1850
-F 0 "#PWR095" H 3950 1950 30  0001 C CNN
+F 0 "#PWR0155" H 3950 1950 30  0001 C CNN
 F 1 "VDD5V" H 3950 1950 30  0000 C CNN
 	1    3950 1850
@@
 $EndComp
 $Comp
-L VDD_BATT #PWR096
+L VDD_BATT #PWR0156
 U 1 1 4BBCCFD0
 P 2450 1850
-F 0 "#PWR096" H 2450 1950 30  0001 C CNN
+F 0 "#PWR0156" H 2450 1950 30  0001 C CNN
 F 1 "VDD_BATT" H 2450 1950 30  0000 C CNN
 	1    2450 1850
@@
 $EndComp
 $Comp
-L VDD4V2 #PWR097
+L VDD4V2 #PWR0157
 U 1 1 4BBCCFCF
 P 2700 1850
-F 0 "#PWR097" H 2700 1950 30  0001 C CNN
+F 0 "#PWR0157" H 2700 1950 30  0001 C CNN
 F 1 "VDD4V2" H 2700 1950 30  0000 C CNN
 	1    2700 1850
@@
 $EndComp
 $Comp
-L VDDIO_3V3 #PWR098
+L VDDIO_3V3 #PWR0158
 U 1 1 4BBCCFCE
 P 3200 1850
-F 0 "#PWR098" H 3200 1950 30  0001 C CNN
+F 0 "#PWR0158" H 3200 1950 30  0001 C CNN
 F 1 "VDDIO_3V3" H 3200 1950 30  0000 C CNN
 	1    3200 1850
@@
 $EndComp
 $Comp
-L VDDD #PWR099
+L VDDD #PWR0159
 U 1 1 4BBCE206
 P 3450 1850
-F 0 "#PWR099" H 3450 1950 30  0001 C CNN
+F 0 "#PWR0159" H 3450 1950 30  0001 C CNN
 F 1 "VDDD" H 3450 1950 30  0000 C CNN
 	1    3450 1850
@@
 $EndComp
 $Comp
-L VDDA #PWR0100
+L VDDA #PWR0160
 U 1 1 4BBCE205
 P 3750 1850
-F 0 "#PWR0100" H 3750 1950 30  0001 C CNN
+F 0 "#PWR0160" H 3750 1950 30  0001 C CNN
 F 1 "VDDA" H 3750 1950 30  0000 C CNN
 	1    3750 1850
@@
 $EndComp
 $Comp
-L VDD_XTAL #PWR0101
+L VDD_XTAL #PWR0161
 U 1 1 4BBCE204
 P 4200 1850
-F 0 "#PWR0101" H 4200 1950 30  0001 C CNN
+F 0 "#PWR0161" H 4200 1950 30  0001 C CNN
 F 1 "VDD_XTAL" H 4200 1950 30  0000 C CNN
 	1    4200 1850
@@
 $EndComp
 $Comp
-L VDDM_2V5 #PWR0102
+L VDDM_2V5 #PWR0162
 U 1 1 4BBCCFC9
 P 4550 1850
-F 0 "#PWR0102" H 4550 1950 30  0001 C CNN
+F 0 "#PWR0162" H 4550 1950 30  0001 C CNN
 F 1 "VDDM_2V5" H 4550 1950 30  0000 C CNN
 	1    4550 1850
 	1    0    0    -1
 $EndComp
+Text GLabel 10300 2950 2    40   BiDi ~ 0
+TSC_IN1
+Text GLabel 10300 3050 2    40   BiDi ~ 0
+TSC_IN2
+Text GLabel 10300 3200 2    40   BiDi ~ 0
+TSC_VBAT1
+Text GLabel 10300 3300 2    40   BiDi ~ 0
+TSC_VBAT2
+Text GLabel 10150 3200 0    40   BiDi ~ 0
+TSC_VREF
 $EndSCHEMATC

Commit message: Minor update to schematic.  Removed USB Power switch and added some notes.
Parts:
- added V325, V326, V327, V328: VIA, symbol VIA
Connections:
- net labels added: DMa, DMb, DPa, DPb, FSUSB20_nOE
- wire segments 56 -> 60
Changed lines of the file:
@@
-EESchema Schematic File Version 2  date 19/04/2010 19:59:31
+EESchema Schematic File Version 2  date 21/04/2010 18:06:05
 LIBS:opendous
 LIBS:device
@@
 Sheet 8 8
 Title "PROpendous"
-Date "19 apr 2010"
+Date "21 apr 2010"
 Rev "1.0"
 Comp "Opendous Inc. (www.opendous.org)"
@@
 Comment4 "www.PROpendous.org"
 $EndDescr
+Text GLabel 1300 6950 0    40   BiDi ~ 0
+DMa
+Text GLabel 1300 7050 0    40   BiDi ~ 0
+DPa
+Text GLabel 10900 5400 0    40   BiDi ~ 0
+DPa
+Text GLabel 10900 5600 0    40   BiDi ~ 0
+DPb
+Text GLabel 10900 5300 0    40   BiDi ~ 0
+DMa
+Text GLabel 10900 5500 0    40   BiDi ~ 0
+DMb
+$Comp
+L VDDIO_3V3 #PWR0138
+U 1 1 4BCED90C
+P 2700 7300
+F 0 "#PWR0138" H 2700 7400 30  0001 C CNN
+F 1 "VDDIO_3V3" V 2700 7500 30  0000 C CNN
+	1    2700 7300
+	1    0    0    -1
+$EndComp
+$Comp
+L VDDIO_3V3 #PWR0139
+U 1 1 4BCED90B
+P 2400 7300
+F 0 "#PWR0139" H 2400 7400 30  0001 C CNN
+F 1 "VDDIO_3V3" V 2400 7500 30  0000 C CNN
+	1    2400 7300
+	1    0    0    -1
+$EndComp
+$Comp
+L VDDIO_3V3 #PWR0140
+U 1 1 4BCED909
+P 2500 7300
+F 0 "#PWR0140" H 2500 7400 30  0001 C CNN
+F 1 "VDDIO_3V3" V 2500 7500 30  0000 C CNN
+	1    2500 7300
+	1    0    0    -1
+$EndComp
+$Comp
+L VIA V325
+U 1 1 4BCED902
+P 2400 7350
+F 0 "V325" V 2425 7450 20  0000 C CNN
+F 1 "VIA" H 2400 7550 60  0001 C CNN
+	1    2400 7350
+	-1   0    0    1
+$EndComp
+$Comp
+L VIA V326
+U 1 1 4BCED8FB
+P 2500 7350
+F 0 "V326" V 2525 7450 20  0000 C CNN
+F 1 "VIA" H 2500 7550 60  0001 C CNN
+	1    2500 7350
+	-1   0    0    1
+$EndComp
+$Comp
+L VIA V327
+U 1 1 4BCED8FA
+P 2600 7350
+F 0 "V327" V 2625 7450 20  0000 C CNN
+F 1 "VIA" H 2600 7550 60  0001 C CNN
+	1    2600 7350
+	-1   0    0    1
+$EndComp
+$Comp
+L VIA V328
+U 1 1 4BCED8F9
+P 2700 7350
+F 0 "V328" V 2725 7450 20  0000 C CNN
+F 1 "VIA" H 2700 7550 60  0001 C CNN
+	1    2700 7350
+	-1   0    0    1
+$EndComp
+Wire Wire Line
+	2400 7350 2400 7300
+Wire Wire Line
+	2700 7350 2700 7300
+Wire Wire Line
+	2500 7350 2500 7300
+Wire Wire Line
+	2600 7350 2600 7300
+$Comp
+L VDDIO_3V3 #PWR0141
+U 1 1 4BCED8F4
+P 2600 7300
+F 0 "#PWR0141" H 2600 7400 30  0001 C CNN
+F 1 "VDDIO_3V3" V 2600 7500 30  0000 C CNN
+	1    2600 7300
+	1    0    0    -1
+$EndComp
+Text GLabel 1300 6850 0    40   BiDi ~ 0
+FSUSB20_nOE
+Text GLabel 1300 6750 0    40   BiDi ~ 0
+PWM2-GPMI_RDY3
 Connection ~ 7950 4300
 Wire Wire Line
@@
 $EndComp
 $Comp
-L VDDM_2V5 #PWR0133
+L VDDM_2V5 #PWR0142
 U 1 1 4BC98266
 P 3200 7300
-F 0 "#PWR0133" H 3200 7400 30  0001 C CNN
+F 0 "#PWR0142" H 3200 7400 30  0001 C CNN
 F 1 "VDDM_2V5" V 3200 7500 30  0000 C CNN
 	1    3200 7300
@@
 $EndComp
 $Comp
-L VDDM_2V5 #PWR0134
+L VDDM_2V5 #PWR0143
 U 1 1 4BC98265
 P 3300 7300
-F 0 "#PWR0134" H 3300 7400 30  0001 C CNN
+F 0 "#PWR0143" H 3300 7400 30  0001 C CNN
 F 1 "VDDM_2V5" V 3300 7500 30  0000 C CNN
 	1    3300 7300
@@
 $EndComp
 $Comp
-L VDDM_2V5 #PWR0135
+L VDDM_2V5 #PWR0144
 U 1 1 4BC98264
 P 3500 7300
-F 0 "#PWR0135" H 3500 7400 30  0001 C CNN
+F 0 "#PWR0144" H 3500 7400 30  0001 C CNN
 F 1 "VDDM_2V5" V 3500 7500 30  0000 C CNN
 	1    3500 7300
@@
 $EndComp
 $Comp
-L VDDM_2V5 #PWR0136
+L VDDM_2V5 #PWR0145
 U 1 1 4BC98263
 P 3400 7300
-F 0 "#PWR0136" H 3400 7400 30  0001 C CNN
+F 0 "#PWR0145" H 3400 7400 30  0001 C CNN
 F 1 "VDDM_2V5" V 3400 7500 30  0000 C CNN
 	1    3400 7300
@@
 $EndComp
 $Comp
-L VDDM_2V5 #PWR0137
+L VDDM_2V5 #PWR0146
 U 1 1 4BC98261
 P 3600 7300
-F 0 "#PWR0137" H 3600 7400 30  0001 C CNN
+F 0 "#PWR0146" H 3600 7400 30  0001 C CNN
 F 1 "VDDM_2V5" V 3600 7500 30  0000 C CNN
 	1    3600 7300
@@
 $EndComp
 $Comp
-L VDDM_2V5 #PWR0138
+L VDDM_2V5 #PWR0147
 U 1 1 4BC98260
 P 3500 7300
-F 0 "#PWR0138" H 3500 7400 30  0001 C CNN
+F 0 "#PWR0147" H 3500 7400 30  0001 C CNN
 F 1 "VDDM_2V5" V 3500 7500 30  0000 C CNN
 	1    3500 7300
@@
 $EndComp
 $Comp
-L VDDM_2V5 #PWR0139
+L VDDM_2V5 #PWR0148
 U 1 1 4BC9825F
 P 3100 7300
-F 0 "#PWR0139" H 3100 7400 30  0001 C CNN
+F 0 "#PWR0148" H 3100 7400 30  0001 C CNN
 F 1 "VDDM_2V5" V 3100 7500 30  0000 C CNN
 	1    3100 7300
@@
 $EndComp
 $Comp
-L VDDM_2V5 #PWR0140
+L VDDM_2V5 #PWR0149
 U 1 1 4BC97F6E
 P 3700 7300
-F 0 "#PWR0140" H 3700 7400 30  0001 C CNN
+F 0 "#PWR0149" H 3700 7400 30  0001 C CNN
 F 1 "VDDM_2V5" V 3700 7500 30  0000 C CNN
 	1    3700 7300
@@
 $EndComp
 $Comp
-L VDDM_2V5 #PWR0141
+L VDDM_2V5 #PWR0150
 U 1 1 4BC97115
 P 4400 7300
-F 0 "#PWR0141" H 4400 7400 30  0001 C CNN
+F 0 "#PWR0150" H 4400 7400 30  0001 C CNN
 F 1 "VDDM_2V5" V 4400 7500 30  0000 C CNN
 	1    4400 7300
@@
 $EndComp
 $Comp
-L VDDM_2V5 #PWR0142
+L VDDM_2V5 #PWR0151
 U 1 1 4BC97114
 P 4500 7300
-F 0 "#PWR0142" H 4500 7400 30  0001 C CNN
+F 0 "#PWR0151" H 4500 7400 30  0001 C CNN
 F 1 "VDDM_2V5" V 4500 7500 30  0000 C CNN
 	1    4500 7300
@@
 $EndComp
 $Comp
-L VDDM_2V5 #PWR0143
+L VDDM_2V5 #PWR0152
 U 1 1 4BC97113
 P 4700 7300
-F 0 "#PWR0143" H 4700 7400 30  0001 C CNN
+F 0 "#PWR0152" H 4700 7400 30  0001 C CNN
 F 1 "VDDM_2V5" V 4700 7500 30  0000 C CNN
 	1    4700 7300
@@
 $EndComp
 $Comp
-L VDDM_2V5 #PWR0144
+L VDDM_2V5 #PWR0153
 U 1 1 4BC97112
 P 4600 7300
-F 0 "#PWR0144" H 4600 7400 30  0001 C CNN
+F 0 "#PWR0153" H 4600 7400 30  0001 C CNN
 F 1 "VDDM_2V5" V 4600 7500 30  0000 C CNN
 	1    4600 7300
@@
 $EndComp
 $Comp
-L VDDM_2V5 #PWR0145
+L VDDM_2V5 #PWR0154
 U 1 1 4BC97110
 P 4800 7300
-F 0 "#PWR0145" H 4800 7400 30  0001 C CNN
+F 0 "#PWR0154" H 4800 7400 30  0001 C CNN
 F 1 "VDDM_2V5" V 4800 7500 30  0000 C CNN
 	1    4800 7300
@@
 $EndComp
 $Comp
-L VDDM_2V5 #PWR0146
+L VDDM_2V5 #PWR0155
 U 1 1 4BC9710F
 P 4700 7300
-F 0 "#PWR0146" H 4700 7400 30  0001 C CNN
+F 0 "#PWR0155" H 4700 7400 30  0001 C CNN
 F 1 "VDDM_2V5" V 4700 7500 30  0000 C CNN
 	1    4700 7300
@@
 $EndComp
 $Comp
-L VDDM_2V5 #PWR0147
+L VDDM_2V5 #PWR0156
 U 1 1 4BC94F2E
 P 4100 7300
-F 0 "#PWR0147" H 4100 7400 30  0001 C CNN
+F 0 "#PWR0156" H 4100 7400 30  0001 C CNN
 F 1 "VDDM_2V5" V 4100 7500 30  0000 C CNN
 	1    4100 7300
@@
 $EndComp
 $Comp
-L VDDM_2V5 #PWR0148
+L VDDM_2V5 #PWR0157
 U 1 1 4BC94F2D
 P 4300 7300
-F 0 "#PWR0148" H 4300 7400 30  0001 C CNN
+F 0 "#PWR0157" H 4300 7400 30  0001 C CNN
 F 1 "VDDM_2V5" V 4300 7500 30  0000 C CNN
 	1    4300 7300
@@
 $EndComp
 $Comp
-L VDDM_2V5 #PWR0149
+L VDDM_2V5 #PWR0158
 U 1 1 4BC94F2C
 P 4200 7300
-F 0 "#PWR0149" H 4200 7400 30  0001 C CNN
+F 0 "#PWR0158" H 4200 7400 30  0001 C CNN
 F 1 "VDDM_2V5" V 4200 7500 30  0000 C CNN
 	1    4200 7300
@@
 $EndComp
 $Comp
-L VDDM_2V5 #PWR0150
+L VDDM_2V5 #PWR0159
 U 1 1 4BC94F1A
 P 4000 7300
-F 0 "#PWR0150" H 4000 7400 30  0001 C CNN
+F 0 "#PWR0159" H 4000 7400 30  0001 C CNN
 F 1 "VDDM_2V5" V 4000 7500 30  0000 C CNN
 	1    4000 7300
@@
 $EndComp
 $Comp
-L VDDM_2V5 #PWR0151
+L VDDM_2V5 #PWR0160
 U 1 1 4BC94F19
 P 4100 7300
-F 0 "#PWR0151" H 4100 7400 30  0001 C CNN
+F 0 "#PWR0160" H 4100 7400 30  0001 C CNN
 F 1 "VDDM_2V5" V 4100 7500 30  0000 C CNN
 	1    4100 7300
@@
 $EndComp
 $Comp
-L VDDM_2V5 #PWR0152
+L VDDM_2V5 #PWR0161
 U 1 1 4BC94F15
 P 3900 7300
-F 0 "#PWR0152" H 3900 7400 30  0001 C CNN
+F 0 "#PWR0161" H 3900 7400 30  0001 C CNN
 F 1 "VDDM_2V5" V 3900 7500 30  0000 C CNN
 	1    3900 7300
@@
 $EndComp
 $Comp
-L VDDM_2V5 #PWR0153
+L VDDM_2V5 #PWR0162
 U 1 1 4BC94EFD
 P 3800 7300
-F 0 "#PWR0153" H 3800 7400 30  0001 C CNN
+F 0 "#PWR0162" H 3800 7400 30  0001 C CNN
 F 1 "VDDM_2V5" V 3800 7500 30  0000 C CNN
 	1    3800 7300
@@
 EMI_DQS1
 $Comp
-L GND #PWR0154
+L GND #PWR0163
 U 1 1 4BC39D91
 P 8100 850
-F 0 "#PWR0154" H 8100 850 30  0001 C CNN
+F 0 "#PWR0163" H 8100 850 30  0001 C CNN
 F 1 "GND" H 8100 780 30  0001 C CNN
 	1    8100 850
@@
 PSWITCH
 $Comp
-L VDD5V #PWR0155
+L VDD5V #PWR0164
 U 1 1 4BBCE20A
 P 3950 1850
-F 0 "#PWR0155" H 3950 1950 30  0001 C CNN
+F 0 "#PWR0164" H 3950 1950 30  0001 C CNN
 F 1 "VDD5V" H 3950 1950 30  0000 C CNN
 	1    3950 1850
@@
 $EndComp
 $Comp
-L VDD_BATT #PWR0156
+L VDD_BATT #PWR0165
 U 1 1 4BBCCFD0
 P 2450 1850
-F 0 "#PWR0156" H 2450 1950 30  0001 C CNN
+F 0 "#PWR0165" H 2450 1950 30  0001 C CNN
 F 1 "VDD_BATT" H 2450 1950 30  0000 C CNN
 	1    2450 1850
@@
 $EndComp
 $Comp
-L VDD4V2 #PWR0157
+L VDD4V2 #PWR0166
 U 1 1 4BBCCFCF
 P 2700 1850
-F 0 "#PWR0157" H 2700 1950 30  0001 C CNN
+F 0 "#PWR0166" H 2700 1950 30  0001 C CNN
 F 1 "VDD4V2" H 2700 1950 30  0000 C CNN
 	1    2700 1850
@@
 $EndComp
 $Comp
-L VDDIO_3V3 #PWR0158
+L VDDIO_3V3 #PWR0167
 U 1 1 4BBCCFCE
 P 3200 1850
-F 0 "#PWR0158" H 3200 1950 30  0001 C CNN
+F 0 "#PWR0167" H 3200 1950 30  0001 C CNN
 F 1 "VDDIO_3V3" H 3200 1950 30  0000 C CNN
 	1    3200 1850
@@
 $EndComp
 $Comp
-L VDDD #PWR0159
+L VDDD #PWR0168
 U 1 1 4BBCE206
 P 3450 1850
-F 0 "#PWR0159" H 3450 1950 30  0001 C CNN
+F 0 "#PWR0168" H 3450 1950 30  0001 C CNN
 F 1 "VDDD" H 3450 1950 30  0000 C CNN
 	1    3450 1850
@@
 $EndComp
 $Comp
-L VDDA #PWR0160
+L VDDA #PWR0169
 U 1 1 4BBCE205
 P 3750 1850
-F 0 "#PWR0160" H 3750 1950 30  0001 C CNN
+F 0 "#PWR0169" H 3750 1950 30  0001 C CNN
 F 1 "VDDA" H 3750 1950 30  0000 C CNN
 	1    3750 1850
@@
 $EndComp
 $Comp
-L VDD_XTAL #PWR0161
+L VDD_XTAL #PWR0170
 U 1 1 4BBCE204
 P 4200 1850
-F 0 "#PWR0161" H 4200 1950 30  0001 C CNN
+F 0 "#PWR0170" H 4200 1950 30  0001 C CNN
 F 1 "VDD_XTAL" H 4200 1950 30  0000 C CNN
 	1    4200 1850
@@
 $EndComp
 $Comp
-L VDDM_2V5 #PWR0162
+L VDDM_2V5 #PWR0171
 U 1 1 4BBCCFC9
 P 4550 1850
-F 0 "#PWR0162" H 4550 1950 30  0001 C CNN
+F 0 "#PWR0171" H 4550 1950 30  0001 C CNN
 F 1 "VDDM_2V5" H 4550 1950 30  0000 C CNN
 	1    4550 1850

Commit message: Updated PROpendous Project.  PCB layout is nearing completion.
Parts:
- added V329, V330, V331: VIA, symbol VIA
Connections:
- net labels added: GNDPWR, VBUS_HOST, VDD4P2
- net labels removed: VDD4V2
- wire segments 60 -> 85
Other:
- moved on the sheet: V308, V309, V310, V311, V312, V325, V326, V327, V328

Commit message: Updated layout.
Connections:
- net GND: now also V261.1 (Via), V262.1 (Via), V263.1 (Via), V264.1 (Via), V265.1 (Via), V266.1 (Via), V267.1 (Via), V268.1 (Via), V269.1 (Via), V270.1 (Via), V271.1 (Via), V272.1 (Via), V273.1 (Via), V274.1 (Via), V275.1 (Via), V276.1 (Via)
- net GPMI_D00-LCD_D8-SSP2_DATA0: now also V57.1 (Via), V59.1 (Via)
- net GPMI_D01-LCD_D9-SSP2_DATA1: now also V58.1 (Via), V60.1 (Via)
- net GPMI_WRn-SSP2_SCK: now also V55.1 (Via), V56.1 (Via)
- net LCD_D04: now also V53.1 (Via)
- net LCD_D05: now also V54.1 (Via)
- net VDDD: now also V305.1 (Via), V306.1 (Via), V307.1 (Via)
Other:
- moved on the sheet: V151, V152, V153, V154, V155, V156, V157, V158, V159, V160, V161, V162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

Commit message: Updated layout.  Extended expansion connector and moved microSD.
Connections:
- net GPMI_D00-LCD_D8-SSP2_DATA0: no longer V57.1 (Via), V59.1 (Via)
- net GPMI_D01-LCD_D9-SSP2_DATA1: no longer V58.1 (Via), V60.1 (Via)
- net GPMI_RDY1-SSP2_CMD: now also V57.1 (Via), V58.1 (Via)
Changed lines of the file:
@@
-EESchema Schematic File Version 2  date 25/04/2010 06:05:24
+EESchema Schematic File Version 2  date 25/04/2010 07:03:32
 LIBS:opendous
 LIBS:device
@@
 Comment4 "www.PROpendous.org"
 $EndDescr
-Text GLabel 2850 2750 0    40   BiDi ~ 0
+Text GLabel 2850 2650 0    40   BiDi ~ 0
+GPMI_RDY1-SSP2_CMD
+Text GLabel 11100 2500 0    40   BiDi ~ 0
 GPMI_D00-LCD_D8-SSP2_DATA0
-Text GLabel 2850 2850 0    40   BiDi ~ 0
+Text GLabel 11100 2600 0    40   BiDi ~ 0
 GPMI_D01-LCD_D9-SSP2_DATA1
-Text GLabel 2850 2650 0    40   BiDi ~ 0
+Text GLabel 11100 2400 0    40   BiDi ~ 0
 GPMI_D01-LCD_D9-SSP2_DATA1
-Text GLabel 2850 2550 0    40   BiDi ~ 0
+Text GLabel 11100 2300 0    40   BiDi ~ 0
 GPMI_D00-LCD_D8-SSP2_DATA0
 Wire Wire Line
@@
 Text GLabel 9600 2550 0    40   BiDi ~ 0
 LCD_ENABLE-I2C_SCL
-Text GLabel 9600 4550 0    40   BiDi ~ 0
+Text GLabel 2850 2550 0    40   BiDi ~ 0
 GPMI_RDY1-SSP2_CMD
 Text GLabel 9600 4350 0    40   BiDi ~ 0
