File: PRopendous/Hardware/PROpendous/PROpendous-Vias.sch (KiCad schematic (older format))
At the start: 265 parts

Commit message: Updated i.MX233-based PROpendous board with EEPROM to fix Freescale Errata #2229.
Parts:
- added V167, V168, V170, V171, V172: VIA, symbol VIA
Connections:
- net I2C_SCL-GPMI_RDY2-AUART1_TX: now also V168.1 (Via)
- net I2C_SDA-GPMI_CE2n-AUART1_RX: now also V167.1 (Via), V171.1 (Via)
- net VDDIO_3V3: now also V170.1 (Via)
- new net EEPROM_WP: V172.1 (Via)

Commit message: Updated design files.  Added picture of finished PCB.
Parts:
- added V331: VIA, symbol VIA
Connections:
- net GND: now also V331.1 (Via)

Commit message: Updated PROpendous design and manufacturing files.
Parts:
- added V332, V333, V334, V335, V336: VIA, symbol VIA
Connections:
- net GND: now also V332.1 (Via), V333.1 (Via), V334.1 (Via), V335.1 (Via), V336.1 (Via)

Commit message: Updated the design.  JTAG header now includes VDD_XTAL and SSP1_Detect.  1.8" LCD has been removed and LCD backlight control is now connected to GPMI_CE1n.  The clock signals for the DDR SDRAM are now the longest EMI traces at 0.76".
Parts:
- added V337, V338, V339, V340, V341, V342, V343, V344, V345: VIA, symbol VIA
Connections:
- net GND: now also V339.1 (Via), V340.1 (Via), V341.1 (Via), V342.1 (Via), V343.1 (Via), V344.1 (Via)
- net LCD_RD: now also V345.1 (Via)
- net PWM2-GPMI_RDY3: no longer V47.1 (Via), V92.1 (Via)
- new net FSUSB20_S: V47.1 (Via), V92.1 (Via)
- new net GPMI_CE1n: V337.1 (Via), V338.1 (Via)
