File: PRopendous/Hardware/PROpendous/PROpendous-Vias.sch (KiCad schematic (older format))
At the start: 285 parts

Commit message: Updated PROpendous design with minor correction to silkscreen and two more bypass capacitors for the microSD connector.  Also added Buttons Module design files.
Parts:
- added V346, V347: VIA, symbol VIA
Connections:
- net GND: now also V347.1 (Via)
- net VDDIO_3V3: now also V346.1 (Via)

Commit message: Updated PROpendous design.  PWM2-GPMI_RDY3 now controls the LCD backlight and GPMI_CE1n now controls USB Host enable.  The function of these pins was switched as PWM2 makes more sense as a backlight control.
Parts:
- added V348, V349, V350, V351: VIA, symbol VIA
Connections:
- net FSUSB20_S: now also V348.1 (Via)
- net GND: now also V350.1 (Via), V351.1 (Via)
- net GPMI_CE1n: now also V349.1 (Via)
