File: PRopendous/Hardware/PROpendous/PROpendous-iMX233.sch (KiCad schematic (older format))
At the start: 1 part

Commit message: Updated files.  DDR SDRAM schematic completed.
Parts:
- removed IC?: IMX233, symbol IMX233
- added C1, C2: 10pF, symbol C_MINI
- added C3, C4: 0.1uF, symbol C_MINI
- added C5: 1uF, symbol C_MINI
- added ENCLOSURE_HAMMOND_1553B_1, TP1: CONN_1, symbol CONN_1
- added IC1: i.MX233, symbol IMX233
- added L1: 15uH, symbol L_MINI
- added R1, R2: 1k, symbol R_MINI
- added R3: 100k, symbol R_MINI
- added R6: 10k, symbol R_MINI
- added SW1: POWER, symbol SWITCH_PUSHBUTTON
- added X1: 24MHz, symbol CRYSTAL
Connections:
- net labels added: GND, GND1, GNDPWR, HP_VGND, VDD4V2, VDD5V, VDDA, VDDD, VDDIO_3V3, VDDM_2V5, VDD_BATT, VDD_XTAL
- wire segments 0 -> 40
Other:
- note added: "C0G"
- note added: "Connecting TP1 to VDDIO_3.3V\nduring ROM boot will start\n'USB Firmware Recovery' mode"
- note added: "GND1 must route to\nstar ground at VSSA2"
- note added: "Global-Local labels are used to\nforce proper net names in pcbnew"
- note added: "X5R"
- note removed: "Global-Local labels are used\nto force net names in pcbnew"

Commit message: Updated PROpendous i.MX233 project.  DDR SDRAM layout is complete.
Connections:
- wire segments 40 -> 42
Changed lines of the file:
@@
-EESchema Schematic File Version 2  date 07/04/2010 20:14:10
+EESchema Schematic File Version 2  date 17/04/2010 17:25:37
 LIBS:opendous
 LIBS:device
@@
 EELAYER END
 $Descr A4 11700 8267
-Sheet 2 6
+Sheet 2 7
 Title "PROpendous"
-Date "8 apr 2010"
+Date "17 apr 2010"
 Rev "1.0"
 Comp "Opendous Inc. (www.opendous.org)"
@@
 Comment4 "www.PROpendous.org"
 $EndDescr
+Connection ~ 5100 950
+Wire Wire Line
+	5100 700  5100 950
+Connection ~ 4700 950
+Wire Wire Line
+	4600 950  4900 950
+Wire Wire Line
+	4550 7350 4550 7250
+Connection ~ 4150 7250
+Wire Wire Line
+	4250 7250 3650 7250
+Connection ~ 3900 7250
+Connection ~ 1300 1500
+Wire Wire Line
+	1300 1700 1300 1500
+Connection ~ 1100 1500
+Wire Wire Line
+	650  1350 650  1500
+Connection ~ 1200 2050
+Wire Wire Line
+	1100 2050 1300 2050
+Wire Wire Line
+	1300 2050 1300 1900
+Wire Wire Line
+	650  1500 750  1500
+Wire Wire Line
+	650  1850 650  1800
+Wire Wire Line
+	5850 7000 5850 7100
+Connection ~ 1900 900
+Wire Wire Line
+	2200 1200 1900 1200
+Wire Wire Line
+	1900 1200 1900 750
+Wire Wire Line
+	1900 550  1300 550
+Wire Wire Line
+	4300 700  4300 950
+Connection ~ 3800 950
+Wire Wire Line
+	3900 950  3700 950
+Connection ~ 4100 950
+Wire Wire Line
+	4100 700  4100 950
+Wire Wire Line
+	3400 900  3400 950
+Wire Wire Line
+	3050 950  3050 700
+Wire Wire Line
+	2800 700  2800 950
+Wire Wire Line
+	2800 950  2900 950
+Connection ~ 2800 950
+Wire Wire Line
+	3200 900  3200 950
+Wire Wire Line
+	4150 950  4050 950
+Wire Wire Line
+	3800 700  3800 950
+Wire Wire Line
+	3550 950  3550 700
+Wire Wire Line
+	4450 850  4450 950
+Wire Wire Line
+	1600 600  1600 550
+Connection ~ 1600 550
+Wire Wire Line
+	1300 750  1300 1300
+Wire Wire Line
+	1300 1300 2200 1300
+Connection ~ 1300 900
+Wire Wire Line
+	5700 6700 5850 6700
+Wire Wire Line
+	5850 6700 5850 6800
+Wire Wire Line
+	650  2100 650  2050
+Wire Wire Line
+	1200 2100 1200 2050
+Wire Wire Line
+	1100 1850 1100 1750
+Wire Wire Line
+	1550 1500 2200 1500
+Wire Wire Line
+	1050 1500 1350 1500
+Wire Wire Line
+	1100 1550 1100 1450
+Wire Wire Line
+	1100 1250 1100 1200
+Connection ~ 3800 7250
+Connection ~ 4000 7250
+Wire Wire Line
+	3950 7250 3950 7350
+Connection ~ 3950 7250
 Wire Wire Line
 	7350 6300 7350 6250
-Connection ~ 3950 7250
-Wire Wire Line
-	3950 7350 3950 7250
-Connection ~ 4000 7250
-Connection ~ 3800 7250
-Wire Wire Line
-	1100 1250 1100 1200
-Wire Wire Line
-	1100 1550 1100 1450
-Wire Wire Line
-	1050 1500 1350 1500
-Wire Wire Line
-	1550 1500 2200 1500
-Wire Wire Line
-	1100 1850 1100 1750
-Wire Wire Line
-	1200 2100 1200 2050
-Wire Wire Line
-	650  2100 650  2050
-Connection ~ 4850 950
-Wire Wire Line
-	4850 950  4850 700
-Wire Wire Line
-	5850 6800 5850 6700
-Wire Wire Line
-	5850 6700 5700 6700
-Connection ~ 1300 900
-Wire Wire Line
-	2200 1300 1300 1300
-Wire Wire Line
-	1300 1300 1300 750
-Connection ~ 1600 550
-Wire Wire Line
-	1600 600  1600 550
-Wire Wire Line
-	4450 850  4450 950
-Wire Wire Line
-	3550 950  3550 700
-Wire Wire Line
-	3800 700  3800 950
-Wire Wire Line
-	4150 950  4050 950
-Connection ~ 5000 950
-Wire Wire Line
-	4600 950  5100 950
+Wire Wire Line
+	5050 950  5150 950
 Connection ~ 4800 950
 Wire Wire Line
-	3200 900  3200 950
-Connection ~ 2800 950
-Wire Wire Line
-	2900 950  2800 950
-Wire Wire Line
-	2800 950  2800 700
-Wire Wire Line
-	3050 950  3050 700
-Wire Wire Line
-	3400 900  3400 950
-Connection ~ 4700 950
-Connection ~ 4900 950
-Wire Wire Line
-	4100 700  4100 950
-Connection ~ 4100 950
-Wire Wire Line
-	3900 950  3700 950
-Connection ~ 3800 950
-Wire Wire Line
-	4300 700  4300 950
-Wire Wire Line
-	1900 550  1300 550
-Wire Wire Line
-	1900 750  1900 1200
-Wire Wire Line
-	1900 1200 2200 1200
-Connection ~ 1900 900
-Wire Wire Line
-	5850 7000 5850 7100
-Wire Wire Line
-	650  1850 650  1800
-Wire Wire Line
-	750  1500 650  1500
-Wire Wire Line
-	1300 1900 1300 2050
-Wire Wire Line
-	1300 2050 1100 2050
-Connection ~ 1200 2050
-Wire Wire Line
-	650  1500 650  1350
-Connection ~ 1100 1500
-Wire Wire Line
-	1300 1700 1300 1500
-Connection ~ 1300 1500
-Connection ~ 3900 7250
-Wire Wire Line
-	4250 7250 3650 7250
-Connection ~ 4150 7250
-Wire Wire Line
-	4550 7350 4550 7250
-$Comp
-L GNDPWR #PWR01
+	4750 700  4750 950
+Connection ~ 4750 950
+$Comp
+L VDDIO_3V3 #PWR01
+U 1 1 4BC3A9DE
+P 5100 700
+F 0 "#PWR01" H 5100 800 30  0001 C CNN
+F 1 "VDDIO_3V3" H 5100 800 30  0000 C CNN
+	1    5100 700
+	1    0    0    -1
+$EndComp
+$Comp
+L GNDPWR #PWR02
 U 1 1 4BBD1ABB
 P 7350 6300
-F 0 "#PWR01" H 7350 6350 40  0001 C CNN
+F 0 "#PWR02" H 7350 6350 40  0001 C CNN
 F 1 "GNDPWR" H 7350 6240 25  0000 C CNN
 	1    7350 6300
@@
 $EndComp
 $Comp
-L HP_VGND #PWR02
+L HP_VGND #PWR03
 U 1 1 4BBCE7B9
 P 4550 7350
-F 0 "#PWR02" H 4550 7350 30  0001 C CNN
+F 0 "#PWR03" H 4550 7350 30  0001 C CNN
 F 1 "HP_VGND" H 4550 7280 30  0000 C CNN
 	1    4550 7350
@@
 PSWITCH
 $Comp
-L GND #PWR03
+L GND #PWR04
 U 1 1 4BBCDC88
 P 1200 2100
-F 0 "#PWR03" H 1200 2100 30  0001 C CNN
+F 0 "#PWR04" H 1200 2100 30  0001 C CNN
 F 1 "GND" H 1200 2030 30  0001 C CNN
 	1    1200 2100
@@
 $EndComp
 $Comp
-L VDD_XTAL #PWR04
+L VDD_XTAL #PWR05
 U 1 1 4BBCDC06
 P 650 1350
-F 0 "#PWR04" H 650 1450 30  0001 C CNN
+F 0 "#PWR05" H 650 1450 30  0001 C CNN
 F 1 "VDD_XTAL" H 650 1450 30  0000 C CNN
 	1    650  1350
@@
 $EndComp
 $Comp
-L GND #PWR05
+L GND #PWR06
 U 1 1 4BBCDB43
 P 650 2100
-F 0 "#PWR05" H 650 2100 30  0001 C CNN
+F 0 "#PWR06" H 650 2100 30  0001 C CNN
 F 1 "GND" H 650 2030 30  0001 C CNN
 	1    650  2100
@@
 $EndComp
 $Comp
-L VDD_XTAL #PWR06
+L VDD_XTAL #PWR07
 U 1 1 4BBCDB1B
 P 650 1800
-F 0 "#PWR06" H 650 1900 30  0001 C CNN
+F 0 "#PWR07" H 650 1900 30  0001 C CNN
 F 1 "VDD_XTAL" H 650 1900 30  0000 C CNN
 	1    650  1800
@@
 $EndComp
 $Comp
-L VDD5V #PWR07
+L VDD5V #PWR08
 U 1 1 4BBCD826
 P 4300 700
-F 0 "#PWR07" H 4300 800 30  0001 C CNN
+F 0 "#PWR08" H 4300 800 30  0001 C CNN
 F 1 "VDD5V" H 4300 800 30  0000 C CNN
 	1    4300 700
@@
 $EndComp
 $Comp
-L GND #PWR08
+L GND #PWR09
 U 1 1 4BBCD031
 P 3950 7350
-F 0 "#PWR08" H 3950 7350 30  0001 C CNN
+F 0 "#PWR09" H 3950 7350 30  0001 C CNN
 F 1 "GND" H 3950 7280 30  0001 C CNN
 	1    3950 7350
@@
 $EndComp
 $Comp
-L GND #PWR09
+L GND #PWR010
 U 1 1 4BBCCF65
 P 1600 600
-F 0 "#PWR09" H 1600 600 30  0001 C CNN
+F 0 "#PWR010" H 1600 600 30  0001 C CNN
 F 1 "GND" H 1600 530 30  0001 C CNN
 	1    1600 600
@@
 GND1 must route to\nstar ground at VSSA2
 $Comp
-L GND1 #PWR010
+L GND1 #PWR011
 U 1 1 4BBCCEB7
 P 5850 7100
-F 0 "#PWR010" H 5850 7100 30  0001 C CNN
+F 0 "#PWR011" H 5850 7100 30  0001 C CNN
 F 1 "GND1" H 5850 7030 30  0000 C CNN
 	1    5850 7100
@@
 $EndComp
 $Comp
-L VDDM_2V5 #PWR011
+L VDDM_2V5 #PWR012
 U 1 1 4BBCCC9E
-P 4850 700
-F 0 "#PWR011" H 4850 800 30  0001 C CNN
-F 1 "VDDM_2V5" H 4850 800 30  0000 C CNN
-	1    4850 700
-	1    0    0    -1
-$EndComp
-$Comp
-L VDD_XTAL #PWR012
+P 4750 700
+F 0 "#PWR012" H 4750 800 30  0001 C CNN
+F 1 "VDDM_2V5" H 4750 800 30  0000 C CNN
+	1    4750 700
+	1    0    0    -1
+$EndComp
+$Comp
+L VDD_XTAL #PWR013
 U 1 1 4BBCCC78
 P 4450 850
-F 0 "#PWR012" H 4450 950 30  0001 C CNN
+F 0 "#PWR013" H 4450 950 30  0001 C CNN
 F 1 "VDD_XTAL" H 4450 950 30  0000 C CNN
 	1    4450 850
@@
 $EndComp
 $Comp
-L VDDA #PWR013
+L VDDA #PWR014
 U 1 1 4BBCCB4A
 P 4100 700
-F 0 "#PWR013" H 4100 800 30  0001 C CNN
+F 0 "#PWR014" H 4100 800 30  0001 C CNN
 F 1 "VDDA" H 4100 800 30  0000 C CNN
 	1    4100 700
@@
 $EndComp
 $Comp
-L VDDD #PWR014
+L VDDD #PWR015
 U 1 1 4BBCCB16
 P 3800 700
-F 0 "#PWR014" H 3800 800 30  0001 C CNN
+F 0 "#PWR015" H 3800 800 30  0001 C CNN
 F 1 "VDDD" H 3800 800 30  0000 C CNN
 	1    3800 700
@@
 $EndComp
 $Comp
-L VDDIO_3V3 #PWR015
+L VDDIO_3V3 #PWR016
 U 1 1 4BBCC974
 P 3550 700
-F 0 "#PWR015" H 3550 800 30  0001 C CNN
+F 0 "#PWR016" H 3550 800 30  0001 C CNN
 F 1 "VDDIO_3V3" H 3550 800 30  0000 C CNN
 	1    3550 700
@@
 $EndComp
 $Comp
-L VDD4V2 #PWR016
+L VDD4V2 #PWR017
 U 1 1 4BBCC950
 P 3050 700
-F 0 "#PWR016" H 3050 800 30  0001 C CNN
+F 0 "#PWR017" H 3050 800 30  0001 C CNN
 F 1 "VDD4V2" H 3050 800 30  0000 C CNN
 	1    3050 700
@@
 $EndComp
 $Comp
-L VDD_BATT #PWR017
+L VDD_BATT #PWR018
 U 1 1 4BBCC942
 P 2800 700
-F 0 "#PWR017" H 2800 800 30  0001 C CNN
+F 0 "#PWR018" H 2800 800 30  0001 C CNN
 F 1 "VDD_BATT" H 2800 800 30  0000 C CNN
 	1    2800 700

Commit message: Updated PROpendous project.  Schematic is complete but not yet finalized.  Layout partially complete.
Parts:
- added L14, L2: FB, symbol L_MINI
Connections:
- net labels added: TSC_IN1, TSC_IN2, TSC_VBAT1, TSC_VBAT2, TSC_VREF
- wire segments 42 -> 50
Other:
- note added: "Use GNDPWR for chassis\nground ring to suppress EMI"
- moved on the sheet: ENCLOSURE_HAMMOND_1553B_1
Changed lines of the file:
@@
-EESchema Schematic File Version 2  date 17/04/2010 17:25:37
+EESchema Schematic File Version 2  date 19/04/2010 19:59:31
 LIBS:opendous
 LIBS:device
@@
 EELAYER END
 $Descr A4 11700 8267
-Sheet 2 7
+Sheet 2 8
 Title "PROpendous"
-Date "17 apr 2010"
+Date "19 apr 2010"
 Rev "1.0"
 Comp "Opendous Inc. (www.opendous.org)"
@@
 Comment4 "www.PROpendous.org"
 $EndDescr
+$Comp
+L L_MINI L14
+U 1 1 4BCCECEA
+P 6300 7450
+F 0 "L14" H 6225 7400 30  0000 C CNN
+F 1 "FB" H 6350 7400 22  0000 C CNN
+	1    6300 7450
+	-1   0    0    1
+$EndComp
+$Comp
+L GND #PWR01
+U 1 1 4BCCECE8
+P 6450 7500
+F 0 "#PWR01" H 6450 7500 30  0001 C CNN
+F 1 "GND" H 6450 7430 30  0001 C CNN
+	1    6450 7500
+	1    0    0    -1
+$EndComp
+Wire Wire Line
+	6450 7500 6450 7450
+Wire Wire Line
+	6450 7450 6400 7450
+Wire Wire Line
+	6200 7450 6150 7450
+Wire Wire Line
+	6150 7450 6150 7500
+$Comp
+L GND1 #PWR02
+U 1 1 4BCCECDD
+P 6150 7500
+F 0 "#PWR02" H 6150 7500 30  0001 C CNN
+F 1 "GND1" H 6150 7430 30  0000 C CNN
+	1    6150 7500
+	1    0    0    -1
+$EndComp
+$Comp
+L IMX233 IC1
+U 1 1 4BCC6F47
+P 3950 4100
+F 0 "IC1" H 2450 1050 60  0000 C CNN
+F 1 "i.MX233" H 2525 7150 60  0000 C CNN
+	1    3950 4100
+	1    0    0    -1
+$EndComp
+Text Label 9900 2100 2    40   ~ 0
+TSC_VREF
+Text Label 9900 2200 2    40   ~ 0
+TSC_VBAT1
+Text Label 9900 2300 2    40   ~ 0
+TSC_VBAT2
+Text Label 9900 2000 2    40   ~ 0
+TSC_IN2
+Text Label 9900 1900 2    40   ~ 0
+TSC_IN1
+Text Notes 6800 6300 0    50   ~ 0
+Use GNDPWR for chassis\nground ring to suppress EMI
+Wire Wire Line
+	7200 6100 7200 6050
+Wire Wire Line
+	7200 6050 7250 6050
 Connection ~ 5100 950
 Wire Wire Line
@@
 Connection ~ 4700 950
 Wire Wire Line
-	4600 950  4900 950
+	4900 950  4600 950
 Wire Wire Line
 	4550 7350 4550 7250
 Connection ~ 4150 7250
 Wire Wire Line
-	4250 7250 3650 7250
+	3650 7250 4250 7250
 Connection ~ 3900 7250
 Connection ~ 1300 1500
@@
 	1900 1200 1900 750
 Wire Wire Line
-	1900 550  1300 550
+	1300 550  1900 550
 Wire Wire Line
 	4300 700  4300 950
 Connection ~ 3800 950
 Wire Wire Line
-	3900 950  3700 950
+	3700 950  3900 950
 Connection ~ 4100 950
 Wire Wire Line
@@
 	3200 900  3200 950
 Wire Wire Line
-	4150 950  4050 950
+	4050 950  4150 950
 Wire Wire Line
 	3800 700  3800 950
@@
 	1550 1500 2200 1500
 Wire Wire Line
-	1050 1500 1350 1500
-Wire Wire Line
-	1100 1550 1100 1450
+	1350 1500 1050 1500
+Wire Wire Line
+	1100 1450 1100 1550
 Wire Wire Line
 	1100 1250 1100 1200
@@
 Connection ~ 3950 7250
 Wire Wire Line
-	7350 6300 7350 6250
-Wire Wire Line
-	5050 950  5150 950
+	7350 5750 7350 5700
+Wire Wire Line
+	5150 950  5050 950
 Connection ~ 4800 950
 Wire Wire Line
-	4750 700  4750 950
+	4750 950  4750 700
 Connection ~ 4750 950
-$Comp
-L VDDIO_3V3 #PWR01
+Wire Wire Line
+	7450 6050 7500 6050
+Wire Wire Line
+	7500 6050 7500 6100
+$Comp
+L GND #PWR03
+U 1 1 4BCC48BC
+P 7500 6100
+F 0 "#PWR03" H 7500 6100 30  0001 C CNN
+F 1 "GND" H 7500 6030 30  0001 C CNN
+	1    7500 6100
+	1    0    0    -1
+$EndComp
+$Comp
+L GNDPWR #PWR04
+U 1 1 4BCC48B6
+P 7200 6100
+F 0 "#PWR04" H 7200 6150 40  0001 C CNN
+F 1 "GNDPWR" H 7200 6040 25  0000 C CNN
+	1    7200 6100
+	1    0    0    -1
+$EndComp
+$Comp
+L L_MINI L2
+U 1 1 4BCC48AC
+P 7350 6050
+F 0 "L2" H 7275 6000 30  0000 C CNN
+F 1 "FB" H 7400 6000 22  0000 C CNN
+	1    7350 6050
+	-1   0    0    1
+$EndComp
+$Comp
+L VDDIO_3V3 #PWR05
 U 1 1 4BC3A9DE
 P 5100 700
-F 0 "#PWR01" H 5100 800 30  0001 C CNN
+F 0 "#PWR05" H 5100 800 30  0001 C CNN
 F 1 "VDDIO_3V3" H 5100 800 30  0000 C CNN
 	1    5100 700
@@
 $EndComp
 $Comp
-L GNDPWR #PWR02
+L GNDPWR #PWR06
 U 1 1 4BBD1ABB
-P 7350 6300
-F 0 "#PWR02" H 7350 6350 40  0001 C CNN
-F 1 "GNDPWR" H 7350 6240 25  0000 C CNN
-	1    7350 6300
+P 7350 5750
+F 0 "#PWR06" H 7350 5800 40  0001 C CNN
+F 1 "GNDPWR" H 7350 5690 25  0000 C CNN
+	1    7350 5750
 	1    0    0    -1
 $EndComp
@@
 L CONN_1 ENCLOSURE_HAMMOND_1553B_1
 U 1 1 4BBD1A8C
-P 7350 6100
-F 0 "ENCLOSURE_HAMMOND_1553B_1" V 7430 6100 40  0000 L CNN
-F 1 "CONN_1" H 7350 6155 30  0001 C CNN
-	1    7350 6100
+P 7350 5550
+F 0 "ENCLOSURE_HAMMOND_1553B_1" V 7430 5550 40  0000 L CNN
+F 1 "CONN_1" H 7350 5605 30  0001 C CNN
+	1    7350 5550
 	0    -1   -1   0
 $EndComp
 $Comp
-L HP_VGND #PWR03
+L HP_VGND #PWR07
 U 1 1 4BBCE7B9
 P 4550 7350
-F 0 "#PWR03" H 4550 7350 30  0001 C CNN
+F 0 "#PWR07" H 4550 7350 30  0001 C CNN
 F 1 "HP_VGND" H 4550 7280 30  0000 C CNN
 	1    4550 7350
@@
 Text Notes 700  1975 0    30   ~ 0
 X5R
-$Comp
-L IMX233 IC1
-U 1 1 4BBCE5E2
-P 3950 4100
-F 0 "IC1" H 2450 1050 60  0000 C CNN
-F 1 "i.MX233" H 2525 7150 60  0000 C CNN
-	1    3950 4100
-	1    0    0    -1
-$EndComp
 Text Notes 500  800  0    30   ~ 0
 Connecting TP1 to VDDIO_3.3V\nduring ROM boot will start\n'USB Firmware Recovery' mode
@@
 PSWITCH
 $Comp
-L GND #PWR04
+L GND #PWR08
 U 1 1 4BBCDC88
 P 1200 2100
-F 0 "#PWR04" H 1200 2100 30  0001 C CNN
+F 0 "#PWR08" H 1200 2100 30  0001 C CNN
 F 1 "GND" H 1200 2030 30  0001 C CNN
 	1    1200 2100
@@
 $EndComp
 $Comp
-L VDD_XTAL #PWR05
+L VDD_XTAL #PWR09
 U 1 1 4BBCDC06
 P 650 1350
-F 0 "#PWR05" H 650 1450 30  0001 C CNN
+F 0 "#PWR09" H 650 1450 30  0001 C CNN
 F 1 "VDD_XTAL" H 650 1450 30  0000 C CNN
 	1    650  1350
@@
 $EndComp
 $Comp
-L GND #PWR06
+L GND #PWR010
 U 1 1 4BBCDB43
 P 650 2100
-F 0 "#PWR06" H 650 2100 30  0001 C CNN
+F 0 "#PWR010" H 650 2100 30  0001 C CNN
 F 1 "GND" H 650 2030 30  0001 C CNN
 	1    650  2100
@@
 $EndComp
 $Comp
-L VDD_XTAL #PWR07
+L VDD_XTAL #PWR011
 U 1 1 4BBCDB1B
 P 650 1800
-F 0 "#PWR07" H 650 1900 30  0001 C CNN
+F 0 "#PWR011" H 650 1900 30  0001 C CNN
 F 1 "VDD_XTAL" H 650 1900 30  0000 C CNN
 	1    650  1800
@@
 $EndComp
 $Comp
-L VDD5V #PWR08
+L VDD5V #PWR012
 U 1 1 4BBCD826
 P 4300 700
-F 0 "#PWR08" H 4300 800 30  0001 C CNN
+F 0 "#PWR012" H 4300 800 30  0001 C CNN
 F 1 "VDD5V" H 4300 800 30  0000 C CNN
 	1    4300 700
@@
 $EndComp
 $Comp
-L GND #PWR09
+L GND #PWR013
 U 1 1 4BBCD031
 P 3950 7350
-F 0 "#PWR09" H 3950 7350 30  0001 C CNN
+F 0 "#PWR013" H 3950 7350 30  0001 C CNN
 F 1 "GND" H 3950 7280 30  0001 C CNN
 	1    3950 7350
@@
 $EndComp
 $Comp
-L GND #PWR010
+L GND #PWR014
 U 1 1 4BBCCF65
 P 1600 600
-F 0 "#PWR010" H 1600 600 30  0001 C CNN
+F 0 "#PWR014" H 1600 600 30  0001 C CNN
 F 1 "GND" H 1600 530 30  0001 C CNN
 	1    1600 600
@@
 GND1 must route to\nstar ground at VSSA2
 $Comp
-L GND1 #PWR011
+L GND1 #PWR015
 U 1 1 4BBCCEB7
 P 5850 7100
-F 0 "#PWR011" H 5850 7100 30  0001 C CNN
+F 0 "#PWR015" H 5850 7100 30  0001 C CNN
 F 1 "GND1" H 5850 7030 30  0000 C CNN
 	1    5850 7100
@@
 $EndComp
 $Comp
-L VDDM_2V5 #PWR012
+L VDDM_2V5 #PWR016
 U 1 1 4BBCCC9E
 P 4750 700
-F 0 "#PWR012" H 4750 800 30  0001 C CNN
+F 0 "#PWR016" H 4750 800 30  0001 C CNN
 F 1 "VDDM_2V5" H 4750 800 30  0000 C CNN
 	1    4750 700
@@
 $EndComp
 $Comp
-L VDD_XTAL #PWR013
+L VDD_XTAL #PWR017
 U 1 1 4BBCCC78
 P 4450 850
-F 0 "#PWR013" H 4450 950 30  0001 C CNN
+F 0 "#PWR017" H 4450 950 30  0001 C CNN
 F 1 "VDD_XTAL" H 4450 950 30  0000 C CNN
 	1    4450 850
@@
 $EndComp
 $Comp
-L VDDA #PWR014
+L VDDA #PWR018
 U 1 1 4BBCCB4A
 P 4100 700
-F 0 "#PWR014" H 4100 800 30  0001 C CNN
+F 0 "#PWR018" H 4100 800 30  0001 C CNN
 F 1 "VDDA" H 4100 800 30  0000 C CNN
 	1    4100 700
@@
 $EndComp
 $Comp
-L VDDD #PWR015
+L VDDD #PWR019
 U 1 1 4BBCCB16
 P 3800 700
-F 0 "#PWR015" H 3800 800 30  0001 C CNN
+F 0 "#PWR019" H 3800 800 30  0001 C CNN
 F 1 "VDDD" H 3800 800 30  0000 C CNN
 	1    3800 700
@@
 $EndComp
 $Comp
-L VDDIO_3V3 #PWR016
+L VDDIO_3V3 #PWR020
 U 1 1 4BBCC974
 P 3550 700
-F 0 "#PWR016" H 3550 800 30  0001 C CNN
+F 0 "#PWR020" H 3550 800 30  0001 C CNN
 F 1 "VDDIO_3V3" H 3550 800 30  0000 C CNN
 	1    3550 700
@@
 $EndComp
 $Comp
-L VDD4V2 #PWR017
+L VDD4V2 #PWR021
 U 1 1 4BBCC950
 P 3050 700
-F 0 "#PWR017" H 3050 800 30  0001 C CNN
+F 0 "#PWR021" H 3050 800 30  0001 C CNN
 F 1 "VDD4V2" H 3050 800 30  0000 C CNN
 	1    3050 700
@@
 $EndComp
 $Comp
-L VDD_BATT #PWR018
+L VDD_BATT #PWR022
 U 1 1 4BBCC942
 P 2800 700
-F 0 "#PWR018" H 2800 800 30  0001 C CNN
+F 0 "#PWR022" H 2800 800 30  0001 C CNN
 F 1 "VDD_BATT" H 2800 800 30  0000 C CNN
 	1    2800 700
@@
 Text GLabel 9050 1550 2    40   BiDi ~ 0
 PSWITCH
+Text GLabel 9900 1900 2    40   BiDi ~ 0
+TSC_IN1
+Text GLabel 9900 2000 2    40   BiDi ~ 0
+TSC_IN2
+Text GLabel 9900 2200 2    40   BiDi ~ 0
+TSC_VBAT1
+Text GLabel 9900 2300 2    40   BiDi ~ 0
+TSC_VBAT2
+Text GLabel 9900 2100 2    40   BiDi ~ 0
+TSC_VREF
 $EndSCHEMATC
