File: PRopendous/Hardware/PROpendous/PROpendous-LCD.sch (KiCad schematic (older format))
At the start: 11 parts, among them Q1 2N7002, U1 NHD-2.4-240320SF-CTXI-T

Commit message: Updated PROpendous project.  Schematic is complete but not yet finalized.  Layout partially complete.
Parts:
- added C35: 0.1uF, symbol C_MINI
- added IC3: TSC2003, symbol TSC2003
- added R16, R19: 47k, symbol R_MINI
- added R17, R18: 1.2k, symbol R_MINI
- added U4: NHD-1.8-128160ZF-CTXL, symbol NHD-1.8-128160ZF-CTXL
- R12, R13, R14, R15: value 50 -> 5
Connections:
- net labels added: LCD_LED_K1, LCD_LED_K2, TSC_IN1, TSC_IN2, TSC_VBAT1, TSC_VBAT2, TSC_VREF, X+, X-, Y+, Y-
- net labels removed: DEBUG, EMI_A00, EMI_A01, EMI_A02, EMI_A03, EMI_A04, EMI_A05, EMI_A06, EMI_A07, EMI_A08, EMI_A09, EMI_A10, EMI_A11, EMI_A12, EMI_BA0, EMI_BA1, EMI_CASn, EMI_CE0n, EMI_CKE, EMI_CLK, EMI_CLKn, EMI_D00, EMI_D01, EMI_D02, EMI_D03, EMI_D04, EMI_D05, EMI_D06, EMI_D07, EMI_D08, EMI_D09, EMI_D10, EMI_D11, EMI_D12, EMI_D13, EMI_D14, EMI_D15, EMI_DQM0, EMI_DQM1, EMI_DQS0, EMI_DQS1, EMI_RASn, EMI_WEn, GPMI_ALE-LCD_D17, GPMI_CE0n, GPMI_CE1n, GPMI_CLE-LCD_D16, GPMI_D00-LCD_D8-SSP2_DATA0, GPMI_D01-LCD_D9-SSP2_DATA1, GPMI_D02-LCD_D10-SSP2_DATA2, GPMI_D03-LCD_D11-SSP2_DATA3, GPMI_D04-LCD_D12-SSP2_DATA4, GPMI_D05-LCD_D13-SSP2_DATA5, GPMI_D06-LCD_D14-SSP2_DATA6, GPMI_D07-LCD_D15-SSP2_DATA7, GPMI_RDY0-SSP2_DETECT, GPMI_RDY1-SSP2_CMD, GPMI_RDn, GPMI_WPn, GPMI_WRn-SSP2_SCK, HPL, HPR, LCD_DOTCK-GPMI_RDY3, LCD_ENABLE-I2C_SCL, LCD_HSYNC-I2C_SDA, LCD_VSYNC-LCD_BUSY, LINE1_INL, LINE1_INR, LRADC0, LRADC1, MIC, PSWITCH, PWM0-ROTARYA-DUART_RX, PWM1-ROTARYB-DUART_TX, PWM2-GPMI_RDY3, SSP1_CMD-JTAG_TDO, SSP1_DATA0-JTAG_TDI, SSP1_DATA1-I2C_SCL-JTAG_TCLK, SSP1_DATA2-I2C_SDA-JTAG_RTCK, SSP1_DATA3-JTAG_TMS, SSP1_DETECT-GPMI_CE3N-USB_ID, SSP1_SCK-JTAG_TRST, USB_DM, USB_DP, VAG, VDAC1, XTALI, XTALO
- wire segments 25 -> 61
- no-connect marks 11 -> 16
Other:
- note added: "1.8" TFT Color LCD"
- note added: "2.4" TFT Color LCD"
- note added: "Notes:\n - Capacitors can be any available 6.3V+\n - Populate only one of the 2.4" or 1.8" LCDs or neither\n - The 1.8" LCD footprint reuses signals from the 2.4" LCD footprint\n - 2.4" LCD can be either of:\n NHD-2.4-240320SF-CTXI-T which has a touchscreen\n NHD-2.4-240320SF-CTXI which does not have a touchscreen\n - TSC2003 Touchscreen controller is only required\n if populating the NHD-2.4-240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"
- note added: "Read Mode Unsupported Per IMX23RM 1.2.19.1 (Write=1)"
- note added: "TSC2003 Device Address is\n0b1001000 = 0x48 = 72"
- note removed: "Notes:\n - All capacitors are X7R, 6.3V, 20% or better unless otherwise noted"
- note removed: "Read Data Unnecessary"
- note removed: "TODO: Select Touch Screen Controller\n1st Choice: STMPE610 $1.50/100 I2C/SPI 12Bit-120kSPS-6CH-ADC, TSC+2GPIO, QFN\n2nd Choice: MSP430F2013 $2.00/100 I2C/SPI 16Bit-100kSPS-4CH-ADC, 2GPIO, TSSOP\n3rd Choice: ATtiny261 $1.50/100 I2C/SPI 10bit-15kSPS-10CH-ADC/GPIO, SOIC/QFN\n4th Choice: TSC2046 $2.15/100 SPI 12Bit-125kSPS-6CH-ADC, TSC, TSSOP/QFN\nOr, some microcontroller with at least 4 ADC inputs a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"
- moved on the sheet: C28, C29, C30, R11, R12, R13, R14, R15, TP2, U1

Commit message: Updated PROpendous Project.  PCB layout is nearing completion.
Connections:
- net labels added: SSP1_DETECT-GPMI_CE3N-USB_ID
- net labels removed: LCD_LED_ON
- wire segments 61 -> 64

Commit message: First revision of i.MX233-based PROpendous board is complete.
Parts:
- added C78: 33uF, symbol CP_TANTALUM_MINI
- added TP3, TP4, TP5, TP6, TP7, TP8: CONN_1, symbol CONN_1
Connections:
- net labels added: TSC_PENIRQ
- wire segments 64 -> 68
Other:
- moved on the sheet: C35
