File: PRopendous/Hardware/PROpendous/PROpendous-LCD.sch (KiCad schematic (older format))
At the start: 24 parts, among them IC3 TSC2007, Q1 2N7002, U1 NHD-2.4-240320SF-CTXI-T

Commit message: Updated PROpendous design.  PWM2-GPMI_RDY3 now controls the LCD backlight and GPMI_CE1n now controls USB Host enable.  The function of these pins was switched as PWM2 makes more sense as a backlight control.
Connections:
- net labels added: PWM2-GPMI_RDY3
- net labels removed: GPMI_CE1n
Changed lines of the file:
@@
-EESchema Schematic File Version 2  date 20/10/2010 05:47:04
+EESchema Schematic File Version 2  date 21/10/2010 09:30:50
 LIBS:opendous
 LIBS:device
@@
 Sheet 5 8
 Title "PROpendous"
-Date "20 oct 2010"
-Rev "1.0"
+Date "21 oct 2010"
+Rev "1.1"
 Comp "Opendous Inc. (www.opendous.org)"
 Comment1 ""
@@
 TSC_VBAT2
 Text GLabel 3900 3600 0    40   BiDi ~ 0
-GPMI_CE1n
+PWM2-GPMI_RDY3
 $Comp
 L VDDIO_3V3 #PWR070
