File: PRopendous/Hardware/PROpendous/PROpendous-Power_Boot.sch (KiCad schematic (older format))
At the start: 52 parts, among them IC6 LM2621

Commit message: Minor update to schematic.  Removed USB Power switch and added some notes.
Parts:
- added C36: 0.01uF, symbol C_MINI
- added C37: 68uF, symbol CP_TANTALUM_MINI
- added F1: 1206L, symbol FUSE-MINI
- added L4, L5: FB, symbol L_MINI
Connections:
- net labels added: GND_USB-B, VBUS
- wire segments 164 -> 173
Other:
- note added: "Littelfuse 1206L035"
- note added: "Power Supply Decoupling"
- moved on the sheet: C39, C40, IC6, L6, R24, R25, R26, R27, R28

Commit message: Updated PROpendous Project.  PCB layout is nearing completion.
Parts:
- removed BT1: BATTERY, symbol BATTERY
- added BT1: BATTERY, symbol CONN_3
- added C76: 0.01uF, symbol C_MINI
- added D3: USB_HOST, symbol D_LED
- added D4: POWERED, symbol D_LED
- added R46, R47: 200, symbol R_MINI
- added R48, R49: 100k, symbol R_MINI
- added R50, R51: 0, symbol R_MINI
- JP1: value 2mm Jumpers -> Boot Jumpers
Connections:
- net labels added: LM2621_Vdd, LRADC0, TSC_IN1, VDD4P2
- net labels removed: VDD4V2, VDDM_2V5
- wire segments 173 -> 183
Other:
- note added: "1%"
- note added: "2.85A Max"
- note added: "Battery Temperature Sense"
- note added: "CF1"
- note added: "Debug/Host Mode Enabled LED"
- note added: "Default Boot is SD/MMC2, the captive microSD card.\nJumpers can be mounted to alter the default setting.\nLCD_RS High enables jumper boot.\nLCD_RS Low enables OTP boot."
- note added: "Li-ION Battery"
- note added: "Notes:\n - Capacitors are X7R, 6.3V, 20% or better unless otherwise noted\n - Tantalum capacitors should have ESR < 300mOhm\n - VDDIO, VDDD, VDDA should have 33uF of decoupling and LPF >1MHz per IMX23RM 32.2.1.1\n - Power Supply Designed to Freescale AppNote AN3883 recommendations\n - The Connectors_JTAG sheet contains power selection circuitry as it is relevant to the USB connector"
- note added: "PWM2-GPMI_RDY3 also controls USB\nUSB Host enable to reduce the number\nof signals stuck on the board."
- note added: "Power ON LED"
- note added: "R50, R51 are copper\ntraces which can be cut"
- note added: "RF1"
- note added: "RF2"
- note added: "RFQ"
- note added: "The LQH6PP meets the 2.5A inductor current limit of the LM2621.\nIt also meets the typical (2.85A) internal current limit. However, it\ndoes not meet the maximum internal current limit of the LM2621 (4A)\nwhich can occur at high temperature during a short of USB-A VBUS+GND."
- note added: "USB-miniB VBUS supplies power for\nLi-Ion Battery charging as well\nas board power."
- note added: "muRata LQH6PP"
- note removed: "Default Boot is SD/MMC1, the captive microSD card.\nJumpers can be mounted to alter the default setting.\nLCD_RS High enables jumper boot.\nLCD_RS Low enables OTP boot."
- note removed: "Notes:\n - Capacitors are X7R, 6.3V, 20% or better unless otherwise noted\n - Tantalum capacitors should have ESR < 300mOhm\n - VDDIO, VDDD, VDDA should have 33uF of decoupling and LPF >1MHz per IMX23RM 32.2.1.1\n - The Connectors_JTAG sheet contains power selection circuitry as it is relevant to the USB connector"
- note removed: "VLF3010"
- moved on the sheet: C39, C40, IC6, L6, R24, R25, R26, R27, R28

Commit message: Updated layout.
Other:
- note added: "I2C Master (AUART)"
- note added: "Notes:\n - Capacitors are X7R, 6.3V, 20% or better unless otherwise noted\n - Tantalum capacitors should have ESR < 300mOhm\n - VDDIO, VDDD, VDDA should have 33uF of decoupling and LPF >1MHz per IMX23RM 32.2.1.1\n - Power Supply Designed to Freescale AppNote AN3883 recommendations"
- note removed: "I2C Master"
- note removed: "Notes:\n - Capacitors are X7R, 6.3V, 20% or better unless otherwise noted\n - Tantalum capacitors should have ESR < 300mOhm\n - VDDIO, VDDD, VDDA should have 33uF of decoupling and LPF >1MHz per IMX23RM 32.2.1.1\n - Power Supply Designed to Freescale AppNote AN3883 recommendations\n - The Connectors_JTAG sheet contains power selection circuitry as it is relevant to the USB connector"
Changed lines of the file:
@@
-EESchema Schematic File Version 2  date 24/04/2010 02:27:16
+EESchema Schematic File Version 2  date 25/04/2010 06:05:23
 LIBS:opendous
 LIBS:device
@@
 Sheet 7 8
 Title "PROpendous"
-Date "24 apr 2010"
+Date "25 apr 2010"
 Rev "1.0"
 Comp "Opendous Inc. (www.opendous.org)"
@@
 SPI SSP1 Flash
 Text Notes 950  5650 0    50   ~ 0
-I2C Master
+I2C Master (AUART)
 Text Notes 950  5550 0    50   ~ 0
 USB
@@
 $EndComp
 Text Notes 600  650  0    60   ~ 0
-Notes:\n - Capacitors are X7R, 6.3V, 20% or better unless otherwise noted\n - Tantalum capacitors should have ESR < 300mOhm\n - VDDIO, VDDD, VDDA should have 33uF of decoupling and LPF >1MHz per IMX23RM 32.2.1.1\n - Power Supply Designed to Freescale AppNote AN3883 recommendations\n - The Connectors_JTAG sheet contains power selection circuitry as it is relevant to the USB connector
+Notes:\n - Capacitors are X7R, 6.3V, 20% or better unless otherwise noted\n - Tantalum capacitors should have ESR < 300mOhm\n - VDDIO, VDDD, VDDA should have 33uF of decoupling and LPF >1MHz per IMX23RM 32.2.1.1\n - Power Supply Designed to Freescale AppNote AN3883 recommendations
 Text GLabel 2900 5600 0    40   BiDi ~ 0
 LCD_D00

Commit message: First revision of i.MX233-based PROpendous board is complete.
Parts:
- removed C36: 0.01uF, symbol C_MINI
- removed C74: 0.1uF, symbol C_MINI
- added TP9: CONN_1, symbol CONN_1
Connections:
- net labels added: BATT_TEMP, LM2621_FB
- wire segments 183 -> 185
Other:
- note added: "Could not route TSC2003\nIN1 to BATT_TEMP so use\nflying wire if it is needed"
- note added: "Could not route TSC2003\nVBAT1 to BATTERY"
- note added: "USB-miniB Power Input"
- moved on the sheet: C56, C57, C58, C60, C61, C62, C63, C64, C65, C66, C68, C70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

Commit message: Updated design files.  Added picture of finished PCB.
Parts:
- C37: value 68uF -> 47uF
Other:
- note added: "ESR <3-Ohm"
- note added: "High Quality <300mOhm\nTantalum Capacitor"
- note added: "Notes:\n - Capacitors are X7R, 6.3V, 20% or better unless otherwise noted\n - Tantalum capacitors should have ESR < 300mOhm but to reduce costs only use them on the noisiest rails\n - VDDIO, VDDD, VDDA should have 33uF of decoupling and LPF >1MHz per IMX23RM 32.2.1.1\n - Power Supply Designed to Freescale AppNote AN3883 recommendations"
- note removed: "Notes:\n - Capacitors are X7R, 6.3V, 20% or better unless otherwise noted\n - Tantalum capacitors should have ESR < 300mOhm\n - VDDIO, VDDD, VDDA should have 33uF of decoupling and LPF >1MHz per IMX23RM 32.2.1.1\n - Power Supply Designed to Freescale AppNote AN3883 recommendations"
Changed lines of the file:
@@
-EESchema Schematic File Version 2  date 27/04/2010 18:25:33
+EESchema Schematic File Version 2  date 07/05/2010 11:28:22
 LIBS:opendous
 LIBS:device
@@
 LIBS:valves
 LIBS:power
-LIBS:PROpendous-cache
 EELAYER 24  0
 EELAYER END
@@
 Sheet 7 8
 Title "PROpendous"
-Date "27 apr 2010"
+Date "7 may 2010"
 Rev "1.0"
 Comp "Opendous Inc. (www.opendous.org)"
@@
 Comment4 "www.PROpendous.org"
 $EndDescr
+Text Notes 1575 2225 0    30   ~ 0
+ESR <3-Ohm
+Text Notes 4600 2225 0    30   ~ 0
+ESR <3-Ohm
+Text Notes 8000 3650 0    30   ~ 0
+High Quality <300mOhm\nTantalum Capacitor
+Text Notes 7800 4600 0    30   ~ 0
+High Quality <300mOhm\nTantalum Capacitor
 Text Notes 5925 1700 0    20   ~ 0
 Could not route TSC2003\nVBAT1 to BATTERY
@@
 $EndComp
 Text Notes 600  650  0    60   ~ 0
-Notes:\n - Capacitors are X7R, 6.3V, 20% or better unless otherwise noted\n - Tantalum capacitors should have ESR < 300mOhm\n - VDDIO, VDDD, VDDA should have 33uF of decoupling and LPF >1MHz per IMX23RM 32.2.1.1\n - Power Supply Designed to Freescale AppNote AN3883 recommendations
+Notes:\n - Capacitors are X7R, 6.3V, 20% or better unless otherwise noted\n - Tantalum capacitors should have ESR < 300mOhm but to reduce costs only use them on the noisiest rails\n - VDDIO, VDDD, VDDA should have 33uF of decoupling and LPF >1MHz per IMX23RM 32.2.1.1\n - Power Supply Designed to Freescale AppNote AN3883 recommendations
 Text GLabel 2900 5700 0    40   BiDi ~ 0
 LCD_D00
@@
 P 6750 3950
 F 0 "C37" V 6700 4000 30  0000 C CNN
-F 1 "68uF" V 6800 4020 25  0000 C CNN
+F 1 "47uF" V 6800 4020 25  0000 C CNN
 	1    6750 3950
 	0    1    1    0
