File: PRopendous/Hardware/PROpendous/PROpendous-Power_Boot.sch (KiCad schematic (older format))
At the start: 65 parts, among them IC6 LM2621

Commit message: Switch to ceramic capacitors for bulk decoupling which are less expensive than similarly low-ESR tantalum capacitors.
Parts:
- removed C54, C55, C59, C69: 33uF, symbol CP_TANTALUM_MINI
- added C54, C55, C59, C69: 47uF, symbol C_MINI
- C50: value 33uF -> 47uF
- R45: value 0.1 -> 0.39
Connections:
- net labels added: TSC_AUX
- net labels removed: TSC_IN1, TSC_VBAT1
Other:
- note added: "Could not route TSC2007\nAUX to BATT_TEMP so use\nflying wire if it is needed"
- note removed: "Could not route TSC2003\nIN1 to BATT_TEMP so use\nflying wire if it is needed"
- note removed: "Could not route TSC2003\nVBAT1 to BATTERY"
- note removed: "High Quality <300mOhm\nTantalum Capacitor"
Changed lines of the file:
@@
-EESchema Schematic File Version 2  date 07/06/2010 07:15:05
+EESchema Schematic File Version 2  date 17/06/2010 09:45:34
 LIBS:opendous
 LIBS:device
@@
 LIBS:valves
 LIBS:power
-LIBS:PROpendous-cache
 EELAYER 24  0
 EELAYER END
@@
 Sheet 7 8
 Title "PROpendous"
-Date "7 jun 2010"
+Date "17 jun 2010"
 Rev "1.0"
 Comp "Opendous Inc. (www.opendous.org)"
@@
 Comment4 "www.PROpendous.org"
 $EndDescr
+$Comp
+L CP_TANTALUM_MINI C50
+U 1 1 4C1A1D46
+P 8400 2500
+F 0 "C50" V 8350 2550 30  0000 C CNN
+F 1 "47uF" V 8450 2570 25  0000 C CNN
+	1    8400 2500
+	0    1    1    0
+$EndComp
+$Comp
+L C_MINI C69
+U 1 1 4C1A1CB1
+P 9450 2700
+F 0 "C69" V 9400 2750 30  0000 C CNN
+F 1 "47uF" V 9500 2750 25  0000 C CNN
+	1    9450 2700
+	0    1    1    0
+$EndComp
+$Comp
+L CP_TANTALUM_MINI C37
+U 1 1 4BCC4827
+P 6750 3950
+F 0 "C37" V 6700 4000 30  0000 C CNN
+F 1 "47uF" V 6800 4020 25  0000 C CNN
+	1    6750 3950
+	0    1    1    0
+$EndComp
+$Comp
+L C_MINI C59
+U 1 1 4C1A193E
+P 8850 5550
+F 0 "C59" V 8800 5600 30  0000 C CNN
+F 1 "47uF" V 8900 5600 25  0000 C CNN
+	1    8850 5550
+	0    1    1    0
+$EndComp
+$Comp
+L C_MINI C54
+U 1 1 4C1A1923
+P 8450 4600
+F 0 "C54" V 8400 4650 30  0000 C CNN
+F 1 "47uF" V 8500 4650 25  0000 C CNN
+	1    8450 4600
+	0    1    1    0
+$EndComp
+$Comp
+L C_MINI C55
+U 1 1 4C1A1921
+P 8650 3650
+F 0 "C55" V 8600 3700 30  0000 C CNN
+F 1 "47uF" V 8700 3700 25  0000 C CNN
+	1    8650 3650
+	0    1    1    0
+$EndComp
 Text Notes 1575 2225 0    30   ~ 0
 ESR <3-Ohm
 Text Notes 4600 2225 0    30   ~ 0
 ESR <3-Ohm
-Text Notes 8000 3650 0    30   ~ 0
-High Quality <300mOhm\nTantalum Capacitor
-Text Notes 7800 4600 0    30   ~ 0
-High Quality <300mOhm\nTantalum Capacitor
-Text Notes 5925 1700 0    20   ~ 0
-Could not route TSC2003\nVBAT1 to BATTERY
 Wire Wire Line
 	5900 4100 5900 4050
@@
 BATT_TEMP
 Text Notes 5725 2075 0    20   ~ 0
-Could not route TSC2003\nIN1 to BATT_TEMP so use\nflying wire if it is needed
+Could not route TSC2007\nAUX to BATT_TEMP so use\nflying wire if it is needed
 $Comp
 L CONN_1 TP9
@@
 $EndComp
 Text GLabel 6000 2200 0    40   BiDi ~ 0
-TSC_IN1
+TSC_AUX
 $Comp
 L VDDIO_3V3 #PWR095
@@
 $EndComp
 $Comp
-L CP_TANTALUM_MINI C59
-U 1 1 4BCCEB1D
-P 8850 5550
-F 0 "C59" V 8800 5600 30  0000 C CNN
-F 1 "33uF" V 8900 5620 25  0000 C CNN
-	1    8850 5550
-	0    1    1    0
-$EndComp
-$Comp
 L C_MINI C65
 U 1 1 4BCCEB1C
@@
 $EndComp
 $Comp
-L CP_TANTALUM_MINI C54
-U 1 1 4BCCEB0C
-P 8450 4600
-F 0 "C54" V 8400 4650 30  0000 C CNN
-F 1 "33uF" V 8500 4670 25  0000 C CNN
-	1    8450 4600
-	0    1    1    0
-$EndComp
-$Comp
 L C_MINI C58
 U 1 1 4BCCEB0B
@@
 $EndComp
 $Comp
-L CP_TANTALUM_MINI C55
-U 1 1 4BCCEAE8
-P 8650 3650
-F 0 "C55" V 8600 3700 30  0000 C CNN
-F 1 "33uF" V 8700 3720 25  0000 C CNN
-	1    8650 3650
-	0    1    1    0
-$EndComp
-$Comp
 L C_MINI C60
 U 1 1 4BCCEAE7
@@
 P 9450 2400
 F 0 "R45" V 9425 2450 25  0000 C CNN
-F 1 "0.1" V 9475 2450 20  0000 C CNN
+F 1 "0.39" V 9475 2450 20  0000 C CNN
 	1    9450 2400
 	0    1    1    0
@@
 $EndComp
 $Comp
-L CP_TANTALUM_MINI C69
-U 1 1 4BCCE949
-P 9450 2700
-F 0 "C69" V 9400 2750 30  0000 C CNN
-F 1 "33uF" V 9500 2770 25  0000 C CNN
-	1    9450 2700
-	0    1    1    0
-$EndComp
-$Comp
 L GND #PWR0113
 U 1 1 4BCCE946
@@
 F 1 "0.1uF" V 8850 2570 25  0000 C CNN
 	1    8800 2500
-	0    1    1    0
-$EndComp
-$Comp
-L CP_TANTALUM_MINI C50
-U 1 1 4BCCE8AB
-P 8400 2500
-F 0 "C50" V 8350 2550 30  0000 C CNN
-F 1 "33uF" V 8450 2570 25  0000 C CNN
-	1    8400 2500
 	0    1    1    0
 $EndComp
@@
 Text GLabel 2900 6100 0    40   BiDi ~ 0
 LCD_RS
-Text GLabel 6300 1600 0    40   BiDi ~ 0
-TSC_VBAT1
 $Comp
 L VDD_BATT #PWR0144
@@
 $EndComp
 $Comp
-L CP_TANTALUM_MINI C37
-U 1 1 4BCC4827
-P 6750 3950
-F 0 "C37" V 6700 4000 30  0000 C CNN
-F 1 "47uF" V 6800 4020 25  0000 C CNN
-	1    6750 3950
-	0    1    1    0
-$EndComp
-$Comp

Commit message: Updated the design.  JTAG header now includes VDD_XTAL and SSP1_Detect.  1.8" LCD has been removed and LCD backlight control is now connected to GPMI_CE1n.  The clock signals for the DDR SDRAM are now the longest EMI traces at 0.76".
Connections:
- net labels added: FSUSB20_S
Other:
- note added: "FSUSB20_S, which is connected to\nPWM2-GPMI_RDY3, controls the\nUSB connector signal switch in\nthe Connectors_JTAG sheet.\n"
- note added: "Only need to mount jumpers to invert signals\nand select boot modes other than SD/MMC2"
- note added: "The LQH6PP meets the 2.5A inductor current limit of the LM2621.\nIt also meets the typical (2.85A) internal current limit. However, it\ndoes not meet the maximum internal current limit of the LM2621 (4A)."
- note removed: "PWM2-GPMI_RDY3 also controls\nUSB connector signal switch in\nthe Connectors_JTAG sheet.\n"
- note removed: "The LQH6PP meets the 2.5A inductor current limit of the LM2621.\nIt also meets the typical (2.85A) internal current limit. However, it\ndoes not meet the maximum internal current limit of the LM2621 (4A)\nwhich can occur at high temperature during a short of USB-A VBUS+GND."
