File: PRopendous/Hardware/PROpendous/PROpendous-Power_Boot.sch (KiCad schematic (older format))
At the start: 65 parts, among them IC6 LM2621

Commit message: Updated PROpendous design.  PWM2-GPMI_RDY3 now controls the LCD backlight and GPMI_CE1n now controls USB Host enable.  The function of these pins was switched as PWM2 makes more sense as a backlight control.
Connections:
- net labels added: GPMI_CE1n
- net labels removed: PWM2-GPMI_RDY3
Other:
- note added: "FSUSB20_S, which is connected to\nGPMI_CE1n, controls the\nUSB connector signal switch in\nthe Connectors_JTAG sheet.\n"
- note added: "GPMI_CE1n also controls USB Hosting\nas it controls the USB Connector Switch and\nVBUS Generator but only if/when R53 in the\nConnectors_JTAG sheet is populated.\nTo use this LED for debug purposes without\nalso switching to USB Host mode simply\ndepopulate R53.\n"
- note added: "Host/Debug Mode Enabled LED"
- note added: "Notes:\n - Capacitors are X7R, 6.3V, 20% or better unless otherwise noted\n - Tantalum capacitors should have ESR < 300mOhm but to reduce costs only use them on the noisiest rails\n - VDDIO, VDDD, VDDA should have 33uF of decoupling and LPF >1MHz per IMX23RM 32.2.1.1\n - Power Supply Designed to Freescale AppNote AN3883 recommendations\n - A PROpendous board must be self/battery-powered to meet t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"
- note added: "USB-miniB VBUS supplies power for\nLi-Ion Battery charging as well\nas board power. However,\ncurrent consumption does\nnot meet USB Suspend Mode\nrequirements."
- note removed: "Debug/Host Mode Enabled LED"
- note removed: "FSUSB20_S, which is connected to\nPWM2-GPMI_RDY3, controls the\nUSB connector signal switch in\nthe Connectors_JTAG sheet.\n"
- note removed: "Notes:\n - Capacitors are X7R, 6.3V, 20% or better unless otherwise noted\n - Tantalum capacitors should have ESR < 300mOhm but to reduce costs only use them on the noisiest rails\n - VDDIO, VDDD, VDDA should have 33uF of decoupling and LPF >1MHz per IMX23RM 32.2.1.1\n - Power Supply Designed to Freescale AppNote AN3883 recommendations"
- note removed: "PWM2-GPMI_RDY3 also controls USB\nUSB Host enable to reduce the number\nof signals stuck on the board."
- note removed: "USB-miniB VBUS supplies power for\nLi-Ion Battery charging as well\nas board power."
Changed lines of the file:
@@
-EESchema Schematic File Version 2  date 20/10/2010 05:47:04
+EESchema Schematic File Version 2  date 21/10/2010 09:30:50
 LIBS:opendous
 LIBS:device
@@
 Sheet 7 8
 Title "PROpendous"
-Date "20 oct 2010"
-Rev "1.0"
+Date "21 oct 2010"
+Rev "1.1"
 Comp "Opendous Inc. (www.opendous.org)"
 Comment1 ""
@@
 Comment4 "www.PROpendous.org"
 $EndDescr
+Text Notes 1450 4200 0    40   ~ 0
+GPMI_CE1n also controls USB Hosting\nas it controls the USB Connector Switch and\nVBUS Generator but only if/when R53 in the\nConnectors_JTAG sheet is populated.\nTo use this LED for debug purposes without\nalso switching to USB Host mode simply\ndepopulate R53.\n
 Text Notes 950  7050 0    50   ~ 0
 Only need to mount jumpers to invert signals\nand select boot modes other than SD/MMC2
@@
 2.85A Max
 Text Notes 5900 4350 0    40   ~ 0
-USB-miniB VBUS supplies power for\nLi-Ion Battery charging as well\nas board power.
-Text Notes 1450 4150 0    40   ~ 0
-PWM2-GPMI_RDY3 also controls USB\nUSB Host enable to reduce the number\nof signals stuck on the board.
+USB-miniB VBUS supplies power for\nLi-Ion Battery charging as well\nas board power.  However,\ncurrent consumption does\nnot meet USB Suspend Mode\nrequirements.
 Text GLabel 1950 3950 0    40   BiDi ~ 0
-PWM2-GPMI_RDY3
+GPMI_CE1n
 $Comp
 L D_LED D3
@@
 $EndComp
 Text Notes 1450 3750 0    50   Italic 10
-Debug/Host Mode Enabled LED
+Host/Debug Mode Enabled LED
 Text Notes 3450 3750 0    50   Italic 10
 Power ON LED
@@
 $EndComp
 Text Notes 700  2700 0    40   ~ 0
-FSUSB20_S, which is connected to\nPWM2-GPMI_RDY3, controls the\nUSB connector signal switch in\nthe Connectors_JTAG sheet.\n
+FSUSB20_S, which is connected to\nGPMI_CE1n, controls the\nUSB connector signal switch in\nthe Connectors_JTAG sheet.\n
 $Comp
 L GND #PWR0117
@@
 $EndComp
 Text Notes 600  650  0    60   ~ 0
-Notes:\n - Capacitors are X7R, 6.3V, 20% or better unless otherwise noted\n - Tantalum capacitors should have ESR < 300mOhm but to reduce costs only use them on the noisiest rails\n - VDDIO, VDDD, VDDA should have 33uF of decoupling and LPF >1MHz per IMX23RM 32.2.1.1\n - Power Supply Designed to Freescale AppNote AN3883 recommendations
+Notes:\n - Capacitors are X7R, 6.3V, 20% or better unless otherwise noted\n - Tantalum capacitors should have ESR < 300mOhm but to reduce costs only use them on the noisiest rails\n - VDDIO, VDDD, VDDA should have 33uF of decoupling and LPF >1MHz per IMX23RM 32.2.1.1\n - Power Supply Designed to Freescale AppNote AN3883 recommendations\n - A PROpendous board must be self/battery-powered to meet the USB Specification's current consumption requirements for USB Suspend mode
 Text GLabel 2900 5700 0    40   BiDi ~ 0
 LCD_D00
