File: PRopendous/Hardware/PROpendous/PROpendous-Audio.sch (KiCad schematic (older format))
At the start: 30 parts, among them IC7 MMA7455, M1 ELECTRET_MIC, U7 Video, U8 Headphones, U9 Line

Commit message: Updated PROpendous design.  PWM2-GPMI_RDY3 now controls the LCD backlight and GPMI_CE1n now controls USB Host enable.  The function of these pins was switched as PWM2 makes more sense as a backlight control.
Other:
- note added: "nCS=1 enables I2C interface"
Changed lines of the file:
@@
-EESchema Schematic File Version 2  date 20/10/2010 05:47:04
+EESchema Schematic File Version 2  date 21/10/2010 09:30:50
 LIBS:opendous
 LIBS:device
@@
 Sheet 6 8
 Title "PROpendous"
-Date "20 oct 2010"
-Rev "1.0"
+Date "21 oct 2010"
+Rev "1.1"
 Comp "Opendous Inc. (www.opendous.org)"
 Comment1 ""
@@
 Comment4 "www.PROpendous.org"
 $EndDescr
+Text Notes 3850 6100 0    30   ~ 0
+nCS=1 enables I2C interface
 Text GLabel 6600 7650 2    40   BiDi ~ 0
 MIC_OUT
