File: PROpendous/Hardware/PROpendous/PROpendous-Connectors_JTAG.sch (KiCad schematic (older format))
At the start: 23 parts, among them IC5 FSUSB20, P1 Serial-JTAG, P2 Expansion, U2 microSD, U3 SD, U4 ARM_JTAG, U5 USB-miniB, U6 USB-A

Commit message: Updated all design files with CC0 Public Domain License.  Added single PDF version of schematic.  Updated the layout's GND fill to solid instead of thermal.  Kept previous revision Gerbers.
Connections:
- net labels added: GPMI_ALE, GPMI_CLE, GPMI_D00-SSP2_DATA0, GPMI_D01-SSP2_DATA1, GPMI_D02-SSP2_DATA2, GPMI_D03-SSP2_DATA3, GPMI_D04-SSP2_DATA4, GPMI_D05-SSP2_DATA5, GPMI_D06-SSP2_DATA6, GPMI_D07-SSP2_DATA7
- net labels removed: GPMI_ALE-LCD_D17, GPMI_CLE-LCD_D16, GPMI_D00-LCD_D8-SSP2_DATA0, GPMI_D01-LCD_D9-SSP2_DATA1, GPMI_D02-LCD_D10-SSP2_DATA2, GPMI_D03-LCD_D11-SSP2_DATA3, GPMI_D04-LCD_D12-SSP2_DATA4, GPMI_D05-LCD_D13-SSP2_DATA5, GPMI_D06-LCD_D14-SSP2_DATA6, GPMI_D07-LCD_D15-SSP2_DATA7
- wire segments 77 -> 89
Changed lines of the file:
@@
-EESchema Schematic File Version 2  date 21/10/2010 18:49:25
-LIBS:opendous
+EESchema Schematic File Version 2  date 10/2/2012 6:21:31 PM
 LIBS:device
 LIBS:transistors
@@
 LIBS:power
 LIBS:PROpendous-cache
-EELAYER 24  0
+EELAYER 25  0
 EELAYER END
 $Descr A4 11700 8267
+encoding utf-8
 Sheet 4 8
 Title "PROpendous"
-Date "21 oct 2010"
-Rev "1.1"
+Date "2 oct 2012"
+Rev "1.2"
 Comp "Opendous Inc. (www.opendous.org)"
-Comment1 ""
-Comment2 "http://creativecommons.org/licenses/by/3.0/"
-Comment3 "Copyright Under the Creative Commons Attribution License"
-Comment4 "www.PROpendous.org"
+Comment1 "Opendous Inc. deeded this hardware design into the Public Domain"
+Comment2 "http://creativecommons.org/publicdomain/zero/1.0/"
+Comment3 "No Copyright - Deeded under the Creative Commons CC0 Public Domain Dedication"
+Comment4 "For more information visit www.PROpendous.org"
 $EndDescr
-Text Notes 2350 2600 0    40   ~ 0
-101-00303-68
-Text Notes 4300 6150 0    40   ~ 0
-Depopulating R53 will allow you\nto use the Host/Debug LED in the\nPower_Boot sheet without also\nenabling USB Hosting
+Connection ~ 3250 5650
+Connection ~ 3250 5750
+Connection ~ 2350 6050
+Connection ~ 2350 5950
+Connection ~ 2350 5750
+Connection ~ 2350 5650
+Wire Wire Line
+	2350 5600 2350 5650
+Wire Wire Line
+	2350 5600 2300 5600
+Wire Wire Line
+	2350 5900 2350 5950
+Wire Wire Line
+	2350 5900 2300 5900
+Wire Wire Line
+	3250 5700 3250 5750
+Wire Wire Line
+	3250 5700 3300 5700
 Wire Wire Line
 	4200 5650 4300 5650
@@
 Wire Wire Line
 	4750 3450 4750 3550
+Wire Wire Line
+	3300 5600 3250 5600
+Wire Wire Line
+	3250 5600 3250 5650
+Wire Wire Line
+	2300 6000 2350 6000
+Wire Wire Line
+	2350 6000 2350 6050
+Wire Wire Line
+	2300 5700 2350 5700
+Wire Wire Line
+	2350 5700 2350 5750
+Text Notes 2350 2600 0    40   ~ 0
+101-00303-68
+Text Notes 4300 6150 0    40   ~ 0
+Depopulating R53 will allow you\nto use the Host/Debug LED in the\nPower_Boot sheet without also\nenabling USB Hosting
 $Comp
 L C_MINI C85
@@
 	0    -1   -1   0
 $EndComp
-Text Label 6450 7650 2    40   ~ 0
-FSUSB20_S
-Text GLabel 6450 7650 2    40   Input ~ 0
-FSUSB20_S
-Text Label 3250 5650 0    30   ~ 0
+Text GLabel 3300 5600 2    20   Input ~ 0
 FSUSB20_S
 $Comp
@@
 	1    0    0    -1
 $EndComp
-Text GLabel 6450 7350 2    40   Input ~ 0
+Text GLabel 2300 5900 0    20   UnSpc ~ 0
 DPb
-Text GLabel 6450 7450 2    40   Input ~ 0
+Text GLabel 2300 6000 0    20   UnSpc ~ 0
 DMb
-Text GLabel 6450 7250 2    40   Input ~ 0
+Text GLabel 2300 5700 0    20   UnSpc ~ 0
 DMa
-Text GLabel 6450 7150 2    40   Input ~ 0
+Text GLabel 2300 5600 0    20   UnSpc ~ 0
 DPa
-Text Label 6450 7150 2    40   ~ 0
-DPa
-Text Label 6450 7250 2    40   ~ 0
-DMa
-Text Label 6450 7450 2    40   ~ 0
-DMb
-Text Label 6450 7350 2    40   ~ 0
-DPb
 $Comp
 L C_MINI C75
@@
 	1    0    0    -1
 $EndComp
-Text GLabel 6450 7550 2    40   Input ~ 0
-FSUSB20_nOE
-Text Label 3250 5750 0    30   ~ 0
-FSUSB20_nOE
-Text Label 6450 7550 2    40   ~ 0
+Text GLabel 3300 5700 2    20   Input ~ 0
 FSUSB20_nOE
 Text Notes 8200 4100 0    80   Italic 16
@@
 	0    1    1    0
 $EndComp
-Text Label 2350 5950 2    40   ~ 0
-DPb
-Text Label 2350 6050 2    40   ~ 0
-DMb
-Text Label 2350 5750 2    40   ~ 0
-DMa
-Text Label 2350 5650 2    40   ~ 0
-DPa
 $Comp
 L GND #PWR052
@@
 GPMI_CE1n
 Text GLabel 2250 1750 0    40   BiDi ~ 0
-GPMI_D00-LCD_D8-SSP2_DATA0
+GPMI_D00-SSP2_DATA0
 Text GLabel 2250 1650 0    40   BiDi ~ 0
-GPMI_D01-LCD_D9-SSP2_DATA1
+GPMI_D01-SSP2_DATA1
 Text GLabel 2250 1900 0    40   BiDi ~ 0
 GPMI_WRn-SSP2_SCK
@@
 SSP1_CMD-JTAG_TDO
 Text GLabel 2250 1550 0    40   BiDi ~ 0
-GPMI_D02-LCD_D10-SSP2_DATA2
+GPMI_D02-SSP2_DATA2
 Text GLabel 4400 2150 0    40   BiDi ~ 0
 SSP1_DATA0-JTAG_TDI
 Text GLabel 2250 1450 0    40   BiDi ~ 0
-GPMI_D03-LCD_D11-SSP2_DATA3
+GPMI_D03-SSP2_DATA3
 Text GLabel 4400 2050 0    40   BiDi ~ 0
 SSP1_DATA1-I2C_SCL-JTAG_TCLK
@@
 LCD_CS
 Text GLabel 8250 2500 0    40   BiDi ~ 0
-GPMI_ALE-LCD_D17
+GPMI_ALE
 Text GLabel 7300 4900 0    40   BiDi ~ 0
 SSP1_SCK-JTAG_TRST
@@
 LCD_RESET-GPMI_CE3n
 Text GLabel 8250 2600 0    40   BiDi ~ 0
-GPMI_D00-LCD_D8-SSP2_DATA0
+GPMI_D00-SSP2_DATA0
 Text GLabel 8250 3100 0    40   BiDi ~ 0
 GPMI_RDY0-SSP2_DETECT
@@
 LCD_WR
 Text GLabel 9050 2700 2    40   BiDi ~ 0
-GPMI_D01-LCD_D9-SSP2_DATA1
+GPMI_D01-SSP2_DATA1
 Text GLabel 9050 3200 2    40   BiDi ~ 0
 GPMI_WRn-SSP2_SCK
@@
 LCD_RS
 Text GLabel 8250 2700 0    40   BiDi ~ 0
-GPMI_D02-LCD_D10-SSP2_DATA2
+GPMI_D02-SSP2_DATA2
 Text GLabel 8250 3200 0    40   BiDi ~ 0
 GPMI_WPn
@@
 LCD_HSYNC-I2C_SDA
 Text GLabel 9050 2800 2    40   BiDi ~ 0
-GPMI_D03-LCD_D11-SSP2_DATA3
+GPMI_D03-SSP2_DATA3
 Text GLabel 9050 2400 2    40   BiDi ~ 0
 LCD_VSYNC-LCD_BUSY
 Text GLabel 9050 2900 2    40   BiDi ~ 0
-GPMI_D05-LCD_D13-SSP2_DATA5
+GPMI_D05-SSP2_DATA5
 Text GLabel 7300 5300 0    40   BiDi ~ 0
 SSP1_DATA2-I2C_SDA-JTAG_RTCK
@@
 LCD_DOTCK-GPMI_RDY3
 Text GLabel 8250 2800 0    40   BiDi ~ 0
-GPMI_D04-LCD_D12-SSP2_DATA4
+GPMI_D04-SSP2_DATA4
 Text GLabel 7300 5100 0    40   BiDi ~ 0
 SSP1_DATA3-JTAG_TMS
 Text GLabel 9050 3000 2    40   BiDi ~ 0
-GPMI_D07-LCD_D15-SSP2_DATA7
+GPMI_D07-SSP2_DATA7
 Text GLabel 9050 2500 2    40   BiDi ~ 0
-GPMI_CLE-LCD_D16
+GPMI_CLE
 Text GLabel 8250 2900 0    40   BiDi ~ 0
-GPMI_D06-LCD_D14-SSP2_DATA6
+GPMI_D06-SSP2_DATA6
 Text GLabel 8250 1500 0    40   BiDi ~ 0
 PWM0-ROTARYA-DUART_RX
