File: PROpendous/Hardware/PROpendous/PROpendous-LCD.sch (KiCad schematic (older format))
At the start: 24 parts, among them IC3 TSC2007, Q1 2N7002, U1 NHD-2.4-240320SF-CTXI-T

Commit message: Updated all design files with CC0 Public Domain License.  Added single PDF version of schematic.  Updated the layout's GND fill to solid instead of thermal.  Kept previous revision Gerbers.
Connections:
- wire segments 65 -> 75
Changed lines of the file:
@@
-EESchema Schematic File Version 2  date 21/10/2010 09:30:50
-LIBS:opendous
+EESchema Schematic File Version 2  date 10/2/2012 6:21:31 PM
 LIBS:device
 LIBS:transistors
@@
 LIBS:power
 LIBS:PROpendous-cache
-EELAYER 24  0
+EELAYER 25  0
 EELAYER END
 $Descr A4 11700 8267
+encoding utf-8
 Sheet 5 8
 Title "PROpendous"
-Date "21 oct 2010"
-Rev "1.1"
+Date "2 oct 2012"
+Rev "1.2"
 Comp "Opendous Inc. (www.opendous.org)"
-Comment1 ""
-Comment2 "http://creativecommons.org/licenses/by/3.0/"
-Comment3 "Copyright Under the Creative Commons Attribution License"
-Comment4 "www.PROpendous.org"
+Comment1 "Opendous Inc. deeded this hardware design into the Public Domain"
+Comment2 "http://creativecommons.org/publicdomain/zero/1.0/"
+Comment3 "No Copyright - Deeded under the Creative Commons CC0 Public Domain Dedication"
+Comment4 "For more information visit www.PROpendous.org"
 $EndDescr
+Connection ~ 5250 3250
+Wire Wire Line
+	5250 3200 5250 3250
+Wire Wire Line
+	5250 3200 5200 3200
+Connection ~ 4100 4250
+Connection ~ 4100 4350
+Connection ~ 4100 4450
+Connection ~ 4100 4550
+Wire Wire Line
+	4100 4500 4100 4550
+Wire Wire Line
+	4100 4500 4150 4500
+Wire Wire Line
+	4100 4300 4100 4350
+Wire Wire Line
+	4100 4300 4150 4300
+Connection ~ 3650 5800
+Wire Wire Line
+	3650 5700 3650 5800
+Connection ~ 3650 6000
+Wire Wire Line
+	3650 6000 3650 6100
+Wire Wire Line
+	2150 6450 2150 6350
+Wire Wire Line
+	2150 6350 2250 6350
+Wire Wire Line
+	3900 3000 3900 2950
+Connection ~ 2500 4350
+Wire Wire Line
+	2100 4350 2275 4350
+Wire Wire Line
+	2275 4350 2275 4325
+Wire Wire Line
+	2275 4325 2325 4325
+Wire Wire Line
+	2325 4325 2325 4350
+Wire Wire Line
+	2325 4350 3200 4350
+Wire Wire Line
+	5050 4100 5250 4100
+Wire Wire Line
+	5050 3900 5250 3900
+Connection ~ 3900 3250
+Wire Wire Line
+	5250 3250 3850 3250
+Wire Wire Line
+	3000 5100 3000 4900
+Wire Wire Line
+	3000 4900 3200 4900
+Connection ~ 2500 3950
+Wire Wire Line
+	2300 3950 2700 3950
+Wire Wire Line
+	2500 4150 2500 4350
+Wire Wire Line
+	3650 5350 3650 5250
+Wire Wire Line
+	4100 4550 5250 4550
+Wire Wire Line
+	4100 4350 5250 4350
+Wire Wire Line
+	4800 3800 4800 4100
+Wire Wire Line
+	4800 3800 4850 3800
+Connection ~ 4800 3900
+Wire Wire Line
+	4850 4000 4800 4000
+Wire Wire Line
+	4200 3650 4200 3700
+Wire Wire Line
+	4200 3700 4300 3700
+Wire Wire Line
+	5850 2750 5950 2750
+Connection ~ 5900 5300
+Wire Wire Line
+	6100 5300 5700 5300
+Wire Wire Line
+	5900 5600 5900 5500
+Connection ~ 5900 4750
+Wire Wire Line
+	5800 4750 6000 4750
+Wire Wire Line
+	5250 3100 4200 3100
+Wire Wire Line
+	5900 4850 5900 4750
+Wire Wire Line
+	6100 5500 5700 5500
+Connection ~ 5900 5500
+Wire Wire Line
+	5250 3700 4700 3700
+Wire Wire Line
+	4200 2900 4200 2650
+Wire Wire Line
+	5900 2650 5900 2750
+Connection ~ 5900 2750
+Wire Wire Line
+	5900 5200 5900 5300
+Wire Wire Line
+	4800 3900 4850 3900
+Wire Wire Line
+	4800 4100 4850 4100
+Connection ~ 4800 4000
+Wire Wire Line
+	4800 3950 4700 3950
+Wire Wire Line
+	4700 3950 4700 4000
+Connection ~ 4800 3950
+Wire Wire Line
+	5250 4250 4100 4250
+Wire Wire Line
+	5250 4450 4100 4450
+Wire Wire Line
+	3650 4050 3650 3950
+Wire Wire Line
+	2700 4150 2700 4250
+Wire Wire Line
+	2300 4500 2300 4150
+Wire Wire Line
+	2500 3850 2500 3950
+Wire Wire Line
+	3200 5000 3000 5000
+Connection ~ 3000 5000
+Wire Wire Line
+	5050 3800 5250 3800
+Wire Wire Line
+	5250 4000 5050 4000
+Wire Wire Line
+	3200 4250 2525 4250
+Wire Wire Line
+	2525 4250 2525 4225
+Wire Wire Line
+	2525 4225 2475 4225
+Wire Wire Line
+	2475 4225 2475 4250
+Wire Wire Line
+	2475 4250 2325 4250
+Wire Wire Line
+	2325 4250 2325 4225
+Wire Wire Line
+	2325 4225 2275 4225
+Wire Wire Line
+	2275 4225 2275 4250
+Wire Wire Line
+	2275 4250 2100 4250
+Connection ~ 2700 4250
+Wire Wire Line
+	3900 3200 3900 3250
+Wire Wire Line
+	4400 4000 4000 4000
+Wire Wire Line
+	4000 4000 4000 3600
+Wire Wire Line
+	4000 3600 3900 3600
+Wire Wire Line
+	3550 6000 3750 6000
+Wire Wire Line
+	3550 5800 3750 5800
+Wire Wire Line
+	4150 4200 4100 4200
+Wire Wire Line
+	4100 4200 4100 4250
+Wire Wire Line
+	4150 4400 4100 4400
+Wire Wire Line
+	4100 4400 4100 4450
+Wire Wire Line
+	2100 4500 3200 4500
+Connection ~ 2300 4500
 Text Notes 1750 5750 0    50   ~ 0
 These signals are exposed\nfor TSC2003 compatibility
@@
 	1    0    0    -1
 $EndComp
-Text GLabel 6300 7550 0    40   BiDi ~ 0
+Text GLabel 5200 3200 0    20   UnSpc ~ 0
 LCD_RD
-Text Label 6300 7550 0    30   ~ 0
-LCD_RD
-Text Label 3200 4500 2    30   ~ 0
+Text GLabel 2100 4500 0    40   Output ~ 0
 TSC_PENIRQ
-Text Label 6300 7650 0    30   ~ 0
-TSC_PENIRQ
-Text GLabel 6300 7650 0    40   BiDi ~ 0
-TSC_PENIRQ
-Connection ~ 3650 5800
-Wire Wire Line
-	3650 5700 3650 5800
-Connection ~ 3650 6000
-Wire Wire Line
-	3650 6000 3650 6100
-Wire Wire Line
-	2150 6450 2150 6350
-Wire Wire Line
-	2150 6350 2250 6350
-Wire Wire Line
-	3900 3000 3900 2950
-Connection ~ 2500 4350
-Wire Wire Line
-	2100 4350 2275 4350
-Wire Wire Line
-	2275 4350 2275 4325
-Wire Wire Line
-	2275 4325 2325 4325
-Wire Wire Line
-	2325 4325 2325 4350
-Wire Wire Line
-	2325 4350 3200 4350
-Wire Wire Line
-	5050 4100 5250 4100
-Wire Wire Line
-	5050 3900 5250 3900
-Connection ~ 3900 3250
-Wire Wire Line
-	3850 3250 5250 3250
-Wire Wire Line
-	3000 5100 3000 4900
-Wire Wire Line
-	3000 4900 3200 4900
-Connection ~ 2500 3950
-Wire Wire Line
-	2300 3950 2700 3950
-Wire Wire Line
-	2500 4150 2500 4350
-Wire Wire Line
-	3650 5350 3650 5250
-Wire Wire Line
-	4100 4550 5250 4550
-Wire Wire Line
-	4100 4350 5250 4350
-Wire Wire Line
-	4800 3800 4800 4100
-Wire Wire Line
-	4800 3800 4850 3800
-Connection ~ 4800 3900
-Wire Wire Line
-	4850 4000 4800 4000
-Wire Wire Line
-	4200 3650 4200 3700
-Wire Wire Line
-	4200 3700 4300 3700
-Wire Wire Line
-	5850 2750 5950 2750
-Connection ~ 5900 5300
-Wire Wire Line
-	6100 5300 5700 5300
-Wire Wire Line
-	5900 5600 5900 5500
-Connection ~ 5900 4750
-Wire Wire Line
-	5800 4750 6000 4750
-Wire Wire Line
-	5250 3100 4200 3100
-Wire Wire Line
-	5900 4850 5900 4750
-Wire Wire Line
-	6100 5500 5700 5500
-Connection ~ 5900 5500
-Wire Wire Line
-	5250 3700 4700 3700
-Wire Wire Line
-	4200 2900 4200 2650
-Wire Wire Line
-	5900 2650 5900 2750
-Connection ~ 5900 2750
-Wire Wire Line
-	5900 5200 5900 5300
-Wire Wire Line
-	4800 3900 4850 3900
-Wire Wire Line
-	4800 4100 4850 4100
-Connection ~ 4800 4000
-Wire Wire Line
-	4800 3950 4700 3950
-Wire Wire Line
-	4700 3950 4700 4000
-Connection ~ 4800 3950
-Wire Wire Line
-	4100 4250 5250 4250
-Wire Wire Line
-	4100 4450 5250 4450
-Wire Wire Line
-	3650 4050 3650 3950
-Wire Wire Line
-	2700 4150 2700 4250
-Wire Wire Line
-	3200 4500 2300 4500
-Wire Wire Line
-	2300 4500 2300 4150
-Wire Wire Line
-	2500 3850 2500 3950
-Wire Wire Line
-	3200 5000 3000 5000
-Connection ~ 3000 5000
-Wire Wire Line
-	5050 3800 5250 3800
-Wire Wire Line
-	5250 4000 5050 4000
-Wire Wire Line
-	3200 4250 2525 4250
-Wire Wire Line
-	2525 4250 2525 4225
-Wire Wire Line
-	2525 4225 2475 4225
-Wire Wire Line
-	2475 4225 2475 4250
-Wire Wire Line
-	2475 4250 2325 4250
-Wire Wire Line
-	2325 4250 2325 4225
-Wire Wire Line
-	2325 4225 2275 4225
-Wire Wire Line
-	2275 4225 2275 4250
-Wire Wire Line
-	2275 4250 2100 4250
-Connection ~ 2700 4250
-Wire Wire Line
-	3900 3200 3900 3250
-Wire Wire Line
-	4400 4000 4000 4000
-Wire Wire Line
-	4000 4000 4000 3600
-Wire Wire Line
-	4000 3600 3900 3600
-Wire Wire Line
-	3550 6000 3750 6000
-Wire Wire Line
-	3550 5800 3750 5800
 $Comp
 L CP_TANTALUM_MINI C78
@@
 	1    0    0    -1
 $EndComp
-Text GLabel 6300 7450 0    40   BiDi ~ 0
+Text GLabel 4150 4500 2    20   UnSpc ~ 0
 Y-
-Text GLabel 6300 7250 0    40   BiDi ~ 0
+Text GLabel 4150 4300 2    20   UnSpc ~ 0
 Y+
-Text GLabel 6300 7350 0    40   BiDi ~ 0
+Text GLabel 4150 4400 2    20   UnSpc ~ 0
 X+
-Text GLabel 6300 7150 0    40   BiDi ~ 0
+Text GLabel 4150 4200 2    20   UnSpc ~ 0
 X-
-Text Label 6300 7350 0    30   ~ 0
-X+
-Text Label 6300 7150 0    30   ~ 0
-X-
-Text Label 6300 7450 0    30   ~ 0
-Y-
-Text Label 6300 7250 0    30   ~ 0
-Y+
 Text GLabel 2250 6050 0    40   BiDi ~ 0
 TSC_VBAT1
@@
 	1    0    0    -1
 $EndComp
-Text Label 4100 4350 0    30   ~ 0
-Y+
-Text Label 4100 4550 0    30   ~ 0
-Y-
-Text Label 4100 4250 0    30   ~ 0
-X-
-Text Label 4100 4450 0    30   ~ 0
-X+
 $Comp
 L VDDIO_3V3 #PWR075
@@
 	1    0    0    -1
 $EndComp
-Text Label 5250 3250 2    30   ~ 0
-LCD_RD
 Text Label 5250 3700 2    30   ~ 0
 LCD_LED_A
