File: PROpendous/Hardware/PROpendous/PROpendous-iMX233.sch (KiCad schematic (older format))
At the start: 21 parts, among them IC1 i.MX233, IC8 24C512, SW1 POWER, X1 24MHz

Commit message: Updated all design files with CC0 Public Domain License.  Added single PDF version of schematic.  Updated the layout's GND fill to solid instead of thermal.  Kept previous revision Gerbers.
Parts:
- removed IC8: 24C512, symbol 24C512
- added IC8: EEPROM, symbol 24XX512_EEPROM
Connections:
- net labels added: GPMI_ALE, GPMI_CLE, GPMI_D00-SSP2_DATA0, GPMI_D01-SSP2_DATA1, GPMI_D02-SSP2_DATA2, GPMI_D03-SSP2_DATA3, GPMI_D04-SSP2_DATA4, GPMI_D05-SSP2_DATA5, GPMI_D06-SSP2_DATA6, GPMI_D07-SSP2_DATA7
- net labels removed: GPMI_ALE-LCD_D17, GPMI_CLE-LCD_D16, GPMI_D00-LCD_D8-SSP2_DATA0, GPMI_D01-LCD_D9-SSP2_DATA1, GPMI_D02-LCD_D10-SSP2_DATA2, GPMI_D03-LCD_D11-SSP2_DATA3, GPMI_D04-LCD_D12-SSP2_DATA4, GPMI_D05-LCD_D13-SSP2_DATA5, GPMI_D06-LCD_D14-SSP2_DATA6, GPMI_D07-LCD_D15-SSP2_DATA7, TSC_AUX, TSC_IN2, TSC_VBAT1, TSC_VBAT2, TSC_VREF
- wire segments 61 -> 67
Other:
- note removed: "Always create netlist from this sheet"
- note removed: "Global-Local labels are used to\nforce proper net names in pcbnew"
- moved on the sheet: ENCLOSURE_HAMMOND_1553B_BAT_1, L15, L17, L2, R52
